Commit message: changed the link base_link visual to actual dimensions of the piro3

File: mybot_description/urdf/piro.xacro (robot description, xacro)
@@ -24,13 +24,15 @@
   <!-- Parametros do base_link-->
   <link name="base_link">
-    <visual>
-      <geometry>
-        <box size="0.3 0.1434 0.232"/>
-      </geometry>
-      <material name="grey"/>
-    </visual>
-    <visual>
-      <geometry>
-        <box size="0.034 0.034 0.279"/>
+    <!-- This visual represents the base body of the piro in which the arms will be coupled -->
+    <visual name = 'base_body'>
+      <geometry>
+        <box size="0.3219 0.1461 0.2357"/>
+      </geometry>
+      <material name="grey"/>
+    </visual>
+    <!-- This visual represents the central stem -->
+    <visual name = 'central_stem'>
+      <geometry>
+        <box size="0.0367 0.0367 0.279"/>
       </geometry>
       <material name="grey"/>
@@ -46,5 +48,6 @@
 		</visual>
     -->
-    <visual>
+    <!-- This visual represents the claw's base in the central stem -->
+    <visual name = 'central_claw_base'>
       <geometry>
         <mesh filename="package://mybot_description/meshes/dxl_mx106.dae"/>

Commit message: add collision name in link  base_link and added collision for central claw base

File: mybot_description/urdf/piro.xacro (robot description, xacro)
@@ -56,15 +56,20 @@
       <origin rpy="0 0 0" xyz="0.0 0.0722 0.3554"/>
     </visual>
-    <collision>
-      <geometry>
-        <box size="0.3 0.1434 0.232"/>
+    <collision name = 'base_body'>
+      <geometry>
+        <box size="0.3219 0.1461 0.2357"/>
       </geometry>
       <origin rpy="0 0 0" xyz="0.0 0.0 0"/>
     </collision>
-    <collision>
-      <geometry>
-        <box size="0.03 0.03 0.232"/>
+    <collision name = 'central_stem'>
+      <geometry>
+        <box size="0.0367 0.0367 0.279"/>
       </geometry>
       <origin rpy="0 0.0 0" xyz="0.0 0.03 0.25"/>
+    </collision>
+    <collision name ='central_claw_base'>
+      <geometry>
+        <mesh filename="package://mybot_description/meshes/dxl_mx106.dae"/>
+      </geometry>
     </collision>
     <inertial>

Commit message: added commits explaining some of the caracteristics of joint named joint_garra_ap and the link named garra_ap, also fixed collision of the link

File: mybot_description/urdf/piro.xacro (robot description, xacro)
@@ -24,5 +24,5 @@
   <!-- Parametros do base_link-->
   <link name="base_link">
-    <!-- This visual represents the base body of the piro in which the arms will be coupled -->
+    <!-- This visual represents the base body-->
     <visual name = 'base_body'>
       <geometry>
@@ -49,4 +49,5 @@
     -->
     <!-- This visual represents the claw's base in the central stem -->
+    <!-- Need to check mesh design to see if dimensions is the same as the actual dimensions of piro3 -->
     <visual name = 'central_claw_base'>
       <geometry>
@@ -56,4 +57,5 @@
       <origin rpy="0 0 0" xyz="0.0 0.0722 0.3554"/>
     </visual>
+    <!-- This collision is for the base_body -->
     <collision name = 'base_body'>
       <geometry>
@@ -62,4 +64,5 @@
       <origin rpy="0 0 0" xyz="0.0 0.0 0"/>
     </collision>
+    <!-- This collision is for the central_stem -->
     <collision name = 'central_stem'>
       <geometry>
@@ -68,4 +71,5 @@
       <origin rpy="0 0.0 0" xyz="0.0 0.03 0.25"/>
     </collision>
+    <!-- This collision is for the central_claw_base -->
     <collision name ='central_claw_base'>
       <geometry>
@@ -95,5 +99,7 @@
   <!-- Parametros da garra-->
   <link name="garra_ap">
-    <visual>
+    <!-- This visual represents the central claw unit -->
+    <!-- Need to check mesh design to see if dimensions is the same as the actual dimensions of piro3 -->
+    <visual name = 'central_claw'>
       <geometry>
         <mesh filename="package://mybot_description/meshes/claw.dae"/>
@@ -101,9 +107,9 @@
       <material name="grey"/>
     </visual>
-    <collision>
-      <geometry>
-        <box size="0.048 0.064 0.1851"/>
-      </geometry>
-      <origin rpy="0 0 0" xyz="0.0 0.017 0.09255"/>
+    <!-- This collision is for the central claw unit -->
+    <collision name = 'central_claw'>
+      <geometry>
+        <mesh filename="package://mybot_description/meshes/claw.dae"/>
+      </geometry>
     </collision>
     <inertial>

Commit message: Addind commits to joint named joint_eixo_tracao_ap and link named eixo_tracao_ap

File: mybot_description/urdf/piro.xacro (robot description, xacro)
@@ -84,5 +84,5 @@
     </inertial>
   </link>
-  <!-- this joint binds the base_link with the claw central unit (represented by the link garra). It can rotate with the z axis fixed, it has an upper limit of 3,14 (180º) and a lower limit of -3,14 (-180º) -->
+  <!-- this joint binds the base_link with the claw central unit (represented by the link garra). It can rotate with the z axis fixed, it has an upper limit of 3,14 (180 degrees) and a lower limit of -3,14 (-180 degrees) -->
   <joint name="joint_garra_ap" type="revolute">
     <parent link="base_link"/>
@@ -114,23 +114,4 @@
     </inertial>
   </link>
-  <!-- Eixo AP -->
-  <!-- Parametros do eixo-->
-  <link name="eixo_tracao_ap">
-    <visual>
-      <geometry>
-        <mesh filename="package://mybot_description/meshes/shaft_simple.dae"/>
-      </geometry>
-    </visual>
-    <collision>
-      <geometry>
-        <mesh filename="package://mybot_description/meshes/shaft_simple.dae"/>
-      </geometry>
-    </collision>
-    <inertial>
-      <origin rpy="0 0 0" xyz="0.0 0.026065 0.0"/>
-      <mass value="0.1"/>
-      <inertia ixx="4.94e-05" ixy="0.0" ixz="0.0" iyy="6.11e-05" iyz="0.0" izz="4.94e-05"/>
-    </inertial>
-  </link>
   <joint name="joint_eixo_tracao_ap" type="continuous">
     <parent link="garra_ap"/>
@@ -140,4 +121,22 @@
     <dynamics damping="0.7" friction="1.0" />
   </joint>
+  <!-- this link involves the central traction unit -->
+  <link name="eixo_tracao_ap">
+    <visual>
+      <geometry>
+        <mesh filename="package://mybot_description/meshes/shaft_simple.dae"/>
+      </geometry>
+    </visual>
+    <collision>
+      <geometry>
+        <mesh filename="package://mybot_description/meshes/shaft_simple.dae"/>
+      </geometry>
+    </collision>
+    <inertial>
+      <origin rpy="0 0 0" xyz="0.0 0.026065 0.0"/>
+      <mass value="0.1"/>
+      <inertia ixx="4.94e-05" ixy="0.0" ixz="0.0" iyy="6.11e-05" iyz="0.0" izz="4.94e-05"/>
+    </inertial>
+  </link>
   <!-- JUNTA 1 -->
   <!-- Dimensoes do link1 collision -->

Commit message: Fixing commits and errors

File: mybot_description/urdf/piro.xacro (robot description, xacro)
@@ -84,5 +84,5 @@
     </inertial>
   </link>
-  <!-- this joint binds the base_link with the claw central unit (represented by the link garra). It can rotate with the z axis fixed, it has an upper limit of 3,14 (180 degrees) and a lower limit of -3,14 (-180 degrees) -->
+  <!-- this joint binds the base_link with the claw central unit (represented by the link garra_ap). It can rotate with the z axis fixed, it has an upper limit of 3,14 (180 degrees) and a lower limit of -3,14 (-180 degrees) -->
   <joint name="joint_garra_ap" type="revolute">
     <parent link="base_link"/>
@@ -114,4 +114,5 @@
     </inertial>
   </link>
+  <!-- this joint binds the claw central unit (represented by the link garra_ap) with the central traction unit (represented by the link eixo_tracao_ap). It can move contunuously with the y axis fixed. It moves forward and backward -->
   <joint name="joint_eixo_tracao_ap" type="continuous">
     <parent link="garra_ap"/>
@@ -123,10 +124,10 @@
   <!-- this link involves the central traction unit -->
   <link name="eixo_tracao_ap">
-    <visual>
-      <geometry>
-        <mesh filename="package://mybot_description/meshes/shaft_simple.dae"/>
-      </geometry>
-    </visual>
-    <collision>
+    <visual name = 'central_traction'>
+      <geometry>
+        <mesh filename="package://mybot_description/meshes/shaft_simple.dae"/>
+      </geometry>
+    </visual>
+    <collision name = 'central_traction'>
       <geometry>
         <mesh filename="package://mybot_description/meshes/shaft_simple.dae"/>

Commit message: add commits of the link named link1_f

File: mybot_description/urdf/piro.xacro (robot description, xacro)
@@ -23,5 +23,5 @@
   <!-- Posicoes da base do sup_apoio para o centro do base link -->
   <!-- Parametros do base_link-->
-  <!-- This link involves the base_body, the central stem and the central's claw base -->
+  <!-- This link represents the base_body, the central stem and the central's claw base -->
   <link name="base_link">
     <!-- This visual represents the base body-->
@@ -70,5 +70,5 @@
         <box size="0.0367 0.0367 0.279"/>
       </geometry>
-      <origin rpy="0 0.0 0" xyz="0.0 0.03 0.25"/>
+      <origin rpy="0 0 0" xyz="0 0.0303 0.23365"/>
     </collision>
     <!-- This collision is for the central_claw_base -->
@@ -77,4 +77,5 @@
         <mesh filename="package://mybot_description/meshes/dxl_mx106.dae"/>
       </geometry>
+      <origin rpy="0 0 0" xyz="0.0 0.0722 0.3554"/>
     </collision>
     <inertial>
@@ -92,5 +93,5 @@
     <axis xyz="0 0 1"/>
   </joint>
-  <!-- this link involves the central claw unit -->
+  <!-- this link represents the central claw unit -->
   <link name="garra_ap">
     <!-- This visual represents the central claw unit -->
@@ -122,5 +123,5 @@
     <dynamics damping="0.7" friction="1.0" />
   </joint>
-  <!-- this link involves the central traction unit -->
+  <!-- this link represents the central traction unit -->
   <link name="eixo_tracao_ap">
     <!-- This visual represents the central traction unit -->
@@ -143,15 +144,7 @@
     </inertial>
   </link>
-  <!-- JUNTA 1 -->
-  <!-- Dimensoes do link1 collision -->
-  <!-- Dimensoes do link1  -->
-  <!-- Link1 collision offset-->
-  <!-- Posicao do link1 -->
-  <!-- Posicao da junta1 -->
-  <!-- Angulo da junta1 -->
-  <!-- Parametros do link1-->
-  <!-- Link F1 -->
+  <!-- This link represents the front arm unit  -->
   <link name="link1_f">
-    <visual>
+    <!-- <visual>
       <geometry>
         <box size="0.185 0.102 0.102"/>
@@ -159,15 +152,16 @@
       <material name="grey"/>
       <origin rpy="0 0 0" xyz="0.1985 0.0 0.0"/>
-    </visual>
-    <visual>
-      <geometry>
-        <box size="0.405 0.102 0.03"/>
+    </visual> -->
+    <!-- This visual represents the front arm unit -->
+    <visual name = 'front_arm'>
+      <geometry>
+        <box size="0.4199 0.05 0.100"/>
       </geometry>
       <material name="grey"/>
       <origin rpy="0 0 0" xyz="0.1885 0.0 0.0"/>
     </visual>
-    <collision>
-      <geometry>
-        <box size="0.185 0.102 0.102"/>
+    <collision name = 'front_arm'>
+      <geometry>
+        <box size="0.4199 0.05 0.100"/>
       </geometry>
       <origin rpy="0 0 0" xyz="0.1885 0.0 0.0"/>

Commit message: add some commits and started trying to position the piro in line in order to have the 5 shafts on line

File: mybot_description/urdf/piro.xacro (robot description, xacro)
@@ -85,5 +85,5 @@
     </inertial>
   </link>
-  <!-- this joint binds the base_link with the central claw unit (represented by the link garra_ap). It can rotate with the z axis fixed, it has an upper limit of 3,14 (180 degrees) and a lower limit of -3,14 (-180 degrees) -->
+  <!-- this joint binds the base body (represented by the link base_link) with the central claw unit (represented by the link garra_ap). It can rotate with the z axis fixed, it has an upper limit of 3,14 (180 degrees) and a lower limit of -3,14 (-180 degrees) -->
   <joint name="joint_garra_ap" type="revolute">
     <parent link="base_link"/>
@@ -144,4 +144,12 @@
     </inertial>
   </link>
+  <!-- This joint binds the base body (represented by the link base_link) and the front arm unit (represented by the link link1_f). it can rotate with the y axis fixed, it has an upper limit of 0.7 (40 degrees) and a lower limit of -1.74 (-100 degrees) -->
+  <joint name="joint1_f" type="revolute">
+    <parent link="base_link"/>
+    <child link="link1_f"/>
+    <origin rpy=" 0 -0.64 3.141592" xyz="-0.13 0.0 0.079"/>
+    <limit effort="1000.0" lower="-1.74" upper="0.7" velocity="0.5"/>
+    <axis xyz="0 1 0"/>
+  </joint>
   <!-- This link represents the front arm unit  -->
   <link name="link1_f">
@@ -161,4 +169,5 @@
       <origin rpy="0 0 0" xyz="0.1885 0.0 0.0"/>
     </visual>
+    <!-- this collision is for the front arm unit -->
     <collision name = 'front_arm'>
       <geometry>
@@ -173,14 +182,15 @@
     </inertial>
   </link>
-  <joint name="joint1_f" type="revolute">
+  <!-- This joint binds the base body (represented by the link base_link) and the back arm unit (represented by the link link1_t). it can rotate with the y axis fixed, it has an upper limit of 0.7 (40 degrees) and a lower limit of -1.74 (-100 degrees) -->
+  <joint name="joint1_t" type="revolute">
     <parent link="base_link"/>
-    <child link="link1_f"/>
-    <origin rpy=" 0 0 3.141592" xyz="-0.13 0.0 0.079"/>
+    <child link="link1_t"/>
+    <origin rpy="0 -0.64 0" xyz="0.13 0.0 0.079"/>
     <limit effort="1000.0" lower="-1.74" upper="0.7" velocity="0.5"/>
     <axis xyz="0 1 0"/>
   </joint>
-  <!-- Link T1 -->
+  <!-- This link represents the front arm unit  -->
   <link name="link1_t">
-    <visual>
+    <!-- <visual>
       <geometry>
         <box size="0.185 0.102 0.102"/>
@@ -188,8 +198,8 @@
       <material name="grey"/>
       <origin rpy="0 0 0" xyz="0.1985 0.0 0.0"/>
-    </visual>
-    <visual>
-      <geometry>
-        <box size="0.405 0.102 0.03"/>
+    </visual> -->
+    <visual>
+      <geometry>
+        <box size="0.4199 0.05 0.100"/>
       </geometry>
       <material name="grey"/>
@@ -198,5 +208,5 @@
     <collision>
       <geometry>
-        <box size="0.185 0.102 0.102"/>
+        <box size="0.4199 0.05 0.100"/>
       </geometry>
       <origin rpy="0 0 0" xyz="0.1885 0.0 0.0"/>
@@ -208,11 +218,4 @@
     </inertial>
   </link>
-  <joint name="joint1_t" type="revolute">
-    <parent link="base_link"/>
-    <child link="link1_t"/>
-    <origin rpy="0 0 0" xyz="0.13 0.0 0.079"/>
-    <limit effort="1000.0" lower="-1.74" upper="0.7" velocity="0.5"/>
-    <axis xyz="0 1 0"/>
-  </joint>
   <!-- TRACAO -->
   <!-- Dimensoes da tracao -->
@@ -267,5 +270,5 @@
     <parent link="link1_f"/>
     <child link="tracao_f"/>
-    <origin rpy="0 0 0" xyz="0.39 0.0 0.0"/>
+    <origin rpy="0 0.57 0" xyz="0.39 0.0 0.0"/>
     <limit effort="1000.0" lower="-1.0" upper="2.18" velocity="0.5"/>
     <axis xyz="0 1 0"/>
@@ -309,5 +312,5 @@
     <parent link="link1_t"/>
     <child link="tracao_t"/>
-    <origin rpy="0 0 0" xyz="0.39 0.0 0.0"/>
+    <origin rpy="0 0.57 0" xyz="0.39 0.0 0.0"/>
     <limit effort="1000.0" lower="-1.0" upper="2.18" velocity="0.5"/>
     <axis xyz="0 1 0"/>

Commit message: adjusted the piro3 arms and position to be in line with shafts in line as well

File: mybot_description/urdf/piro.xacro (robot description, xacro)
@@ -148,5 +148,5 @@
     <parent link="base_link"/>
     <child link="link1_f"/>
-    <origin rpy=" 0 -0.64 3.141592" xyz="-0.13 0.0 0.079"/>
+    <origin rpy=" 0 -0.60 3.141592" xyz="-0.13 0.0 0.079"/>
     <limit effort="1000.0" lower="-1.74" upper="0.7" velocity="0.5"/>
     <axis xyz="0 1 0"/>
@@ -186,9 +186,9 @@
     <parent link="base_link"/>
     <child link="link1_t"/>
-    <origin rpy="0 -0.64 0" xyz="0.13 0.0 0.079"/>
+    <origin rpy="0 -0.60 0" xyz="0.13 0.0 0.079"/>
     <limit effort="1000.0" lower="-1.74" upper="0.7" velocity="0.5"/>
     <axis xyz="0 1 0"/>
   </joint>
-  <!-- This link represents the front arm unit  -->
+  <!-- This link represents the back arm unit  -->
   <link name="link1_t">
     <!-- <visual>
@@ -199,5 +199,6 @@
       <origin rpy="0 0 0" xyz="0.1985 0.0 0.0"/>
     </visual> -->
-    <visual>
+    <!-- This visual represents the back arm unit -->
+    <visual name = 'back_arm'>
       <geometry>
         <box size="0.4199 0.05 0.100"/>
@@ -206,5 +207,6 @@
       <origin rpy="0 0 0" xyz="0.1885 0.0 0.0"/>
     </visual>
-    <collision>
+    <!-- this collision is for the back arm unit -->
+    <collision name = 'back_arm'>
       <geometry>
         <box size="0.4199 0.05 0.100"/>
