Commit message: commits and adjustment for joint joint2_t and link tracao_t

File: mybot_description/urdf/piro.xacro (robot description, xacro)
@@ -235,39 +235,5 @@
   <!-- Parametros da tracao-->
   <!-- TRACAO F -->
-  <!-- This link represents the front traction body unit -->
-  <link name="tracao_f">
-    <visual>
-      <geometry>
-        <box size="0.233 0.102 0.102"/>
-      </geometry>
-      <material name="grey"/>
-      <origin rpy="0 0 0" xyz="0.0885 0.0 0.0201"/>
-    </visual>
-    <visual>
-      <geometry>
-        <mesh filename="package://mybot_description/meshes/dxl_mx106.dae"/>
-      </geometry>
-      <material name="grey"/>
-      <origin rpy="0 0 0" xyz="0.0005 0.075 0.0521"/>
-    </visual>
-    <visual>
-      <geometry>
-        <mesh filename="package://mybot_description/meshes/dxl_mx106.dae"/>
-      </geometry>
-      <material name="grey"/>
-      <origin rpy="0 0 3.141592" xyz="0.1765 -0.075 0.0521"/>
-    </visual>
-    <collision>
-      <geometry>
-        <box size="0.233 0.198 0.102"/>
-      </geometry>
-      <origin rpy="0 0 0" xyz="0.0885 0.0 0.0201"/>
-    </collision>
-    <inertial>
-      <origin rpy="0 0 0" xyz="0.03499 0.0 0.0"/>
-      <mass value="0.792"/>
-      <inertia ixx="0.5622" ixy="0.161" ixz="0.0008" iyy="1.0746" iyz="0.0" izz="1.2126"/>
-    </inertial>
-  </link>
+  <!-- This joint binds the front arm unit (represented by the link link1_f) and the front traction body unit (represented by the link tracao_f). It can rotate with the y axis fixed, it has an upper limit of 2.18 (125 degrees) and a lower limit of -1.0 (-57 degrees) -->
   <joint name="joint2_f" type="revolute">
     <parent link="link1_f"/>
@@ -277,32 +243,52 @@
     <axis xyz="0 1 0"/>
   </joint>
-  <!-- TRACAO T -->
-  <link name="tracao_t">
-    <visual>
-      <geometry>
-        <box size="0.233 0.102 0.102"/>
+  <!-- This link represents the front traction body unit that contains front traction body, claw f1 support and claw f2 support -->
+  <link name="tracao_f">
+    <!-- This visual represents the front traction body -->
+    <visual name = 'front_traction_body'>
+      <geometry>
+        <box size="0.233 0.100 0.100"/>
       </geometry>
       <material name="grey"/>
       <origin rpy="0 0 0" xyz="0.0885 0.0 0.0201"/>
     </visual>
-    <visual>
-      <geometry>
-        <mesh filename="package://mybot_description/meshes/dxl_mx106.dae"/>
-      </geometry>
-      <material name="grey"/>
-      <origin rpy="0 0 0" xyz="0.0005 -0.075 0.0521"/>
-    </visual>
-    <visual>
-      <geometry>
-        <mesh filename="package://mybot_description/meshes/dxl_mx106.dae"/>
-      </geometry>
-      <material name="grey"/>
-      <origin rpy="0 0 3.141592" xyz="0.1765 0.075 0.0521"/>
-    </visual>
-    <collision>
-      <geometry>
-        <box size="0.233 0.198 0.102"/>
+    <!-- This visual represents the front traction claw f2 support -->
+    <!-- Need to check mesh design to see if dimensions is the same as the actual dimensions of piro3 -->
+    <visual name = 'front_traction_claw_f2_support'>
+      <geometry>
+        <mesh filename="package://mybot_description/meshes/dxl_mx106.dae"/>
+      </geometry>
+      <material name="grey"/>
+      <origin rpy="0 0 0" xyz="0.0005 0.075 0.0521"/>
+    </visual>
+    <!-- This visual represents the front traction claw f1 support -->
+    <!-- Need to check mesh design to see if dimensions is the same as the actual dimensions of piro3 -->
+    <visual name = 'front_traction_claw_f1_support'>
+      <geometry>
+        <mesh filename="package://mybot_description/meshes/dxl_mx106.dae"/>
+      </geometry>
+      <material name="grey"/>
+      <origin rpy="0 0 3.141592" xyz="0.1765 -0.075 0.0521"/>
+    </visual>
+    <!-- this collision is for the front traction body -->
+    <collision name = 'front_traction_body'>
+      <geometry>
+        <box size="0.233 0.100 0.100"/>
       </geometry>
       <origin rpy="0 0 0" xyz="0.0885 0.0 0.0201"/>
+    </collision>
+    <!-- this collision is for the front traction claw f2 support -->
+    <collision name = 'front_traction_claw_f2_support'>
+      <geometry>
+        <mesh filename="package://mybot_description/meshes/dxl_mx106.dae"/>
+      </geometry>
+      <origin rpy="0 0 0" xyz="0.0005 0.075 0.0521"/>
+    </collision>
+    <!-- this collision is for the front traction claw f1 support -->
+    <collision name = 'front_traction_claw_f1_support'>
+      <geometry>
+        <mesh filename="package://mybot_description/meshes/dxl_mx106.dae"/>
+      </geometry>
+      <origin rpy="0 0 3.141592" xyz="0.1765 -0.075 0.0521"/>
     </collision>
     <inertial>
@@ -312,4 +298,6 @@
     </inertial>
   </link>
+  <!-- TRACAO T -->
+  <!-- This joint binds the back arm unit (represented by the link link1_t) and the back traction body unit (represented by the link tracao_t). It can rotate with the y axis fixed, it has an upper limit of 2.18 (125 degrees) and a lower limit of -1.0 (-57 degrees) -->
   <joint name="joint2_t" type="revolute">
     <parent link="link1_t"/>
@@ -319,4 +307,57 @@
     <axis xyz="0 1 0"/>
   </joint>
+  <!-- This link represents the back traction body unit that contains back traction body, claw f1 support and claw f2 support -->
+  <link name="tracao_t">
+    <!-- This visual represents the  back traction body -->
+    <visual name = 'back_traction_body'>
+      <geometry>
+        <box size="0.233 0.100 0.100"/>
+      </geometry>
+      <material name="grey"/>
+      <origin rpy="0 0 0" xyz="0.0885 0.0 0.0201"/>
+    </visual>
+    <!-- This visual represents the  back traction claw f1 support -->
+    <visual name = 'back_traction_claw_f1_support'>
+      <geometry>
+        <mesh filename="package://mybot_description/meshes/dxl_mx106.dae"/>
+      </geometry>
+      <material name="grey"/>
+      <origin rpy="0 0 0" xyz="0.0005 -0.075 0.0521"/>
+    </visual>
+    <!-- This visual represents the  back traction claw f2 support -->
+    <visual name = 'back_traction_claw_f2_support'>
+      <geometry>
+        <mesh filename="package://mybot_description/meshes/dxl_mx106.dae"/>
+      </geometry>
+      <material name="grey"/>
+      <origin rpy="0 0 3.141592" xyz="0.1765 0.075 0.0521"/>
+    </visual>
+    <!-- this collision is for the back traction body -->
+    <collision name = 'back_traction_body'>
+      <geometry>
+        <box size="0.233 0.100 0.100"/>
+      </geometry>
+      <origin rpy="0 0 0" xyz="0.0885 0.0 0.0201"/>
+    </collision>
+    <!-- this collision is for the back traction claw f1 support -->
+    <collision name = 'back_traction_claw_f1_support'>
+      <geometry>
+        <mesh filename="package://mybot_description/meshes/dxl_mx106.dae"/>
+      </geometry>
+      <origin rpy="0 0 0" xyz="0.0005 -0.075 0.0521"/>
+    </collision>
+    <!-- this collision is for the back traction claw f2 support -->
+    <collision name = 'back_traction_claw_f2_support'>
+      <geometry>
+        <mesh filename="package://mybot_description/meshes/dxl_mx106.dae"/>
+      </geometry>
+      <origin rpy="0 0 3.141592" xyz="0.1765 0.075 0.0521"/>
+    </collision>
+    <inertial>
+      <origin rpy="0 0 0" xyz="0.03499 0.0 0.0"/>
+      <mass value="0.792"/>
+      <inertia ixx="0.5622" ixy="0.161" ixz="0.0008" iyy="1.0746" iyz="0.0" izz="1.2126"/>
+    </inertial>
+  </link>
   <!-- GARRAS DE TRACAO -->
   <!-- Posicoes das garras de tracao-->

Commit message: Change some collisions and added some commits

File: mybot_description/urdf/piro.xacro (robot description, xacro)
@@ -220,19 +220,4 @@
     </inertial>
   </link>
-  <!-- TRACAO -->
-  <!-- Dimensoes da tracao -->
-  <!-- Posicao da tracao em relacao a junta1-->
-  <!-- Dimensao dos servos -->
-  <!-- Posicao dos servos das garras em relacao ao centro da tracao-->
-  <!--
-	<xacro:property name="x_servo_garra_1" value="-0.007" />
-	<xacro:property name="y_servo_garra_1" value="0.0750" />
-	<xacro:property name="z_servo_garra_1" value="0.0521" />
--->
-  <!-- Posicao dos servos das garras em relacao ao centro da tracao-->
-  <!-- Posicao da junta2 -->
-  <!-- Angulo da junta2 -->
-  <!-- Parametros da tracao-->
-  <!-- TRACAO F -->
   <!-- This joint binds the front arm unit (represented by the link link1_f) and the front traction body unit (represented by the link tracao_f). It can rotate with the y axis fixed, it has an upper limit of 2.18 (125 degrees) and a lower limit of -1.0 (-57 degrees) -->
   <joint name="joint2_f" type="revolute">
@@ -360,29 +345,5 @@
     </inertial>
   </link>
-  <!-- GARRAS DE TRACAO -->
-  <!-- Posicoes das garras de tracao-->
-  <!-- Angulos da garra de tracao -->
-  <!-- GARRAS TRACAO DIANTEIRA -->
-  <!-- F1 -->
-  <link name="garra_tracao_f1">
-    <visual>
-      <geometry>
-        <mesh filename="package://mybot_description/meshes/claw.dae"/>
-      </geometry>
-      <material name="grey"/>
-      <origin rpy="0 0 0" xyz="0.0 0.012 0.0"/>
-    </visual>
-    <collision>
-      <geometry>
-        <box size="0.048 0.064 0.1851"/>
-      </geometry>
-      <origin rpy="0 0 0" xyz="0.0 0.017 0.09255"/>
-    </collision>
-    <inertial>
-      <origin rpy="0 0 0" xyz="0.0 0.015953 0.116844"/>
-      <mass value="0.22"/>
-      <inertia ixx="0.000598" ixy="0.0" ixz="0.0" iyy="0.000866" iyz="0.000169" izz="0.000866"/>
-    </inertial>
-  </link>
+  <!-- This joint binds the front traction body unit (represented by the link tracao_f) and the front f1 claw unit (represented by the link garra_tracao_f1). It can rotate with the z axis fixed, it has an upper limit of 3.14 (360 degrees) and lower limit of -3.14 (-360 degrees) -->
   <joint name="joint_garra_tracao_f1" type="revolute">
     <parent link="tracao_f"/>
@@ -392,24 +353,29 @@
     <axis xyz="0 0 1"/>
   </joint>
-  <!-- Eixo F1 -->
-  <link name="eixo_tracao_f1">
-    <visual>
-      <geometry>
-        <mesh filename="package://mybot_description/meshes/shaft_simple.dae"/>
-      </geometry>
-      <material name="grey"/>
-      <!-- <origin rpy="0 0 0" xyz="0.0 0.012 0.025"/> -->
-    </visual>
+  <!-- this link represents the front f1 claw unit -->
+  <link name="garra_tracao_f1">
+    <!-- Need to check mesh design to see if dimensions is the same as the actual dimensions of piro3 -->
+    <!-- This visual represents the front f1 claw unit -->
+    <visual>
+      <geometry>
+        <mesh filename="package://mybot_description/meshes/claw.dae"/>
+      </geometry>
+      <material name="grey"/>
+      <origin rpy="0 0 0" xyz="0.0 0.012 0.0"/>
+    </visual>
+    <!-- this collision is for the front f1 claw unit -->
     <collision>
       <geometry>
-        <mesh filename="package://mybot_description/meshes/shaft_simple.dae"/>
-      </geometry>
-    </collision>
-    <inertial>
-      <origin rpy="0 0 0" xyz="0.0 0.026065 0.0"/>
-      <mass value="0.1"/>
-      <inertia ixx="4.94e-05" ixy="0.0" ixz="0.0" iyy="6.11e-05" iyz="0.0" izz="4.94e-05"/>
-    </inertial>
-  </link>
+        <mesh filename="package://mybot_description/meshes/claw.dae"/>
+      </geometry>
+      <origin rpy="0 0 0" xyz="0.0 0.012 0.0"/>
+    </collision>
+    <inertial>
+      <origin rpy="0 0 0" xyz="0.0 0.015953 0.116844"/>
+      <mass value="0.22"/>
+      <inertia ixx="0.000598" ixy="0.0" ixz="0.0" iyy="0.000866" iyz="0.000169" izz="0.000866"/>
+    </inertial>
+  </link>
+  <!-- this joint binds the front f1 claw unit (represented by the link garra_tracao_f1) with the front f1 traction unit (represented by the link eixo_tracao_f1). It can move contunuously with the y axis fixed. It moves forward and backward -->
   <joint name="joint_eixo_tracao_f1" type="continuous">
     <parent link="garra_tracao_f1"/>
@@ -419,6 +385,31 @@
     <dynamics damping="0.7" friction="1.0" />
   </joint>
-  <!-- F2 -->
+  <!-- this link represents the front f1 traction unit -->
+  <link name="eixo_tracao_f1">
+    <!-- This visual represents the front f1 traction unit -->
+    <!-- Need to check mesh design to see if dimensions is the same as the actual dimensions of piro3 -->
+    <visual>
+      <geometry>
+        <mesh filename="package://mybot_description/meshes/shaft_simple.dae"/>
+      </geometry>
+      <material name="grey"/>
+      <!-- <origin rpy="0 0 0" xyz="0.0 0.012 0.025"/> -->
+    </visual>
+    <!-- This collision is for the central traction unit -->
+    <collision>
+      <geometry>
+        <mesh filename="package://mybot_description/meshes/shaft_simple.dae"/>
+      </geometry>
+    </collision>
+    <inertial>
+      <origin rpy="0 0 0" xyz="0.0 0.026065 0.0"/>
+      <mass value="0.1"/>
+      <inertia ixx="4.94e-05" ixy="0.0" ixz="0.0" iyy="6.11e-05" iyz="0.0" izz="4.94e-05"/>
+    </inertial>
+  </link>
+  <!-- this link represents the front f2 claw unit -->
   <link name="garra_tracao_f2">
+    <!-- Need to check mesh design to see if dimensions is the same as the actual dimensions of piro3 -->
+    <!-- This visual represents the front f2 claw unit -->
     <visual>
       <geometry>
@@ -428,9 +419,10 @@
       <origin rpy="0 0 0" xyz="0.0 0.012 0.0"/>
     </visual>
+    <!-- this collision is for the front f2 claw unit -->
     <collision>
       <geometry>
-        <box size="0.048 0.064 0.1851"/>
-      </geometry>
-      <origin rpy="0 0 0" xyz="0.0 0.017 0.09255"/>
+        <mesh filename="package://mybot_description/meshes/claw.dae"/>
+      </geometry>
+      <origin rpy="0 0 0" xyz="0.0 0.012 0.0"/>
     </collision>
     <inertial>
