Commit message: add more commits and fixed the last collisions that had problems

File: mybot_description/urdf/piro.xacro (robot description, xacro)
@@ -396,5 +396,5 @@
       <!-- <origin rpy="0 0 0" xyz="0.0 0.012 0.025"/> -->
     </visual>
-    <!-- This collision is for the central traction unit -->
+    <!-- This collision is for the front f1 traction unit -->
     <collision>
       <geometry>
@@ -408,28 +408,5 @@
     </inertial>
   </link>
-  <!-- this link represents the front f2 claw unit -->
-  <link name="garra_tracao_f2">
-    <!-- Need to check mesh design to see if dimensions is the same as the actual dimensions of piro3 -->
-    <!-- This visual represents the front f2 claw unit -->
-    <visual>
-      <geometry>
-        <mesh filename="package://mybot_description/meshes/claw.dae"/>
-      </geometry>
-      <material name="grey"/>
-      <origin rpy="0 0 0" xyz="0.0 0.012 0.0"/>
-    </visual>
-    <!-- this collision is for the front f2 claw unit -->
-    <collision>
-      <geometry>
-        <mesh filename="package://mybot_description/meshes/claw.dae"/>
-      </geometry>
-      <origin rpy="0 0 0" xyz="0.0 0.012 0.0"/>
-    </collision>
-    <inertial>
-      <origin rpy="0 0 0" xyz="0.0 0.015953 0.116844"/>
-      <mass value="0.22"/>
-      <inertia ixx="0.000598" ixy="0.0" ixz="0.0" iyy="0.000866" iyz="0.000169" izz="0.000866"/>
-    </inertial>
-  </link>
+  <!-- This joint binds the front traction body unit (represented by the link tracao_f) and the front f2 claw unit (represented by the link garra_tracao_f2). It can rotate with the z axis fixed, it has an upper limit of 3.14 (360 degrees) and lower limit of -3.14 (-360 degrees) -->
   <joint name="joint_garra_tracao_f2" type="revolute">
     <parent link="tracao_f"/>
@@ -439,25 +416,29 @@
     <axis xyz="0 0 1"/>
   </joint>
-   --&gt;
-  <!-- Eixo F2 -->
-  <link name="eixo_tracao_f2">
-    <visual>
-      <geometry>
-        <mesh filename="package://mybot_description/meshes/shaft_simple.dae"/>
-      </geometry>
-      <material name="grey"/>
-      <!-- <origin rpy="0 0 0" xyz="0.0 0.012 0.025"/> -->
-    </visual>
+  <!-- this link represents the front f2 claw unit -->
+  <link name="garra_tracao_f2">
+    <!-- Need to check mesh design to see if dimensions is the same as the actual dimensions of piro3 -->
+    <!-- This visual represents the front f2 claw unit -->
+    <visual>
+      <geometry>
+        <mesh filename="package://mybot_description/meshes/claw.dae"/>
+      </geometry>
+      <material name="grey"/>
+      <origin rpy="0 0 0" xyz="0.0 0.012 0.0"/>
+    </visual>
+    <!-- this collision is for the front f2 claw unit -->
     <collision>
       <geometry>
-        <mesh filename="package://mybot_description/meshes/shaft_simple.dae"/>
-      </geometry>
-    </collision>
-    <inertial>
-      <origin rpy="0 0 0" xyz="0.0 0.026065 0.0"/>
-      <mass value="0.1"/>
-      <inertia ixx="4.94e-05" ixy="0.0" ixz="0.0" iyy="6.11e-05" iyz="0.0" izz="4.94e-05"/>
-    </inertial>
-  </link>
+        <mesh filename="package://mybot_description/meshes/claw.dae"/>
+      </geometry>
+      <origin rpy="0 0 0" xyz="0.0 0.012 0.0"/>
+    </collision>
+    <inertial>
+      <origin rpy="0 0 0" xyz="0.0 0.015953 0.116844"/>
+      <mass value="0.22"/>
+      <inertia ixx="0.000598" ixy="0.0" ixz="0.0" iyy="0.000866" iyz="0.000169" izz="0.000866"/>
+    </inertial>
+  </link>
+  <!-- this joint binds the front f2 claw unit (represented by the link garra_tracao_f2) with the front f2 traction unit (represented by the link eixo_tracao_f2). It can move contunuously with the y axis fixed. It moves forward and backward -->
   <joint name="joint_eixo_tracao_f2" type="continuous">
     <parent link="garra_tracao_f2"/>
@@ -467,26 +448,30 @@
     <dynamics damping="0.7" friction="1.0" />
   </joint>
+  <!-- this link represents the front f2 traction unit -->
+  <link name="eixo_tracao_f2">
+    <!-- This visual represents the front f2 traction unit -->
+    <!-- Need to check mesh design to see if dimensions is the same as the actual dimensions of piro3 -->
+    <visual>
+      <geometry>
+        <mesh filename="package://mybot_description/meshes/shaft_simple.dae"/>
+      </geometry>
+      <material name="grey"/>
+      <!-- <origin rpy="0 0 0" xyz="0.0 0.012 0.025"/> -->
+    </visual>
+    <!-- This collision is for the front f2 traction unit -->
+    <collision>
+      <geometry>
+        <mesh filename="package://mybot_description/meshes/shaft_simple.dae"/>
+      </geometry>
+    </collision>
+    <inertial>
+      <origin rpy="0 0 0" xyz="0.0 0.026065 0.0"/>
+      <mass value="0.1"/>
+      <inertia ixx="4.94e-05" ixy="0.0" ixz="0.0" iyy="6.11e-05" iyz="0.0" izz="4.94e-05"/>
+    </inertial>
+  </link>
   <!-- GARRAS TRACAO TRASEIRA -->
   <!-- T1 -->
-  <link name="garra_tracao_t1">
-    <visual>
-      <geometry>
-        <mesh filename="package://mybot_description/meshes/claw.dae"/>
-      </geometry>
-      <material name="grey"/>
-      <origin rpy="0 0 0" xyz="0.0 0.012 0.0"/>
-    </visual>
-    <collision>
-      <geometry>
-        <box size="0.048 0.064 0.1851"/>
-      </geometry>
-      <origin rpy="0 0 0" xyz="0.0 0.017 0.09255"/>
-    </collision>
-    <inertial>
-      <origin rpy="0 0 0" xyz="0.0 0.015953 0.116844"/>
-      <mass value="0.22"/>
-      <inertia ixx="0.000598" ixy="0.0" ixz="0.0" iyy="0.000866" iyz="0.000169" izz="0.000866"/>
-    </inertial>
-  </link>
+  <!-- This joint binds the front traction body unit (represented by the link tracao_f) and the back t1 claw unit (represented by the link garra_tracao_t1). It can rotate with the z axis fixed, it has an upper limit of 3.14 (360 degrees) and lower limit of -3.14 (-360 degrees) -->
   <joint name="joint_garra_tracao_t1" type="revolute">
     <parent link="tracao_t"/>
@@ -496,25 +481,30 @@
     <axis xyz="0 0 1"/>
   </joint>
-   --&gt;
+  <!-- this link represents the back t1 claw unit -->
+  <link name="garra_tracao_t1">
+    <!-- Need to check mesh design to see if dimensions is the same as the actual dimensions of piro3 -->
+    <!-- This visual represents the back t1 claw unit -->
+    <visual>
+      <geometry>
+        <mesh filename="package://mybot_description/meshes/claw.dae"/>
+      </geometry>
+      <material name="grey"/>
+      <origin rpy="0 0 0" xyz="0.0 0.012 0.0"/>
+    </visual>
+    <!-- this collision is for the back t1 claw unit -->
+    <collision>
+      <geometry>
+        <mesh filename="package://mybot_description/meshes/claw.dae"/>
+      </geometry>
+      <origin rpy="0 0 0" xyz="0.0 0.012 0.0"/>
+    </collision>
+    <inertial>
+      <origin rpy="0 0 0" xyz="0.0 0.015953 0.116844"/>
+      <mass value="0.22"/>
+      <inertia ixx="0.000598" ixy="0.0" ixz="0.0" iyy="0.000866" iyz="0.000169" izz="0.000866"/>
+    </inertial>
+  </link>
   <!-- Eixo T1 -->
-  <link name="eixo_tracao_t1">
-    <visual>
-      <geometry>
-        <mesh filename="package://mybot_description/meshes/shaft_simple.dae"/>
-      </geometry>
-      <material name="grey"/>
-      <!-- <origin rpy="0 0 0" xyz="0.0 0.012 0.025"/> -->
-    </visual>
-    <collision>
-      <geometry>
-        <mesh filename="package://mybot_description/meshes/shaft_simple.dae"/>
-      </geometry>
-    </collision>
-    <inertial>
-      <origin rpy="0 0 0" xyz="0.0 0.026065 0.0"/>
-      <mass value="0.1"/>
-      <inertia ixx="4.94e-05" ixy="0.0" ixz="0.0" iyy="6.11e-05" iyz="0.0" izz="4.94e-05"/>
-    </inertial>
-  </link>
+  <!-- this joint binds the back t1 claw unit (represented by the link garra_tracao_t1) with the back t1 traction unit (represented by the link eixo_tracao_t1). It can move contunuously with the y axis fixed. It moves forward and backward -->
   <joint name="joint_eixo_tracao_t1" type="continuous">
     <parent link="garra_tracao_t1"/>
@@ -524,25 +514,29 @@
     <dynamics damping="0.7" friction="1.0" />
   </joint>
+  <!-- this link represents the back t1 traction unit -->
+  <link name="eixo_tracao_t1">
+    <!-- This visual represents the back t1 traction unit -->
+    <!-- Need to check mesh design to see if dimensions is the same as the actual dimensions of piro3 -->
+    <visual>
+      <geometry>
+        <mesh filename="package://mybot_description/meshes/shaft_simple.dae"/>
+      </geometry>
+      <material name="grey"/>
+      <!-- <origin rpy="0 0 0" xyz="0.0 0.012 0.025"/> -->
+    </visual>
+    <!-- This collision is for the back t1 traction unit -->
+    <collision>
+      <geometry>
+        <mesh filename="package://mybot_description/meshes/shaft_simple.dae"/>
+      </geometry>
+    </collision>
+    <inertial>
+      <origin rpy="0 0 0" xyz="0.0 0.026065 0.0"/>
+      <mass value="0.1"/>
+      <inertia ixx="4.94e-05" ixy="0.0" ixz="0.0" iyy="6.11e-05" iyz="0.0" izz="4.94e-05"/>
+    </inertial>
+  </link>
   <!-- T2 -->
-  <link name="garra_tracao_t2">
-    <visual>
-      <geometry>
-        <mesh filename="package://mybot_description/meshes/claw.dae"/>
-      </geometry>
-      <material name="grey"/>
-      <origin rpy="0 0 0" xyz="0.0 0.012 0.0"/>
-    </visual>
-    <collision>
-      <geometry>
-        <box size="0.048 0.064 0.1851"/>
-      </geometry>
-      <origin rpy="0 0 0" xyz="0.0 0.017 0.09255"/>
-    </collision>
-    <inertial>
-      <origin rpy="0 0 0" xyz="0.0 0.015953 0.116844"/>
-      <mass value="0.22"/>
-      <inertia ixx="0.000598" ixy="0.0" ixz="0.0" iyy="0.000866" iyz="0.000169" izz="0.000866"/>
-    </inertial>
-  </link>
+  <!-- This joint binds the front traction body unit (represented by the link tracao_f) and the back t2 claw unit (represented by the link garra_tracao_t2). It can rotate with the z axis fixed, it has an upper limit of 3.14 (360 degrees) and lower limit of -3.14 (-360 degrees) -->
   <joint name="joint_garra_tracao_t2" type="revolute">
     <parent link="tracao_t"/>
@@ -552,24 +546,30 @@
     <axis xyz="0 0 1"/>
   </joint>
+  <!-- this link represents the back t2 claw unit -->
+  <link name="garra_tracao_t2">
+    <!-- Need to check mesh design to see if dimensions is the same as the actual dimensions of piro3 -->
+    <!-- This visual represents the back t2 claw unit -->
+    <visual>
+      <geometry>
+        <mesh filename="package://mybot_description/meshes/claw.dae"/>
+      </geometry>
+      <material name="grey"/>
+      <origin rpy="0 0 0" xyz="0.0 0.012 0.0"/>
+    </visual>
+    <!-- this collision is for the back t2 claw unit -->
+    <collision>
+      <geometry>
+        <mesh filename="package://mybot_description/meshes/claw.dae"/>
+      </geometry>
+      <origin rpy="0 0 0" xyz="0.0 0.012 0.0"/>
+    </collision>
+    <inertial>
+      <origin rpy="0 0 0" xyz="0.0 0.015953 0.116844"/>
+      <mass value="0.22"/>
+      <inertia ixx="0.000598" ixy="0.0" ixz="0.0" iyy="0.000866" iyz="0.000169" izz="0.000866"/>
+    </inertial>
+  </link>
   <!-- Eixo F2 -->
-  <link name="eixo_tracao_t2">
-    <visual>
-      <geometry>
-        <mesh filename="package://mybot_description/meshes/shaft_simple.dae"/>
-      </geometry>
-      <material name="grey"/>
-      <!-- <origin rpy="0 0 0" xyz="0.0 0.012 0.025"/> -->
-    </visual>
-    <collision>
-      <geometry>
-        <mesh filename="package://mybot_description/meshes/shaft_simple.dae"/>
-      </geometry>
-    </collision>
-    <inertial>
-      <origin rpy="0 0 0" xyz="0.0 0.026065 0.0"/>
-      <mass value="0.1"/>
-      <inertia ixx="4.94e-05" ixy="0.0" ixz="0.0" iyy="6.11e-05" iyz="0.0" izz="4.94e-05"/>
-    </inertial>
-  </link>
+  <!-- this joint binds the back t2 claw unit (represented by the link garra_tracao_t2) with the back t2 traction unit (represented by the link eixo_tracao_t2). It can move contunuously with the y axis fixed. It moves forward and backward -->
   <joint name="joint_eixo_tracao_t2" type="continuous">
     <parent link="garra_tracao_t2"/>
@@ -579,4 +579,27 @@
     <dynamics damping="0.7" friction="1.0" />
   </joint>
+  <!-- this link represents the back t2 traction unit -->
+  <link name="eixo_tracao_t2">
+    <!-- This visual represents the back t2 traction unit -->
+    <!-- Need to check mesh design to see if dimensions is the same as the actual dimensions of piro3 -->
+    <visual>
+      <geometry>
+        <mesh filename="package://mybot_description/meshes/shaft_simple.dae"/>
+      </geometry>
+      <material name="grey"/>
+      <!-- <origin rpy="0 0 0" xyz="0.0 0.012 0.025"/> -->
+    </visual>
+    <!-- This collision is for the back t2 traction unit -->
+    <collision>
+      <geometry>
+        <mesh filename="package://mybot_description/meshes/shaft_simple.dae"/>
+      </geometry>
+    </collision>
+    <inertial>
+      <origin rpy="0 0 0" xyz="0.0 0.026065 0.0"/>
+      <mass value="0.1"/>
+      <inertia ixx="4.94e-05" ixy="0.0" ixz="0.0" iyy="6.11e-05" iyz="0.0" izz="4.94e-05"/>
+    </inertial>
+  </link>
   <!-- SENSORES -->
   <!-- Hokuyo -->

Commit message: Added new shaft model, still in test phase

File: mybot_description/urdf/piro.xacro (robot description, xacro)
@@ -18,5 +18,5 @@
 	<xacro:property name="h_eletr_ap" value="0.120" />
 	<xacro:property name="w_eletr_ap" value="0.120" />
--->
+  -->
   <!-- Suporte da garra da unidade de apoio -->
   <!-- Dimensoes do sup_apoio -->
@@ -40,13 +40,4 @@
       <origin rpy="0 0 0" xyz="0 0.0303 0.23365"/>
     </visual>
-    <!--
-		<visual>
-			<geometry>
-				<box size="${l_eletr_ap} ${w_eletr_ap} ${h_eletr_ap}"/>
-			</geometry>
-			<xacro:cor />
-			<origin xyz="0 0 ${-h_ap/2 + -h_eletr_ap/2}" rpy="0 0 0" />
-		</visual>
-    -->
     <!-- This visual represents the claw's base in the central stem -->
     <!-- Need to check mesh design to see if dimensions is the same as the actual dimensions of piro3 -->
@@ -129,12 +120,14 @@
     <visual name = 'central_traction'>
       <geometry>
-        <mesh filename="package://mybot_description/meshes/shaft_simple.dae"/>
-      </geometry>
+        <mesh filename="package://mybot_description/meshes/Shaft_piro3.dae"/>
+      </geometry>
+      <origin rpy="1.57 0 0" xyz="0.01 0.045 0.042"/>
     </visual>
     <!-- This collision is for the central traction unit -->
     <collision name = 'central_traction'>
       <geometry>
-        <mesh filename="package://mybot_description/meshes/shaft_simple.dae"/>
-      </geometry>
+        <mesh filename="package://mybot_description/meshes/Shaft_piro3.dae"/>
+      </geometry>
+      <origin rpy="1.57 0 0" xyz="0.01 0.045 0.042"/>
     </collision>
     <inertial>
@@ -283,5 +276,4 @@
     </inertial>
   </link>
-  <!-- TRACAO T -->
   <!-- This joint binds the back arm unit (represented by the link link1_t) and the back traction body unit (represented by the link tracao_t). It can rotate with the y axis fixed, it has an upper limit of 2.18 (125 degrees) and a lower limit of -1.0 (-57 degrees) -->
   <joint name="joint2_t" type="revolute">
@@ -391,7 +383,8 @@
     <visual>
       <geometry>
-        <mesh filename="package://mybot_description/meshes/shaft_simple.dae"/>
-      </geometry>
-      <material name="grey"/>
+        <mesh filename="package://mybot_description/meshes/Shaft_piro3.dae"/>
+      </geometry>
+      <material name="grey"/>
+      <origin rpy="1.57 0 0" xyz="0.01 0.045 0.042"/>
       <!-- <origin rpy="0 0 0" xyz="0.0 0.012 0.025"/> -->
     </visual>
@@ -399,6 +392,7 @@
     <collision>
       <geometry>
-        <mesh filename="package://mybot_description/meshes/shaft_simple.dae"/>
-      </geometry>
+        <mesh filename="package://mybot_description/meshes/Shaft_piro3.dae"/>
+      </geometry>
+      <origin rpy="1.57 0 0" xyz="0.01 0.045 0.042"/>
     </collision>
     <inertial>
@@ -454,6 +448,7 @@
     <visual>
       <geometry>
-        <mesh filename="package://mybot_description/meshes/shaft_simple.dae"/>
-      </geometry>
+        <mesh filename="package://mybot_description/meshes/Shaft_piro3.dae"/>
+      </geometry>
+      <origin rpy="1.57 0 0" xyz="0.01 0.045 0.042"/>
       <material name="grey"/>
       <!-- <origin rpy="0 0 0" xyz="0.0 0.012 0.025"/> -->
@@ -462,6 +457,7 @@
     <collision>
       <geometry>
-        <mesh filename="package://mybot_description/meshes/shaft_simple.dae"/>
-      </geometry>
+        <mesh filename="package://mybot_description/meshes/Shaft_piro3.dae"/>
+      </geometry>
+      <origin rpy="1.57 0 0" xyz="0.01 0.045 0.042"/>
     </collision>
     <inertial>
@@ -520,6 +516,7 @@
     <visual>
       <geometry>
-        <mesh filename="package://mybot_description/meshes/shaft_simple.dae"/>
-      </geometry>
+        <mesh filename="package://mybot_description/meshes/Shaft_piro3.dae"/>
+      </geometry>
+      <origin rpy="1.57 0 0" xyz="0.01 0.045 0.042"/>
       <material name="grey"/>
       <!-- <origin rpy="0 0 0" xyz="0.0 0.012 0.025"/> -->
@@ -528,6 +525,7 @@
     <collision>
       <geometry>
-        <mesh filename="package://mybot_description/meshes/shaft_simple.dae"/>
-      </geometry>
+        <mesh filename="package://mybot_description/meshes/Shaft_piro3.dae"/>
+      </geometry>
+      <origin rpy="1.57 0 0" xyz="0.01 0.045 0.042"/>
     </collision>
     <inertial>
@@ -585,6 +583,7 @@
     <visual>
       <geometry>
-        <mesh filename="package://mybot_description/meshes/shaft_simple.dae"/>
-      </geometry>
+        <mesh filename="package://mybot_description/meshes/Shaft_piro3.dae"/>
+      </geometry>
+      <origin rpy="1.57 0 0" xyz="0.01 0.045 0.042"/>
       <material name="grey"/>
       <!-- <origin rpy="0 0 0" xyz="0.0 0.012 0.025"/> -->
@@ -593,6 +592,7 @@
     <collision>
       <geometry>
-        <mesh filename="package://mybot_description/meshes/shaft_simple.dae"/>
-      </geometry>
+        <mesh filename="package://mybot_description/meshes/Shaft_piro3.dae"/>
+      </geometry>
+      <origin rpy="1.57 0 0" xyz="0.01 0.045 0.042"/>
     </collision>
     <inertial>
@@ -612,19 +612,27 @@
   <!-- Posicoes dos frames virtuais -->
   <!-- Apoio -->
-  <!--<link name="laser" >
-		<visual>
-			<geometry>
-				<mesh filename="package://mybot_description/meshes/hokuyo.dae"/>
-			</geometry>
-			<xacro:cor />
-		</visual>
-	</link>
-	<joint name="hokuyo_base" type="fixed">
-		<parent link="tracao_f" />
-		<child link="laser" />
-		<origin xyz="${x_hokuyo} ${y_hokuyo} ${z_hokuyo}" rpy="0 ${pi - pitch_angle_hokuyo} ${pi}" />
-	</joint> -->
+  <link name="laser">
+    <visual>
+      <geometry>
+        <mesh filename="package://mybot_description/meshes/hokuyo.dae"/>
+      </geometry>
+    </visual>
+    <collision>
+      <geometry>
+        <mesh filename="package://mybot_description/meshes/hokuyo.dae"/>
+      </geometry>
+    </collision>
+    <inertial>
+      <mass value="0.001"/>
+      <inertia ixx="4.94e-05" ixy="0.0" ixz="0.0" iyy="6.11e-05" iyz="0.0" izz="4.94e-05"/>
+    </inertial>
+  </link>
+  <joint name="hokuyo_base" type="fixed">
+    <parent link="tracao_f"/>
+    <child link="laser"/>
+    <origin rpy="0 3.661592 3.141592" xyz="0.233 0.0 -0.1"/>
+  </joint>
   <!-- Sonares -->
-  <!-- <link name="obstacle_sonar_down">
+  <link name="obstacle_sonar_down">
     <visual>
       <geometry>
@@ -633,4 +641,9 @@
       <material name="grey"/>
     </visual>
+    <collision>
+      <geometry>
+        <mesh filename="package://mybot_description/meshes/maxsonar.dae"/>
+      </geometry>
+    </collision>
     <inertial>
       <mass value="1e-5"/>
@@ -638,6 +651,6 @@
       <inertia ixx="1e-6" ixy="0" ixz="0" iyy="1e-6" iyz="0" izz="1e-6"/>
     </inertial>
-  </link> -->
-  <!-- <joint name="obstacle_sonar_down_base" type="fixed">
+  </link>
+  <joint name="obstacle_sonar_down_base" type="fixed">
     <parent link="tracao_f"/>
     <child link="obstacle_sonar_down"/>
@@ -651,4 +664,9 @@
       <material name="grey"/>
     </visual>
+    <collision>
+      <geometry>
+        <mesh filename="package://mybot_description/meshes/maxsonar.dae"/>
+      </geometry>
+    </collision>
     <inertial>
       <mass value="1e-5"/>
@@ -663,11 +681,16 @@
       <origin rpy="0 0 0" xyz="-0.0025 -0.02395 0.0"/>
     </visual>
-  </link> -->
-  <!-- <joint name="obstacle_sonar_up_base" type="fixed">
+    <collision>
+      <geometry>
+        <box size="0.005 0.07 0.0221"/>
+      </geometry>
+      <origin rpy="0 0 0" xyz="-0.0025 -0.02395 0.0"/>
+    </collision>
+  </link>
+  <joint name="obstacle_sonar_up_base" type="fixed">
     <parent link="garra_tracao_f2"/>
     <child link="obstacle_sonar_up"/>
     <origin rpy="0 0 0" xyz="0.024 0.075 0.19615"/>
-  </joint> -->
-  <!--
+  </joint>
 	<link name="ground_sonar" >
 		<visual>
@@ -675,12 +698,20 @@
 				<mesh filename="package://mybot_description/meshes/groundsonar.dae"/>
 			</geometry>
-			<xacro:cor />
 		</visual>
+    <collision>
+      <geometry>
+        <mesh filename="package://mybot_description/meshes/groundsonar.dae"/>
+      </geometry>
+    </collision>
+    <inertial>
+      <mass value="1e-5"/>
+      <inertia ixx="1e-6" ixy="0" ixz="0" iyy="1e-6" iyz="0" izz="1e-6"/>
+    </inertial>
 	</link>
 	<joint name="ground_sonar_base" type="fixed">
 		<parent link="base_link" />
 		<child link="ground_sonar" />
-		<origin xyz="${x_ground_sonar} ${w_eletr_ap/2 + y_ground_sonar} ${z_ground_sonar}" rpy="0 0 0" />
-	</joint> -->
+		<origin xyz="0 0 -0.135" rpy="0 0 0" />
+	</joint>
   <!-- FRAMES VIRTUAIS NO CABO -->
   <!-- Tracao -->
