Commit message: testing new shafts

File: mybot_description/urdf/piro.xacro (robot description, xacro)
@@ -120,14 +120,14 @@
     <visual name = 'central_traction'>
       <geometry>
-        <mesh filename="package://mybot_description/meshes/Shaft_piro3.dae"/>
-      </geometry>
-      <origin rpy="1.57 0 0" xyz="0.01 0.045 0.042"/>
+        <mesh filename="package://mybot_description/meshes/Shaft_piro3_V2.dae"/>
+      </geometry>
+      <origin rpy="1.57 0 0" xyz="0.00 0.045 0.0"/>
     </visual>
     <!-- This collision is for the central traction unit -->
     <collision name = 'central_traction'>
       <geometry>
-        <mesh filename="package://mybot_description/meshes/Shaft_piro3.dae"/>
-      </geometry>
-      <origin rpy="1.57 0 0" xyz="0.01 0.045 0.042"/>
+        <mesh filename="package://mybot_description/meshes/Shaft_piro3_V2.dae"/>
+      </geometry>
+      <origin rpy="1.57 0 0" xyz="0.00 0.045 0.0"/>
     </collision>
     <inertial>
@@ -383,8 +383,8 @@
     <visual>
       <geometry>
-        <mesh filename="package://mybot_description/meshes/Shaft_piro3.dae"/>
-      </geometry>
-      <material name="grey"/>
-      <origin rpy="1.57 0 0" xyz="0.01 0.045 0.042"/>
+        <mesh filename="package://mybot_description/meshes/Shaft_piro3_V2.dae"/>
+      </geometry>
+      <material name="grey"/>
+      <origin rpy="1.57 0 0" xyz="0.00 0.045 0.0"/>
       <!-- <origin rpy="0 0 0" xyz="0.0 0.012 0.025"/> -->
     </visual>
@@ -392,7 +392,7 @@
     <collision>
       <geometry>
-        <mesh filename="package://mybot_description/meshes/Shaft_piro3.dae"/>
-      </geometry>
-      <origin rpy="1.57 0 0" xyz="0.01 0.045 0.042"/>
+        <mesh filename="package://mybot_description/meshes/Shaft_piro3_V2.dae"/>
+      </geometry>
+      <origin rpy="1.57 0 0" xyz="0.00 0.045 0.0"/>
     </collision>
     <inertial>
@@ -448,7 +448,7 @@
     <visual>
       <geometry>
-        <mesh filename="package://mybot_description/meshes/Shaft_piro3.dae"/>
-      </geometry>
-      <origin rpy="1.57 0 0" xyz="0.01 0.045 0.042"/>
+        <mesh filename="package://mybot_description/meshes/Shaft_piro3_V2.dae"/>
+      </geometry>
+      <origin rpy="1.57 0 0" xyz="0.00 0.045 0.0"/>
       <material name="grey"/>
       <!-- <origin rpy="0 0 0" xyz="0.0 0.012 0.025"/> -->
@@ -457,7 +457,7 @@
     <collision>
       <geometry>
-        <mesh filename="package://mybot_description/meshes/Shaft_piro3.dae"/>
-      </geometry>
-      <origin rpy="1.57 0 0" xyz="0.01 0.045 0.042"/>
+        <mesh filename="package://mybot_description/meshes/Shaft_piro3_V2.dae"/>
+      </geometry>
+      <origin rpy="1.57 0 0" xyz="0.00 0.045 0.0"/>
     </collision>
     <inertial>
@@ -516,7 +516,7 @@
     <visual>
       <geometry>
-        <mesh filename="package://mybot_description/meshes/Shaft_piro3.dae"/>
-      </geometry>
-      <origin rpy="1.57 0 0" xyz="0.01 0.045 0.042"/>
+        <mesh filename="package://mybot_description/meshes/Shaft_piro3_V2.dae"/>
+      </geometry>
+      <origin rpy="1.57 0 0" xyz="0.00 0.045 0.0"/>
       <material name="grey"/>
       <!-- <origin rpy="0 0 0" xyz="0.0 0.012 0.025"/> -->
@@ -525,7 +525,7 @@
     <collision>
       <geometry>
-        <mesh filename="package://mybot_description/meshes/Shaft_piro3.dae"/>
-      </geometry>
-      <origin rpy="1.57 0 0" xyz="0.01 0.045 0.042"/>
+        <mesh filename="package://mybot_description/meshes/Shaft_piro3_V2.dae"/>
+      </geometry>
+      <origin rpy="1.57 0 0" xyz="0.00 0.045 0.0"/>
     </collision>
     <inertial>
@@ -583,7 +583,7 @@
     <visual>
       <geometry>
-        <mesh filename="package://mybot_description/meshes/Shaft_piro3.dae"/>
-      </geometry>
-      <origin rpy="1.57 0 0" xyz="0.01 0.045 0.042"/>
+        <mesh filename="package://mybot_description/meshes/Shaft_piro3_V2.dae"/>
+      </geometry>
+      <origin rpy="1.57 0 0" xyz="0.00 0.045 0.0"/>
       <material name="grey"/>
       <!-- <origin rpy="0 0 0" xyz="0.0 0.012 0.025"/> -->
@@ -592,7 +592,7 @@
     <collision>
       <geometry>
-        <mesh filename="package://mybot_description/meshes/Shaft_piro3.dae"/>
-      </geometry>
-      <origin rpy="1.57 0 0" xyz="0.01 0.045 0.042"/>
+        <mesh filename="package://mybot_description/meshes/Shaft_piro3_V2.dae"/>
+      </geometry>
+      <origin rpy="1.57 0 0" xyz="0.00 0.045 0.0"/>
     </collision>
     <inertial>

Commit message: Fixed the central shaft position and changed shafts to old model that works

File: mybot_description/urdf/piro.xacro (robot description, xacro)
@@ -110,5 +110,5 @@
     <parent link="garra_ap"/>
     <child link="eixo_tracao_ap"/>
-    <origin rpy="0 0 0" xyz="0.0 0.049 0.1345"/>
+    <origin rpy="0 0 0" xyz="0.0 0.049 0.172"/>
     <axis xyz="0 1 0"/>
     <dynamics damping="0.7" friction="1.0" />
@@ -120,14 +120,14 @@
     <visual name = 'central_traction'>
       <geometry>
-        <mesh filename="package://mybot_description/meshes/Shaft_piro3_V2.dae"/>
-      </geometry>
-      <origin rpy="1.57 0 0" xyz="0.00 0.045 0.0"/>
+        <mesh filename="package://mybot_description/meshes/shaft_simple.dae"/>
+      </geometry>
+      <origin rpy="0 0 0" xyz="0.0 0.0 0.0"/>
     </visual>
     <!-- This collision is for the central traction unit -->
     <collision name = 'central_traction'>
       <geometry>
-        <mesh filename="package://mybot_description/meshes/Shaft_piro3_V2.dae"/>
-      </geometry>
-      <origin rpy="1.57 0 0" xyz="0.00 0.045 0.0"/>
+        <mesh filename="package://mybot_description/meshes/shaft_simple.dae"/>
+      </geometry>
+      <origin rpy="0 0 0" xyz="0.0 0.0 0.0"/>
     </collision>
     <inertial>
@@ -383,8 +383,8 @@
     <visual>
       <geometry>
-        <mesh filename="package://mybot_description/meshes/Shaft_piro3_V2.dae"/>
-      </geometry>
-      <material name="grey"/>
-      <origin rpy="1.57 0 0" xyz="0.00 0.045 0.0"/>
+        <mesh filename="package://mybot_description/meshes/shaft_simple.dae"/>
+      </geometry>
+      <material name="grey"/>
+      <origin rpy="0 0 0" xyz="0.0 0.0 0.0"/>
       <!-- <origin rpy="0 0 0" xyz="0.0 0.012 0.025"/> -->
     </visual>
@@ -392,7 +392,7 @@
     <collision>
       <geometry>
-        <mesh filename="package://mybot_description/meshes/Shaft_piro3_V2.dae"/>
-      </geometry>
-      <origin rpy="1.57 0 0" xyz="0.00 0.045 0.0"/>
+        <mesh filename="package://mybot_description/meshes/shaft_simple.dae"/>
+      </geometry>
+      <origin rpy="0 0 0" xyz="0.0 0.0 0.0"/>
     </collision>
     <inertial>
@@ -448,7 +448,7 @@
     <visual>
       <geometry>
-        <mesh filename="package://mybot_description/meshes/Shaft_piro3_V2.dae"/>
-      </geometry>
-      <origin rpy="1.57 0 0" xyz="0.00 0.045 0.0"/>
+        <mesh filename="package://mybot_description/meshes/shaft_simple.dae"/>
+      </geometry>
+      <origin rpy="0 0 0" xyz="0.0 0.0 0.0"/>
       <material name="grey"/>
       <!-- <origin rpy="0 0 0" xyz="0.0 0.012 0.025"/> -->
@@ -457,7 +457,7 @@
     <collision>
       <geometry>
-        <mesh filename="package://mybot_description/meshes/Shaft_piro3_V2.dae"/>
-      </geometry>
-      <origin rpy="1.57 0 0" xyz="0.00 0.045 0.0"/>
+        <mesh filename="package://mybot_description/meshes/shaft_simple.dae"/>
+      </geometry>
+      <origin rpy="0 0 0" xyz="0.0 0.0 0.0"/>
     </collision>
     <inertial>
@@ -516,7 +516,7 @@
     <visual>
       <geometry>
-        <mesh filename="package://mybot_description/meshes/Shaft_piro3_V2.dae"/>
-      </geometry>
-      <origin rpy="1.57 0 0" xyz="0.00 0.045 0.0"/>
+        <mesh filename="package://mybot_description/meshes/shaft_simple.dae"/>
+      </geometry>
+      <origin rpy="0 0 0" xyz="0.0 0.0 0.0"/>
       <material name="grey"/>
       <!-- <origin rpy="0 0 0" xyz="0.0 0.012 0.025"/> -->
@@ -525,7 +525,7 @@
     <collision>
       <geometry>
-        <mesh filename="package://mybot_description/meshes/Shaft_piro3_V2.dae"/>
-      </geometry>
-      <origin rpy="1.57 0 0" xyz="0.00 0.045 0.0"/>
+        <mesh filename="package://mybot_description/meshes/shaft_simple.dae"/>
+      </geometry>
+      <origin rpy="0 0 0" xyz="0.0 0.0 0.0"/>
     </collision>
     <inertial>
@@ -583,7 +583,7 @@
     <visual>
       <geometry>
-        <mesh filename="package://mybot_description/meshes/Shaft_piro3_V2.dae"/>
-      </geometry>
-      <origin rpy="1.57 0 0" xyz="0.00 0.045 0.0"/>
+        <mesh filename="package://mybot_description/meshes/shaft_simple.dae"/>
+      </geometry>
+      <origin rpy="0 0 0" xyz="0.0 0.0 0.0"/>
       <material name="grey"/>
       <!-- <origin rpy="0 0 0" xyz="0.0 0.012 0.025"/> -->
@@ -592,7 +592,7 @@
     <collision>
       <geometry>
-        <mesh filename="package://mybot_description/meshes/Shaft_piro3_V2.dae"/>
-      </geometry>
-      <origin rpy="1.57 0 0" xyz="0.00 0.045 0.0"/>
+        <mesh filename="package://mybot_description/meshes/shaft_simple.dae"/>
+      </geometry>
+      <origin rpy="0 0 0" xyz="0.0 0.0 0.0"/>
     </collision>
     <inertial>

Commit message: Corrected shaft positions

File: mybot_description/urdf/piro.xacro (robot description, xacro)
@@ -373,5 +373,5 @@
     <parent link="garra_tracao_f1"/>
     <child link="eixo_tracao_f1"/>
-    <origin rpy="0 0 0" xyz="0.0 0.049 0.145"/>
+    <origin rpy="0 0 0" xyz="0.0 0.06 0.172"/>
     <axis xyz="0 1 0"/>
     <dynamics damping="0.7" friction="1.0" />
@@ -438,5 +438,5 @@
     <parent link="garra_tracao_f2"/>
     <child link="eixo_tracao_f2"/>
-    <origin rpy="0 0 0" xyz="0.0 0.049 0.145"/>
+    <origin rpy="0 0 0" xyz="0.0 0.06 0.172"/>
     <axis xyz="0 1 0"/>
     <dynamics damping="0.7" friction="1.0" />
@@ -506,5 +506,5 @@
     <parent link="garra_tracao_t1"/>
     <child link="eixo_tracao_t1"/>
-    <origin rpy="0 0 0" xyz="0.0 0.049 0.145"/>
+    <origin rpy="0 0 0" xyz="0.0 0.06 0.172"/>
     <axis xyz="0 1 0"/>
     <dynamics damping="0.7" friction="1.0" />
@@ -573,5 +573,5 @@
     <parent link="garra_tracao_t2"/>
     <child link="eixo_tracao_t2"/>
-    <origin rpy="0 0 0" xyz="0.0 0.049 0.145"/>
+    <origin rpy="0 0 0" xyz="0.0 0.06 0.172"/>
     <axis xyz="0 1 0"/>
     <dynamics damping="0.7" friction="1.0" />

Commit message: Adjusted claws position

File: mybot_description/urdf/piro.xacro (robot description, xacro)
@@ -341,5 +341,5 @@
     <parent link="tracao_f"/>
     <child link="garra_tracao_f1"/>
-    <origin rpy="0 0 3.141592" xyz="0.0005 0.075 0.06985"/>
+    <origin rpy="0 0 3.141592" xyz="0.0005 0.09 0.06985"/>
     <limit effort="1000.0" lower="-3.14" upper="3.14" velocity="0.5"/>
     <axis xyz="0 0 1"/>
@@ -406,5 +406,5 @@
     <parent link="tracao_f"/>
     <child link="garra_tracao_f2"/>
-    <origin rpy="0 0 0" xyz="0.1765 -0.075 0.06985"/>
+    <origin rpy="0 0 0" xyz="0.1765 -0.09 0.06985"/>
     <limit effort="1000.0" lower="-3.14" upper="3.14" velocity="0.5"/>
     <axis xyz="0 0 1"/>
@@ -473,5 +473,5 @@
     <parent link="tracao_t"/>
     <child link="garra_tracao_t1"/>
-    <origin rpy="0 0 0" xyz="0.0005 -0.075 0.06985"/>
+    <origin rpy="0 0 0" xyz="0.0005 -0.09 0.06985"/>
     <limit effort="1000.0" lower="-3.14" upper="3.14" velocity="0.5"/>
     <axis xyz="0 0 1"/>
@@ -540,5 +540,5 @@
     <parent link="tracao_t"/>
     <child link="garra_tracao_t2"/>
-    <origin rpy="0 0 3.141592" xyz="0.1765 0.075 0.06985"/>
+    <origin rpy="0 0 3.141592" xyz="0.1765 0.09 0.06985"/>
     <limit effort="1000.0" lower="-3.14" upper="3.14" velocity="0.5"/>
     <axis xyz="0 0 1"/>

Commit message: fixed shaft visual, collision and position

File: mybot_description/urdf/piro.xacro (robot description, xacro)
@@ -120,14 +120,14 @@
     <visual name = 'central_traction'>
       <geometry>
-        <mesh filename="package://mybot_description/meshes/shaft_simple.dae"/>
-      </geometry>
-      <origin rpy="0 0 0" xyz="0.0 0.0 0.0"/>
+        <mesh filename="package://mybot_description/meshes/Shaft_piro3_V2.dae"/>
+      </geometry>
+      <origin rpy="1.57 0 0" xyz="0.0 0.05 0.0"/>
     </visual>
     <!-- This collision is for the central traction unit -->
     <collision name = 'central_traction'>
       <geometry>
-        <mesh filename="package://mybot_description/meshes/shaft_simple.dae"/>
-      </geometry>
-      <origin rpy="0 0 0" xyz="0.0 0.0 0.0"/>
+        <mesh filename="package://mybot_description/meshes/Shaft_piro3_V2.dae"/>
+      </geometry>
+      <origin rpy="1.57 0 0" xyz="0.0 0.05 0.0"/>
     </collision>
     <inertial>
@@ -141,5 +141,6 @@
     <parent link="base_link"/>
     <child link="link1_f"/>
-    <origin rpy=" 0 -0.60 3.141592" xyz="-0.13 0.0 0.079"/>
+    <!-- <origin rpy=" 0 -0.60 3.141592" xyz="-0.13 0.0 0.079"/> -->
+    <origin rpy=" 0 0 3.141592" xyz="-0.13 0.0 0.079"/>
     <limit effort="1000.0" lower="-1.74" upper="0.7" velocity="0.5"/>
     <axis xyz="0 1 0"/>
@@ -179,5 +180,6 @@
     <parent link="base_link"/>
     <child link="link1_t"/>
-    <origin rpy="0 -0.60 0" xyz="0.13 0.0 0.079"/>
+    <!-- <origin rpy="0 -0.60 0" xyz="0.13 0.0 0.079"/> -->
+    <origin rpy=" 0 0 0" xyz="0.13 0.0 0.079"/>
     <limit effort="1000.0" lower="-1.74" upper="0.7" velocity="0.5"/>
     <axis xyz="0 1 0"/>
@@ -383,16 +385,17 @@
     <visual>
       <geometry>
-        <mesh filename="package://mybot_description/meshes/shaft_simple.dae"/>
-      </geometry>
-      <material name="grey"/>
-      <origin rpy="0 0 0" xyz="0.0 0.0 0.0"/>
-      <!-- <origin rpy="0 0 0" xyz="0.0 0.012 0.025"/> -->
+        <mesh filename="package://mybot_description/meshes/Shaft_piro3_V2.dae"/>
+      </geometry>
+      <material name="grey"/>
+      <!-- <origin rpy="0 0 0" xyz="0.0 0.0 0.0"/> -->
+      <origin rpy="1.57 0 0" xyz="0.0 0.05 0.0"/>
     </visual>
     <!-- This collision is for the front f1 traction unit -->
     <collision>
       <geometry>
-        <mesh filename="package://mybot_description/meshes/shaft_simple.dae"/>
-      </geometry>
-      <origin rpy="0 0 0" xyz="0.0 0.0 0.0"/>
+        <mesh filename="package://mybot_description/meshes/Shaft_piro3_V2.dae"/>
+      </geometry>
+      <!-- <origin rpy="0 0 0" xyz="0.0 0.0 0.0"/> -->
+      <origin rpy="1.57 0 0" xyz="0.0 0.05 0.0"/>
     </collision>
     <inertial>
@@ -448,16 +451,17 @@
     <visual>
       <geometry>
-        <mesh filename="package://mybot_description/meshes/shaft_simple.dae"/>
-      </geometry>
-      <origin rpy="0 0 0" xyz="0.0 0.0 0.0"/>
-      <material name="grey"/>
-      <!-- <origin rpy="0 0 0" xyz="0.0 0.012 0.025"/> -->
+        <mesh filename="package://mybot_description/meshes/Shaft_piro3_V2.dae"/>
+      </geometry>
+      <!-- <origin rpy="0 0 0" xyz="0.0 0.0 0.0"/> -->
+      <material name="grey"/>
+      <origin rpy="1.57 0 0" xyz="0.0 0.05 0.0"/>
     </visual>
     <!-- This collision is for the front f2 traction unit -->
     <collision>
       <geometry>
-        <mesh filename="package://mybot_description/meshes/shaft_simple.dae"/>
-      </geometry>
-      <origin rpy="0 0 0" xyz="0.0 0.0 0.0"/>
+        <mesh filename="package://mybot_description/meshes/Shaft_piro3_V2.dae"/>
+      </geometry>
+      <!-- <origin rpy="0 0 0" xyz="0.0 0.0 0.0"/> -->
+      <origin rpy="1.57 0 0" xyz="0.0 0.05 0.0"/>
     </collision>
     <inertial>
@@ -516,16 +520,17 @@
     <visual>
       <geometry>
-        <mesh filename="package://mybot_description/meshes/shaft_simple.dae"/>
-      </geometry>
-      <origin rpy="0 0 0" xyz="0.0 0.0 0.0"/>
-      <material name="grey"/>
-      <!-- <origin rpy="0 0 0" xyz="0.0 0.012 0.025"/> -->
+        <mesh filename="package://mybot_description/meshes/Shaft_piro3_V2.dae"/>
+      </geometry>
+      <!-- <origin rpy="0 0 0" xyz="0.0 0.0 0.0"/> -->
+      <material name="grey"/>
+      <origin rpy="1.57 0 0" xyz="0.0 0.05 0.0"/>
     </visual>
     <!-- This collision is for the back t1 traction unit -->
     <collision>
       <geometry>
-        <mesh filename="package://mybot_description/meshes/shaft_simple.dae"/>
-      </geometry>
-      <origin rpy="0 0 0" xyz="0.0 0.0 0.0"/>
+        <mesh filename="package://mybot_description/meshes/Shaft_piro3_V2.dae"/>
+      </geometry>
+      <!-- <origin rpy="0 0 0" xyz="0.0 0.0 0.0"/> -->
+      <origin rpy="1.57 0 0" xyz="0.0 0.05 0.0"/>
     </collision>
     <inertial>
@@ -583,16 +588,17 @@
     <visual>
       <geometry>
-        <mesh filename="package://mybot_description/meshes/shaft_simple.dae"/>
-      </geometry>
-      <origin rpy="0 0 0" xyz="0.0 0.0 0.0"/>
-      <material name="grey"/>
-      <!-- <origin rpy="0 0 0" xyz="0.0 0.012 0.025"/> -->
+        <mesh filename="package://mybot_description/meshes/Shaft_piro3_V2.dae"/>
+      </geometry>
+      <!-- <origin rpy="0 0 0" xyz="0.0 0.0 0.0"/> -->
+      <material name="grey"/>
+      <origin rpy="1.57 0 0" xyz="0.0 0.05 0.0"/>
     </visual>
     <!-- This collision is for the back t2 traction unit -->
     <collision>
       <geometry>
-        <mesh filename="package://mybot_description/meshes/shaft_simple.dae"/>
-      </geometry>
-      <origin rpy="0 0 0" xyz="0.0 0.0 0.0"/>
+        <mesh filename="package://mybot_description/meshes/Shaft_piro3_V2.dae"/>
+      </geometry>
+      <!-- <origin rpy="0 0 0" xyz="0.0 0.0 0.0"/> -->
+      <origin rpy="1.57 0 0" xyz="0.0 0.05 0.0"/>
     </collision>
     <inertial>

Commit message: Change arm position to start with the 5 shafts on line.

File: mybot_description/urdf/piro.xacro (robot description, xacro)
@@ -138,5 +138,5 @@
     <child link="link1_f"/>
     <!-- <origin rpy=" 0 -0.60 3.141592" xyz="-0.13 0.0 0.079"/> -->
-    <origin rpy=" 0 0 3.141592" xyz="-0.13 0.0 0.079"/>
+    <origin rpy=" 0 -0.6 3.141592" xyz="-0.13 0.0 0.079"/>
     <limit effort="1000.0" lower="-1.74" upper="0.7" velocity="0.5"/>
     <axis xyz="0 1 0"/>
@@ -177,5 +177,5 @@
     <child link="link1_t"/>
     <!-- <origin rpy="0 -0.60 0" xyz="0.13 0.0 0.079"/> -->
-    <origin rpy=" 0 0 0" xyz="0.13 0.0 0.079"/>
+    <origin rpy=" 0 -0.6 0" xyz="0.13 0.0 0.079"/>
     <limit effort="1000.0" lower="-1.74" upper="0.7" velocity="0.5"/>
     <axis xyz="0 1 0"/>

Commit message: Alianged the shafts

File: mybot_description/urdf/piro.xacro (robot description, xacro)
@@ -385,5 +385,5 @@
       <material name="grey"/>
       <!-- <origin rpy="0 0 0" xyz="0.0 0.0 0.0"/> -->
-      <origin rpy="1.57 0 0" xyz="0.0 0.05 0.0"/>
+      <origin rpy="1.57 0 0" xyz="0.0 0.045 0.0"/>
     </visual>
     <!-- This collision is for the front f1 traction unit -->
@@ -393,5 +393,5 @@
       </geometry>
       <!-- <origin rpy="0 0 0" xyz="0.0 0.0 0.0"/> -->
-      <origin rpy="1.57 0 0" xyz="0.0 0.05 0.0"/>
+      <origin rpy="1.57 0 0" xyz="0.0 0.045 0.0"/>
     </collision>
     <inertial>
@@ -451,5 +451,5 @@
       <!-- <origin rpy="0 0 0" xyz="0.0 0.0 0.0"/> -->
       <material name="grey"/>
-      <origin rpy="1.57 0 0" xyz="0.0 0.05 0.0"/>
+      <origin rpy="1.57 0 0" xyz="0.0 0.055 0.0"/>
     </visual>
     <!-- This collision is for the front f2 traction unit -->
@@ -459,5 +459,5 @@
       </geometry>
       <!-- <origin rpy="0 0 0" xyz="0.0 0.0 0.0"/> -->
-      <origin rpy="1.57 0 0" xyz="0.0 0.05 0.0"/>
+      <origin rpy="1.57 0 0" xyz="0.0 0.055 0.0"/>
     </collision>
     <inertial>
@@ -520,5 +520,5 @@
       <!-- <origin rpy="0 0 0" xyz="0.0 0.0 0.0"/> -->
       <material name="grey"/>
-      <origin rpy="1.57 0 0" xyz="0.0 0.05 0.0"/>
+      <origin rpy="1.57 0 0" xyz="0.0 0.045 0.0"/>
     </visual>
     <!-- This collision is for the back t1 traction unit -->
@@ -528,5 +528,5 @@
       </geometry>
       <!-- <origin rpy="0 0 0" xyz="0.0 0.0 0.0"/> -->
-      <origin rpy="1.57 0 0" xyz="0.0 0.05 0.0"/>
+      <origin rpy="1.57 0 0" xyz="0.0 0.045 0.0"/>
     </collision>
     <inertial>
@@ -588,5 +588,5 @@
       <!-- <origin rpy="0 0 0" xyz="0.0 0.0 0.0"/> -->
       <material name="grey"/>
-      <origin rpy="1.57 0 0" xyz="0.0 0.05 0.0"/>
+      <origin rpy="1.57 0 0" xyz="0.0 0.055 0.0"/>
     </visual>
     <!-- This collision is for the back t2 traction unit -->
@@ -596,5 +596,5 @@
       </geometry>
       <!-- <origin rpy="0 0 0" xyz="0.0 0.0 0.0"/> -->
-      <origin rpy="1.57 0 0" xyz="0.0 0.05 0.0"/>
+      <origin rpy="1.57 0 0" xyz="0.0 0.055 0.0"/>
     </collision>
     <inertial>

Commit message: fixed arms position

File: mybot_description/urdf/piro.xacro (robot description, xacro)
@@ -157,5 +157,5 @@
       </geometry>
       <material name="grey"/>
-      <origin rpy="0 0 0" xyz="0.1885 0.0 0.0"/>
+      <origin rpy="0 0 0" xyz="0.20995 0.0 0.0"/>
     </visual>
     <!-- this collision is for the front arm unit -->
@@ -164,5 +164,5 @@
         <box size="0.4199 0.05 0.100"/>
       </geometry>
-      <origin rpy="0 0 0" xyz="0.1885 0.0 0.0"/>
+      <origin rpy="0 0 0" xyz="0.20995 0.0 0.0"/>
     </collision>
     <inertial>
@@ -196,5 +196,5 @@
       </geometry>
       <material name="grey"/>
-      <origin rpy="0 0 0" xyz="0.1885 0.0 0.0"/>
+      <origin rpy="0 0 0" xyz="0.20995 0.0 0.0"/>
     </visual>
     <!-- this collision is for the back arm unit -->
@@ -203,5 +203,5 @@
         <box size="0.4199 0.05 0.100"/>
       </geometry>
-      <origin rpy="0 0 0" xyz="0.1885 0.0 0.0"/>
+      <origin rpy="0 0 0" xyz="0.20995 0.0 0.0"/>
     </collision>
     <inertial>
@@ -227,5 +227,5 @@
       </geometry>
       <material name="grey"/>
-      <origin rpy="0 0 0" xyz="0.0885 0.0 0.0201"/>
+      <origin rpy="0 0 0" xyz="0.1165 0.0 0.0201"/>
     </visual>
     <!-- This visual represents the front traction claw f2 support -->
@@ -252,5 +252,5 @@
         <box size="0.233 0.100 0.100"/>
       </geometry>
-      <origin rpy="0 0 0" xyz="0.0885 0.0 0.0201"/>
+      <origin rpy="0 0 0" xyz="0.1165 0.0 0.0201"/>
     </collision>
     <!-- this collision is for the front traction claw f2 support -->
@@ -290,5 +290,5 @@
       </geometry>
       <material name="grey"/>
-      <origin rpy="0 0 0" xyz="0.0885 0.0 0.0201"/>
+      <origin rpy="0 0 0" xyz="0.1165 0.0 0.0201"/>
     </visual>
     <!-- This visual represents the  back traction claw f1 support -->
@@ -313,5 +313,5 @@
         <box size="0.233 0.100 0.100"/>
       </geometry>
-      <origin rpy="0 0 0" xyz="0.0885 0.0 0.0201"/>
+      <origin rpy="0 0 0" xyz="0.1165 0.0 0.0201"/>
     </collision>
     <!-- this collision is for the back traction claw f1 support -->
