Commit message: Add Ir Camera simulation
The line obstacles color were changed to RED, so the plugin will recognize it as
an OOI (Object of Interest), the piro.gazebo file was renamed to piro.gazebo.xacro
in order to use it with VSCode

File: mybot_description/urdf/piro.gazebo.xacro (robot description, xacro)
@@ -1,3 +1,6 @@
-<robot name="robo_cemig" xmlns:xacro="http://www.ros.org/wiki/xacro">
+<robot name="robo_cemig" xmlns:xacro="http://www.ros.org/wiki/xacro"
+xmlns:sensor="http://playerstage.sourceforge.net/gazebo/xmlschema/#sensor"
+xmlns:controller="http://playerstage.sourceforge.net/gazebo/xmlschema/#controller"
+xmlns:interface="http://playerstage.sourceforge.net/gazebo/xmlschema/#interface">
   <gazebo>
     <plugin filename="libgazebo_ros_control.so" name="gazebo_ros_control">
@@ -93,7 +96,4 @@
         <noise>
           <type>gaussian</type>
-          <!-- Noise is sampled independently per pixel on each frame.
-               That pixel's noise value is added to each of its color
-               channels, which at that point lie in the range [0,1]. -->
           <mean>0.0</mean>
           <stddev>0.007</stddev>
@@ -103,5 +103,5 @@
         <alwaysOn>true</alwaysOn>
         <updateRate>0.0</updateRate>
-        <cameraName>elir/zed_left_camera</cameraName>
+        <cameraName>detection/zed_left_camera</cameraName>
         <imageTopicName>image_raw</imageTopicName>
         <cameraInfoTopicName>camera_info</cameraInfoTopicName>
@@ -132,7 +132,4 @@
         <noise>
           <type>gaussian</type>
-          <!-- Noise is sampled independently per pixel on each frame.
-               That pixel's noise value is added to each of its color
-               channels, which at that point lie in the range [0,1]. -->
           <mean>0.0</mean>
           <stddev>0.007</stddev>
@@ -142,5 +139,5 @@
         <alwaysOn>true</alwaysOn>
         <updateRate>0.0</updateRate>
-        <cameraName>elir/zed_right_camera</cameraName>
+        <cameraName>detection/zed_right_camera</cameraName>
         <imageTopicName>image_raw</imageTopicName>
         <cameraInfoTopicName>camera_info</cameraInfoTopicName>
@@ -155,35 +152,30 @@
     </sensor>
   </gazebo>
-  <!--gazebo reference ="flir_camera">
-    <sensor:camera name="thermal_cam_sensor">
-      <imageSize>640 480</imageSize>
-      <imageFormat>R8G8B8</imageFormat>
-      <hfov>90</hfov>
-      <nearClip>0.01</nearClip>
-      <farClip>100</farClip>
-      <updateRate>5</updateRate>
-      <controller:gazebo_ros_thermal_camera name="thermal_cam_controller" plugin="libgazebo_ros_thermal_depth_camera.so">
-        <alwaysOn>true</alwaysOn>
-        <updateRate>5</updateRate>
-        <cameraName>thermal_cam</cameraName>
-        <imageTopicName>image_raw</imageTopicName>
-        <cameraInfoTopicName>camera_info</cameraInfoTopicName>
-        <frameName>thermal_cam_optical_frame</frameName>
-        <hackBaseline>0</hackBaseline>
-        <CxPrime>320.5</CxPrime>
-        <Cx>320.5</Cx>
-        <Cy>240.5</Cy>
-        <focalLength>320</focalLength>
-        <distortionK1>0.00000001</distortionK1>
-        <distortionK2>0.00000001</distortionK2>
-        <distortionK3>0.00000001</distortionK3>
-        <distortionT1>0.00000001</distortionT1>
-        <distortionT2>0.00000001</distortionT2>
-        <interface:camera name="thermal_cam_iface"/>
-      </controller:gazebo_ros_thermal_camera>
-    </sensor:camera>
-    <turnGravityOff>true</turnGravityOff>
-    <material>PR2/Blue</material>
-</gazebo-->
+ <xacro:macro name="ir_camera" params="name ros_topic update_rate height width">
+    <gazebo reference="${name}">
+      <sensor type="camera" name="thermal_camera_sensor">
+        <update_rate>30</update_rate>
+        <camera>
+          <horizontal_fov>${90.0*M_PI/180.0}</horizontal_fov>
+          <image>
+            <format>R8G8B8</format>
+            <width>${width}</width>
+            <height>${height}</height>
+          </image>
+          <clip>
+            <near>0.1</near>
+            <far>300</far>
+          </clip>
+        </camera>
+        <plugin name="thermal_camera_controller" filename="libgazebo_ros_thermal_camera.so">
+          <alwaysOn>true</alwaysOn>
+          <updateRate>${update_rate}</updateRate>
+          <imageTopicName>/${ros_topic}/image_raw</imageTopicName>
+          <cameraInfoTopicName>/${ros_topic}/camera_info</cameraInfoTopicName>
+          <frameName>${name}_optical_frame</frameName>
+        </plugin>
+      </sensor>
+    </gazebo>
+</xacro:macro>
   <xacro:macro name="sonar_sensor" params="name ros_topic update_rate min_range max_range field_of_view ray_count">
     <gazebo reference="${name}">
@@ -222,5 +214,5 @@
     </gazebo>
   </xacro:macro>
-  <xacro:sonar_sensor name="obstacle_sonar_up" ros_topic="sonar/up" update_rate="20" min_range="0.1524" max_range="100" field_of_view="1.0471" ray_count="100" />
-  <!--xacro:sonar_sensor name="ground_sonar" ros_topic="sonar/ground" update_rate="20" min_range="0.1524" max_range="0.645" field_of_view="60" ray_count="1" /-->
+  <xacro:sonar_sensor name="ground_sonar" ros_topic="perception/ground_sonar" update_rate="20" min_range="0.0" max_range="100" field_of_view="1.0471" ray_count="1" />
+  <xacro:ir_camera name="flir_camera" ros_topic = "perception/flir_camera" update_rate = "30" height = "800" width = "800" />
 </robot>

File: mybot_description/urdf/piro.urdf.xacro (robot description, xacro)
@@ -6,5 +6,5 @@
   <!-- ros_control plugin -->
   <xacro:include filename="$(find mybot_description)/urdf/materials.xacro" />
-  <xacro:include filename="$(find mybot_description)/urdf/piro.gazebo" />
+  <xacro:include filename="$(find mybot_description)/urdf/piro.gazebo.xacro" />
   <xacro:property name="M_PI" value="3.141592" />
   <!-- BASE LINK-->
@@ -741,5 +741,5 @@
     <link name="flir_camera">
         <visual>
-            <origin xyz="0 0 0" rpy="0 0 0"/>
+            <origin xyz="0 0 0" rpy="0 ${M_PI/2} 0"/>
             <geometry>
                 <mesh filename="package://mybot_description/meshes/LeptonBreakoutBoardWithLepton3.stl" scale="0.001 0.001 0.001"/>
@@ -750,13 +750,16 @@
         </visual>
     </link>
+    <!--<gazebo reference="flir_camera">
+      <material>Gazebo/Blue</material>
+    </gazebo>-->
   <joint name="zed_camera_joint" type="fixed">
     <parent link="base_link"/>
     <child link="zed_center"/>
-    <origin rpy="0 0 ${M_PI}" xyz="-0.17 0.0 -0.05"/>
+    <origin rpy="0 0 0" xyz="0.17 0.0 -0.1"/>
   </joint>
   <joint name="flir_camera_joint" type="fixed">
     <parent link="base_link"/>
     <child link="flir_camera"/>
-    <origin rpy="0 ${-M_PI/2} 0" xyz="-0.17 0.0 0.00"/>
+    <origin rpy="0 0 0" xyz="0.17 0.0 -0.05"/>
   </joint>
   <!-- Sonares -->

Commit message: Fix sonar sensor

File: mybot_description/urdf/piro.gazebo.xacro (robot description, xacro)
@@ -214,5 +214,5 @@
     </gazebo>
   </xacro:macro>
-  <xacro:sonar_sensor name="ground_sonar" ros_topic="perception/ground_sonar" update_rate="20" min_range="0.0" max_range="100" field_of_view="1.0471" ray_count="1" />
+  <xacro:sonar_sensor name="ground_sonar" ros_topic="perception/ground_sonar" update_rate="30" min_range="0.1" max_range="100" field_of_view="1.0471" ray_count="1" />
   <xacro:ir_camera name="flir_camera" ros_topic = "perception/flir_camera" update_rate = "30" height = "800" width = "800" />
 </robot>

File: mybot_description/urdf/piro.urdf.xacro (robot description, xacro)
@@ -202,4 +202,7 @@
     </inertial>
   </link>
+  <gazebo reference="traction_left_pallet">
+    <material>Gazebo/Black</material>
+  </gazebo>
   <!-- This joint binds the base body (represented by the link base_link) and the back arm unit (represented by the link link1_t). it can rotate with the y axis fixed, it has an upper limit of 0.7 (40 degrees) and a lower limit of -1.74 (-100 degrees) -->
   <joint name="joint1_t" type="revolute">
@@ -750,7 +753,4 @@
         </visual>
     </link>
-    <!--<gazebo reference="flir_camera">
-      <material>Gazebo/Blue</material>
-    </gazebo>-->
   <joint name="zed_camera_joint" type="fixed">
     <parent link="base_link"/>
@@ -800,14 +800,16 @@
     <origin rpy="0 0 0" xyz="0.024 0.075 0.19615"/>
   </joint>
-	<link name="ground_sonar" >
+<link name="ground_sonar" >
 		<visual>
 			<geometry>
-				<mesh filename="package://mybot_description/meshes/groundsonar.dae"/>
+      <mesh filename="package://mybot_description/meshes/groundsonar.dae"/>
 			</geometry>
-		</visual>
+      <origin rpy="0 ${-M_PI/2} 0" />
+    </visual>
     <collision>
       <geometry>
         <mesh filename="package://mybot_description/meshes/groundsonar.dae"/>
       </geometry>
+      <origin rpy="0 ${-M_PI/2} 0" />
     </collision>
     <inertial>
@@ -816,8 +818,11 @@
     </inertial>
 	</link>
+  <gazebo reference="ground_sonar">
+    <material>Gazebo/Blue</material>
+  </gazebo>
 	<joint name="ground_sonar_base" type="fixed">
 		<parent link="base_link" />
 		<child link="ground_sonar" />
-		<origin xyz="0 0 -0.135" rpy="0 0 0" />
+		<origin xyz="0 0 -0.155" rpy="0 ${M_PI/2} 0" />
 	</joint>
   <!-- FRAMES VIRTUAIS NO CABO -->

Commit message: Change the _t tag to _b tag, to represent the back of the robot and change the front and back links that were inverted

File: mybot_description/urdf/piro.gazebo.xacro (robot description, xacro)
@@ -29,5 +29,5 @@
     <material name="grey"/>
     </gazebo>
-  <gazebo reference="tracao_t">
+  <gazebo reference="tracao_b">
     <dampingFactor>0.01</dampingFactor>
     <material name="grey"/>
@@ -46,9 +46,9 @@
     <material name="grey"/>
     </gazebo>
-  <gazebo reference="garra_tracao_t1">
-    <dampingFactor>0.02</dampingFactor>
-    <material name="grey"/>
-    </gazebo>
-  <gazebo reference="garra_tracao_t2">
+  <gazebo reference="garra_tracao_b1">
+    <dampingFactor>0.02</dampingFactor>
+    <material name="grey"/>
+    </gazebo>
+  <gazebo reference="garra_tracao_b2">
     <dampingFactor>0.02</dampingFactor>
     <material name="grey"/>
@@ -70,10 +70,10 @@
     <material name="black"/>
     </gazebo>
-  <gazebo reference="eixo_tracao_t1">
-    <mu1>0.3</mu1>
-    <mu2>0.3</mu2>
-    <material name="black"/>
-    </gazebo>
-  <gazebo reference="eixo_tracao_t2">
+  <gazebo reference="eixo_tracao_b1">
+    <mu1>0.3</mu1>
+    <mu2>0.3</mu2>
+    <material name="black"/>
+    </gazebo>
+  <gazebo reference="eixo_tracao_b2">
     <mu1>0.3</mu1>
     <mu2>0.3</mu2>

File: mybot_description/urdf/piro.urdf.xacro (robot description, xacro)
@@ -136,7 +136,7 @@
   </link>
   <!-- This joint binds the base body (represented by the link base_link) and the front arm unit (represented by the link link1_f). it can rotate with the y axis fixed, it has an upper limit of 0.7 (40 degrees) and a lower limit of -1.74 (-100 degrees) -->
-  <joint name="joint1_f" type="revolute">
+  <joint name="joint1_b" type="revolute">
     <parent link="base_link"/>
-    <child link="link1_f"/>
+    <child link="link1_b"/>
     <!-- <origin rpy=" 0 -0.60 3.141592" xyz="-0.13 0.0 0.079"/> -->
     <origin rpy=" 0 -0.6 ${M_PI}" xyz="-0.13 0.0 0.079"/>
@@ -145,5 +145,5 @@
   </joint>
   <!-- This link represents the front arm unit  -->
-  <link name="link1_f">
+  <link name="link1_b">
     <!-- <visual>
       <geometry>
@@ -154,5 +154,5 @@
     </visual> -->
     <!-- This visual represents the front arm unit -->
-    <visual name = 'front_arm'>
+    <visual name = 'back_arm'>
       <geometry>
         <box size="0.19 0.100 0.05"/>
@@ -190,5 +190,5 @@
     </visual>
     <!-- this collision is for the front arm unit -->
-    <collision name = 'front_arm'>
+    <collision name = 'back_arm'>
       <geometry>
         <box size="0.19 0.100 0.05"/>
@@ -203,7 +203,7 @@
   </link>
   <!-- This joint binds the base body (represented by the link base_link) and the back arm unit (represented by the link link1_t). it can rotate with the y axis fixed, it has an upper limit of 0.7 (40 degrees) and a lower limit of -1.74 (-100 degrees) -->
-  <joint name="joint1_t" type="revolute">
+  <joint name="joint1_f" type="revolute">
     <parent link="base_link"/>
-    <child link="link1_t"/>
+    <child link="link1_f"/>
     <!-- <origin rpy="0 -0.60 0" xyz="0.13 0.0 0.079"/> -->
     <origin rpy=" 0 -0.6 0" xyz="0.13 0.0 0.079"/>
@@ -212,5 +212,5 @@
   </joint>
   <!-- This link represents the back arm unit  -->
-  <link name="link1_t">
+  <link name="link1_f">
     <!-- <visual>
       <geometry>
@@ -221,5 +221,5 @@
     </visual> -->
     <!-- This visual represents the back arm unit -->
-    <visual name = 'back_arm'>
+    <visual name = 'front_arm'>
       <geometry>
         <box size="0.19 0.100 0.05"/>
@@ -257,5 +257,5 @@
       <origin rpy="-${M_PI/2} -${M_PI} 0" xyz="${0.20995*2} -0.06 -${0.05/2}"/>
     </visual>
-    <collision name = 'back_arm'>
+    <collision name = 'front_arm'>
       <geometry>
         <box size="0.19 0.100 0.05"/>
@@ -332,8 +332,8 @@
     </inertial>
   </link>
-  <!-- This joint binds the back arm unit (represented by the link link1_t) and the back traction body unit (represented by the link tracao_t). It can rotate with the y axis fixed, it has an upper limit of 2.18 (125 degrees) and a lower limit of -1.0 (-57 degrees) -->
-  <joint name="joint2_t" type="revolute">
-    <parent link="link1_t"/>
-    <child link="tracao_t"/>
+  <!-- This joint binds the back arm unit (represented by the link link1_t) and the back traction body unit (represented by the link tracao_b). It can rotate with the y axis fixed, it has an upper limit of 2.18 (125 degrees) and a lower limit of -1.0 (-57 degrees) -->
+  <joint name="joint2_b" type="revolute">
+    <parent link="link1_b"/>
+    <child link="tracao_b"/>
     <origin rpy="0 0.57 0" xyz="0.39 0.0 0.0"/>
     <limit effort="1000.0" lower="-1.0" upper="2.18" velocity="0.5"/>
@@ -341,5 +341,5 @@
   </joint>
   <!-- This link represents the back traction body unit that contains back traction body, claw f1 support and claw f2 support -->
-  <link name="tracao_t">
+  <link name="tracao_b">
     <!-- This visual represents the  back traction body -->
     <visual name = 'back_traction_body'>
@@ -527,8 +527,8 @@
   <!-- GARRAS TRACAO TRASEIRA -->
   <!-- T1 -->
-  <!-- This joint binds the front traction body unit (represented by the link tracao_f) and the back t1 claw unit (represented by the link garra_tracao_t1). It can rotate with the z axis fixed, it has an upper limit of 3.14 (360 degrees) and lower limit of -3.14 (-360 degrees) -->
-  <joint name="joint_garra_tracao_t1" type="revolute">
-    <parent link="tracao_t"/>
-    <child link="garra_tracao_t1"/>
+  <!-- This joint binds the front traction body unit (represented by the link tracao_f) and the back t1 claw unit (represented by the link garra_tracao_b1). It can rotate with the z axis fixed, it has an upper limit of 3.14 (360 degrees) and lower limit of -3.14 (-360 degrees) -->
+  <joint name="joint_garra_tracao_b1" type="revolute">
+    <parent link="tracao_b"/>
+    <child link="garra_tracao_b1"/>
     <origin rpy="0 0 0" xyz="0.0005 -0.09 0.06985"/>
     <limit effort="1000.0" lower="-3.14" upper="3.14" velocity="0.5"/>
@@ -536,5 +536,5 @@
   </joint>
   <!-- this link represents the back t1 claw unit -->
-  <link name="garra_tracao_t1">
+  <link name="garra_tracao_b1">
     <!-- Need to check mesh design to see if dimensions is the same as the actual dimensions of piro3 -->
     <!-- This visual represents the back t1 claw unit -->
@@ -560,8 +560,8 @@
   </link>
   <!-- Eixo T1 -->
-  <!-- this joint binds the back t1 claw unit (represented by the link garra_tracao_t1) with the back t1 traction unit (represented by the link eixo_tracao_t1). It can move contunuously with the y axis fixed. It moves forward and backward -->
-  <joint name="joint_eixo_tracao_t1" type="continuous">
-    <parent link="garra_tracao_t1"/>
-    <child link="eixo_tracao_t1"/>
+  <!-- this joint binds the back t1 claw unit (represented by the link garra_tracao_b1) with the back t1 traction unit (represented by the link eixo_tracao_b1). It can move contunuously with the y axis fixed. It moves forward and backward -->
+  <joint name="joint_eixo_tracao_b1" type="continuous">
+    <parent link="garra_tracao_b1"/>
+    <child link="eixo_tracao_b1"/>
     <origin rpy="0 0 0" xyz="0.0 0.06 0.172"/>
     <axis xyz="0 1 0"/>
@@ -569,5 +569,5 @@
   </joint>
   <!-- this link represents the back t1 traction unit -->
-  <link name="eixo_tracao_t1">
+  <link name="eixo_tracao_b1">
     <!-- This visual represents the back t1 traction unit -->
     <!-- Need to check mesh design to see if dimensions is the same as the actual dimensions of piro3 -->
@@ -595,8 +595,8 @@
   </link>
   <!-- T2 -->
-  <!-- This joint binds the front traction body unit (represented by the link tracao_f) and the back t2 claw unit (represented by the link garra_tracao_t2). It can rotate with the z axis fixed, it has an upper limit of 3.14 (360 degrees) and lower limit of -3.14 (-360 degrees) -->
-  <joint name="joint_garra_tracao_t2" type="revolute">
-    <parent link="tracao_t"/>
-    <child link="garra_tracao_t2"/>
+  <!-- This joint binds the front traction body unit (represented by the link tracao_f) and the back t2 claw unit (represented by the link garra_tracao_b2). It can rotate with the z axis fixed, it has an upper limit of 3.14 (360 degrees) and lower limit of -3.14 (-360 degrees) -->
+  <joint name="joint_garra_tracao_b2" type="revolute">
+    <parent link="tracao_b"/>
+    <child link="garra_tracao_b2"/>
     <origin rpy="0 0 ${M_PI}" xyz="0.1765 0.09 0.06985"/>
     <limit effort="1000.0" lower="-3.14" upper="3.14" velocity="0.5"/>
@@ -604,5 +604,5 @@
   </joint>
   <!-- this link represents the back t2 claw unit -->
-  <link name="garra_tracao_t2">
+  <link name="garra_tracao_b2">
     <!-- Need to check mesh design to see if dimensions is the same as the actual dimensions of piro3 -->
     <!-- This visual represents the back t2 claw unit -->
@@ -628,8 +628,8 @@
   </link>
   <!-- Eixo F2 -->
-  <!-- this joint binds the back t2 claw unit (represented by the link garra_tracao_t2) with the back t2 traction unit (represented by the link eixo_tracao_t2). It can move contunuously with the y axis fixed. It moves forward and backward -->
-  <joint name="joint_eixo_tracao_t2" type="continuous">
-    <parent link="garra_tracao_t2"/>
-    <child link="eixo_tracao_t2"/>
+  <!-- this joint binds the back t2 claw unit (represented by the link garra_tracao_b2) with the back t2 traction unit (represented by the link eixo_tracao_b2). It can move contunuously with the y axis fixed. It moves forward and backward -->
+  <joint name="joint_eixo_tracao_b2" type="continuous">
+    <parent link="garra_tracao_b2"/>
+    <child link="eixo_tracao_b2"/>
     <origin rpy="0 0 0" xyz="0.0 0.06 0.172"/>
     <axis xyz="0 1 0"/>
@@ -637,5 +637,5 @@
   </joint>
   <!-- this link represents the back t2 traction unit -->
-  <link name="eixo_tracao_t2">
+  <link name="eixo_tracao_b2">
     <!-- This visual represents the back t2 traction unit -->
     <!-- Need to check mesh design to see if dimensions is the same as the actual dimensions of piro3 -->
@@ -829,6 +829,6 @@
 	<link name="cabo_tracao_f1"/>
 	<link name="cabo_tracao_f2"/>
-	<link name="cabo_tracao_t1"/>
-	<link name="cabo_tracao_t2"/>
+	<link name="cabo_tracao_b1"/>
+	<link name="cabo_tracao_b2"/>
 	<joint name="joint_cabo_ap" type="fixed">
 		<parent link="base_link" />
@@ -846,12 +846,12 @@
 		<origin xyz="${x_joint_garra_tracao2} ${y_joint_cabo_tracao} ${z_joint_cabo_tracao + h_tracao/2 + z_tracao}" rpy="0 0 0" />
 	</joint>
-	<joint name="joint_cabo_tracao_t1" type="fixed">
-		<parent link="tracao_t" />
-		<child link="cabo_tracao_t1" />
+	<joint name="joint_cabo_tracao_b1" type="fixed">
+		<parent link="tracao_b" />
+		<child link="cabo_tracao_b1" />
 		<origin xyz="${x_joint_garra_tracao1} ${y_joint_cabo_tracao} ${z_joint_cabo_tracao + h_tracao/2 + z_tracao}" rpy="0 0 0" />
 	</joint>
-	<joint name="joint_cabo_tracao_t2" type="fixed">
-		<parent link="tracao_t" />
-		<child link="cabo_tracao_t2" />
+	<joint name="joint_cabo_tracao_b2" type="fixed">
+		<parent link="tracao_b" />
+		<child link="cabo_tracao_b2" />
 		<origin xyz="${x_joint_garra_tracao2} ${y_joint_cabo_tracao} ${z_joint_cabo_tracao + h_tracao/2 + z_tracao}" rpy="0 0 0" />
 	</joint>-->
@@ -880,5 +880,5 @@
   <transmission name="tran_joint_1t">
     <type>transmission_interface/SimpleTransmission</type>
-    <joint name="joint1_t">
+    <joint name="joint1_b">
       <hardwareInterface>hardware_interface/EffortJointInterface</hardwareInterface>
     </joint>
@@ -890,5 +890,5 @@
   <transmission name="tran_joint_2t">
     <type>transmission_interface/SimpleTransmission</type>
-    <joint name="joint2_t">
+    <joint name="joint2_b">
       <hardwareInterface>hardware_interface/EffortJointInterface</hardwareInterface>
     </joint>
@@ -931,5 +931,5 @@
   <transmission name="tran_claw_t1">
     <type>transmission_interface/SimpleTransmission</type>
-    <joint name="joint_garra_tracao_t1">
+    <joint name="joint_garra_tracao_b1">
       <hardwareInterface>hardware_interface/EffortJointInterface</hardwareInterface>
     </joint>
@@ -941,5 +941,5 @@
   <transmission name="tran_claw_t2">
     <type>transmission_interface/SimpleTransmission</type>
-    <joint name="joint_garra_tracao_t2">
+    <joint name="joint_garra_tracao_b2">
       <hardwareInterface>hardware_interface/EffortJointInterface</hardwareInterface>
     </joint>
@@ -982,5 +982,5 @@
   <transmission name="tran_tracao_1t">
     <type>transmission_interface/SimpleTransmission</type>
-    <joint name="joint_eixo_tracao_t1">
+    <joint name="joint_eixo_tracao_b1">
       <hardwareInterface>hardware_interface/VelocityJointInterface</hardwareInterface>
     </joint>
@@ -992,5 +992,5 @@
   <transmission name="tran_tracao_2t">
     <type>transmission_interface/SimpleTransmission</type>
-    <joint name="joint_eixo_tracao_t2">
+    <joint name="joint_eixo_tracao_b2">
       <hardwareInterface>hardware_interface/VelocityJointInterface</hardwareInterface>
     </joint>

Commit message: Add M_PI define to piro.gazebo
The moveit setup assistant needs the M_PI definition in the .gazebo file

File: mybot_description/urdf/piro.gazebo.xacro (robot description, xacro)
@@ -3,4 +3,5 @@
 xmlns:controller="http://playerstage.sourceforge.net/gazebo/xmlschema/#controller"
 xmlns:interface="http://playerstage.sourceforge.net/gazebo/xmlschema/#interface">
+<xacro:property name="M_PI" value="3.141592" />
   <gazebo>
     <plugin filename="libgazebo_ros_control.so" name="gazebo_ros_control">
