Commit message: Add the piro_view launch file mybot_descrpition, in order to visualize piro in the Rviz; Add the stereo camera to simulation; Change up sonar location; Delete beginner_tutorials package; Fix simulation bug, the robot was starting the simulation falling from the line;

File: mybot_description/urdf/piro.urdf.xacro (robot description, xacro)
@@ -7,4 +7,5 @@
   <xacro:include filename="$(find mybot_description)/urdf/materials.xacro" />
   <xacro:include filename="$(find mybot_description)/urdf/piro.gazebo" />
+  <xacro:property name="PI" value="3.141592" />
   <!-- BASE LINK-->
   <!-- Dimensoes da unidade de apoio -->
@@ -24,5 +25,5 @@
     <visual name = 'base_body'>
       <geometry>
-        <box size="0.3219 0.1461 0.2357"/>
+        <box size= "0.3219 0.1461 0.2357"/>
       </geometry>
       <material name="grey"/>
@@ -34,4 +35,5 @@
       </geometry>
       <material name="grey"/>
+      <!-- <xacro:insert_block name="a.test_central_stem_origin" /> -->
       <origin rpy="0 0 0" xyz="0 0.0303 0.23365"/>
     </visual>
@@ -614,24 +616,26 @@
   <!-- Posicoes dos frames virtuais -->
   <!-- Apoio -->
-  <link name="laser">
-    <visual>
-      <geometry>
-        <mesh filename="package://mybot_description/meshes/hokuyo.dae"/>
-      </geometry>
-    </visual>
-    <collision>
-      <geometry>
-        <mesh filename="package://mybot_description/meshes/hokuyo.dae"/>
+  <!-- Camera -->
+  <link name="stereo_camera_link">
+    <visual>
+      <geometry>
+        <box size="0.03 0.175 0.033"/>
+        <material>Gazebo/Orange</material>
+      </geometry>
+    </visual>
+    <collision>
+      <geometry>
+          <box size="0.03 0.175 0.033"/>
       </geometry>
     </collision>
     <inertial>
       <mass value="0.001"/>
-      <inertia ixx="4.94e-05" ixy="0.0" ixz="0.0" iyy="6.11e-05" iyz="0.0" izz="4.94e-05"/>
-    </inertial>
-  </link>
-  <joint name="hokuyo_base" type="fixed">
-    <parent link="tracao_f"/>
-    <child link="laser"/>
-    <origin rpy="0 3.661592 3.141592" xyz="0.233 0.0 -0.1"/>
+      <inertia ixx="1e-6" ixy="0" ixz="0" iyy="1e-6" iyz="0" izz="1e-6"/>
+    </inertial>
+  </link>
+  <joint name="stereo_camera_joint" type="fixed">
+    <parent link="base_link"/>
+    <child link="stereo_camera_link"/>
+    <origin rpy="0 3.61592 0" xyz="-0.17 0.0 -0.05"/>
   </joint>
   <!-- Sonares -->
@@ -657,5 +661,5 @@
     <parent link="tracao_f"/>
     <child link="obstacle_sonar_down"/>
-    <origin rpy="0 0 0" xyz="0.205 0.0 0.0569"/>
+    <origin rpy="0 0 0" xyz="0.24 0.0 0.0569"/>
   </joint>
   <link name="obstacle_sonar_up">

Commit message: Add zed cameras

File: mybot_description/urdf/piro.urdf.xacro (robot description, xacro)
@@ -7,5 +7,5 @@
   <xacro:include filename="$(find mybot_description)/urdf/materials.xacro" />
   <xacro:include filename="$(find mybot_description)/urdf/piro.gazebo" />
-  <xacro:property name="PI" value="3.141592" />
+  <xacro:property name="M_PI" value="3.141592" />
   <!-- BASE LINK-->
   <!-- Dimensoes da unidade de apoio -->
@@ -78,5 +78,5 @@
     <parent link="base_link"/>
     <child link="garra_ap"/>
-    <origin rpy="0 0 3.141592" xyz="0.0 0.0722 0.3554"/>
+    <origin rpy="0 0 ${M_PI}" xyz="0.0 0.0722 0.3554"/>
     <limit effort="1000.0" lower="-3.14" upper="3.14" velocity="0.5"/>
     <axis xyz="0 0 1"/>
@@ -140,5 +140,5 @@
     <child link="link1_f"/>
     <!-- <origin rpy=" 0 -0.60 3.141592" xyz="-0.13 0.0 0.079"/> -->
-    <origin rpy=" 0 -0.6 3.141592" xyz="-0.13 0.0 0.079"/>
+    <origin rpy=" 0 -0.6 ${M_PI}" xyz="-0.13 0.0 0.079"/>
     <limit effort="1000.0" lower="-1.74" upper="0.7" velocity="0.5"/>
     <axis xyz="0 1 0"/>
@@ -247,5 +247,5 @@
       </geometry>
       <material name="grey"/>
-      <origin rpy="0 0 3.141592" xyz="0.1765 -0.075 0.0521"/>
+      <origin rpy="0 0 ${M_PI}" xyz="0.1765 -0.075 0.0521"/>
     </visual>
     <!-- this collision is for the front traction body -->
@@ -268,5 +268,5 @@
         <mesh filename="package://mybot_description/meshes/dxl_mx106.dae"/>
       </geometry>
-      <origin rpy="0 0 3.141592" xyz="0.1765 -0.075 0.0521"/>
+      <origin rpy="0 0 ${M_PI}" xyz="0.1765 -0.075 0.0521"/>
     </collision>
     <inertial>
@@ -308,5 +308,5 @@
       </geometry>
       <material name="grey"/>
-      <origin rpy="0 0 3.141592" xyz="0.1765 0.075 0.0521"/>
+      <origin rpy="0 0 ${M_PI}" xyz="0.1765 0.075 0.0521"/>
     </visual>
     <!-- this collision is for the back traction body -->
@@ -329,5 +329,5 @@
         <mesh filename="package://mybot_description/meshes/dxl_mx106.dae"/>
       </geometry>
-      <origin rpy="0 0 3.141592" xyz="0.1765 0.075 0.0521"/>
+      <origin rpy="0 0 ${M_PI}" xyz="0.1765 0.075 0.0521"/>
     </collision>
     <inertial>
@@ -341,5 +341,5 @@
     <parent link="tracao_f"/>
     <child link="garra_tracao_f1"/>
-    <origin rpy="0 0 3.141592" xyz="0.0005 0.09 0.06985"/>
+    <origin rpy="0 0 ${M_PI}" xyz="0.0005 0.09 0.06985"/>
     <limit effort="1000.0" lower="-3.14" upper="3.14" velocity="0.5"/>
     <axis xyz="0 0 1"/>
@@ -543,5 +543,5 @@
     <parent link="tracao_t"/>
     <child link="garra_tracao_t2"/>
-    <origin rpy="0 0 3.141592" xyz="0.1765 0.09 0.06985"/>
+    <origin rpy="0 0 ${M_PI}" xyz="0.1765 0.09 0.06985"/>
     <limit effort="1000.0" lower="-3.14" upper="3.14" velocity="0.5"/>
     <axis xyz="0 0 1"/>
@@ -617,5 +617,5 @@
   <!-- Apoio -->
   <!-- Camera -->
-  <link name="stereo_camera_link">
+  <!--link name="stereo_camera_link">
     <visual>
       <geometry>
@@ -633,9 +633,58 @@
       <inertia ixx="1e-6" ixy="0" ixz="0" iyy="1e-6" iyz="0" izz="1e-6"/>
     </inertial>
-  </link>
-  <joint name="stereo_camera_joint" type="fixed">
+  </link-->
+  <link name="zed_left_camera">
+        <visual>
+            <origin xyz="0 0 0" rpy="0 1.57 0"/>
+            <geometry>
+                <cylinder radius="0.007" length=".031"/>
+            </geometry>
+            <material name="dark_grey">
+                <color rgba="0.1 0.1 0.1 1"/>
+            </material>
+        </visual>
+    </link>
+    <link name="zed_center">
+        <visual>
+            <origin xyz="0 0 0" rpy="0 0 0"/>
+            <geometry>
+                <mesh filename="package://mybot_description/urdf/ZED.stl" />
+            </geometry>
+            <material name="light_grey">
+                <color rgba="0.8 0.8 0.8 0.8"/>
+            </material>
+        </visual>
+    </link>
+  <link name="zed_right_camera">
+        <visual>
+            <origin xyz="0 0 0" rpy="0 1.57 0"/>
+            <geometry>
+                <cylinder radius="0.007" length=".031"/>
+            </geometry>
+            <material name="dark_grey">
+                <color rgba="0.1 0.1 0.1 1"/>
+            </material>
+        </visual>
+    </link>
+    <link name="zed_depth_camera" />
+    <joint name="zed_left_camera_joint" type="fixed">
+        <parent link="zed_center"/>
+        <child link="zed_left_camera"/>
+        <origin xyz="0 0.06 0" rpy="0 0 0" />
+    </joint>
+    <joint name="zed_depth_camera_joint" type="fixed">
+        <parent link="zed_left_camera"/>
+        <child link="zed_depth_camera"/>
+        <origin xyz="0 0 0" rpy="-1.5707963267948966 0 -1.5707963267948966" />
+    </joint>
+    <joint name="zed_right_camera_joint" type="fixed">
+        <parent link="zed_center"/>
+        <child link="zed_right_camera"/>
+        <origin xyz="0 -0.06 0" rpy="0 0 0" />
+    </joint>
+  <joint name="zed_camera_joint" type="fixed">
     <parent link="base_link"/>
-    <child link="stereo_camera_link"/>
-    <origin rpy="0 3.61592 0" xyz="-0.17 0.0 -0.05"/>
+    <child link="zed_center"/>
+    <origin rpy="0 0 ${M_PI}" xyz="-0.17 0.0 -0.05"/>
   </joint>
   <!-- Sonares -->

Commit message: Add ZED and Flir Camera, and add Zed right and left camera simulation

File: mybot_description/urdf/piro.urdf.xacro (robot description, xacro)
@@ -649,5 +649,5 @@
             <origin xyz="0 0 0" rpy="0 0 0"/>
             <geometry>
-                <mesh filename="package://mybot_description/urdf/ZED.stl" />
+                <mesh filename="package://mybot_description/meshes/ZED.stl" />
             </geometry>
             <material name="light_grey">
@@ -683,4 +683,15 @@
         <origin xyz="0 -0.06 0" rpy="0 0 0" />
     </joint>
+    <link name="flir_camera">
+        <visual>
+            <origin xyz="0 0 0" rpy="0 0 0"/>
+            <geometry>
+                <mesh filename="package://mybot_description/meshes/LeptonBreakoutBoardWithLepton3.stl" scale="0.001 0.001 0.001"/>
+            </geometry>
+            <material name="light_grey">
+                <color rgba="0.8 0.8 0.8 0.8"/>
+            </material>
+        </visual>
+    </link>
   <joint name="zed_camera_joint" type="fixed">
     <parent link="base_link"/>
@@ -688,28 +699,10 @@
     <origin rpy="0 0 ${M_PI}" xyz="-0.17 0.0 -0.05"/>
   </joint>
+  <joint name="flir_camera_joint" type="fixed">
+    <parent link="base_link"/>
+    <child link="flir_camera"/>
+    <origin rpy="0 ${-M_PI/2} 0" xyz="-0.17 0.0 0.00"/>
+  </joint>
   <!-- Sonares -->
-  <link name="obstacle_sonar_down">
-    <visual>
-      <geometry>
-        <mesh filename="package://mybot_description/meshes/maxsonar.dae"/>
-      </geometry>
-      <material name="grey"/>
-    </visual>
-    <collision>
-      <geometry>
-        <mesh filename="package://mybot_description/meshes/maxsonar.dae"/>
-      </geometry>
-    </collision>
-    <inertial>
-      <mass value="1e-5"/>
-      <origin rpy="0 0 0" xyz="0 0 0"/>
-      <inertia ixx="1e-6" ixy="0" ixz="0" iyy="1e-6" iyz="0" izz="1e-6"/>
-    </inertial>
-  </link>
-  <joint name="obstacle_sonar_down_base" type="fixed">
-    <parent link="tracao_f"/>
-    <child link="obstacle_sonar_down"/>
-    <origin rpy="0 0 0" xyz="0.24 0.0 0.0569"/>
-  </joint>
   <link name="obstacle_sonar_up">
     <visual>

Commit message: Change front arm visual and collision to adept to the real model

File: mybot_description/urdf/piro.urdf.xacro (robot description, xacro)
@@ -156,13 +156,41 @@
     <visual name = 'front_arm'>
       <geometry>
-        <box size="0.4199 0.05 0.100"/>
+        <box size="0.19 0.100 0.05"/>
       </geometry>
       <material name="grey"/>
       <origin rpy="0 0 0" xyz="0.20995 0.0 0.0"/>
+    </visual>
+    <visual name = 'base_left_pallet'>
+      <geometry>
+        <mesh filename="package://mybot_description/meshes/PIR-M01-003-0_HolderWingWide.STL" scale="0.001 0.001 0.001"/>
+      </geometry>
+      <material name="grey"/>
+      <origin rpy="${M_PI/2} 0 0" xyz="0 0.085 ${-0.05/2}"/>
+    </visual>
+    <visual name = 'base_right_pallet'>
+      <geometry>
+        <mesh filename="package://mybot_description/meshes/PIR-M01-003-0_HolderWingWide.STL" scale="0.001 0.001 0.001"/>
+      </geometry>
+      <material name="grey"/>
+      <origin rpy="-${M_PI/2} 0 0" xyz="0 -0.085 ${0.05/2}"/>
+    </visual>
+    <visual name = 'traction_left_pallet'>
+      <geometry>
+        <mesh filename="package://mybot_description/meshes/PIR-M01-002-0_HolderWing.STL" scale="0.001 0.001 0.001"/>
+      </geometry>
+      <material name="grey"/>
+      <origin rpy="${M_PI/2} -${M_PI} 0" xyz="${0.20995*2} 0.06 ${0.05/2}"/>
+    </visual>]
+    <visual name = 'traction_right_pallet'>
+      <geometry>
+        <mesh filename="package://mybot_description/meshes/PIR-M01-002-0_HolderWing.STL" scale="0.001 0.001 0.001"/>
+      </geometry>
+      <material name="grey"/>
+      <origin rpy="-${M_PI/2} -${M_PI} 0" xyz="${0.20995*2} -0.06 -${0.05/2}"/>
     </visual>
     <!-- this collision is for the front arm unit -->
     <collision name = 'front_arm'>
       <geometry>
-        <box size="0.4199 0.05 0.100"/>
+        <box size="0.19 0.100 0.05"/>
       </geometry>
       <origin rpy="0 0 0" xyz="0.20995 0.0 0.0"/>

Commit message: Change visual and colision of back arm

File: mybot_description/urdf/piro.urdf.xacro (robot description, xacro)
@@ -44,5 +44,5 @@
         <mesh filename="package://mybot_description/meshes/dxl_mx106.dae"/>
       </geometry>
-      <material name="grey"/>
+      <material name="black"/>
       <origin rpy="0 0 0" xyz="0.0 0.0722 0.3554"/>
     </visual>
@@ -165,5 +165,5 @@
         <mesh filename="package://mybot_description/meshes/PIR-M01-003-0_HolderWingWide.STL" scale="0.001 0.001 0.001"/>
       </geometry>
-      <material name="grey"/>
+      <material name="black"/>
       <origin rpy="${M_PI/2} 0 0" xyz="0 0.085 ${-0.05/2}"/>
     </visual>
@@ -172,5 +172,5 @@
         <mesh filename="package://mybot_description/meshes/PIR-M01-003-0_HolderWingWide.STL" scale="0.001 0.001 0.001"/>
       </geometry>
-      <material name="grey"/>
+      <material name="black"/>
       <origin rpy="-${M_PI/2} 0 0" xyz="0 -0.085 ${0.05/2}"/>
     </visual>
@@ -179,12 +179,12 @@
         <mesh filename="package://mybot_description/meshes/PIR-M01-002-0_HolderWing.STL" scale="0.001 0.001 0.001"/>
       </geometry>
-      <material name="grey"/>
+      <material name="black"/>
       <origin rpy="${M_PI/2} -${M_PI} 0" xyz="${0.20995*2} 0.06 ${0.05/2}"/>
-    </visual>]
+    </visual>
     <visual name = 'traction_right_pallet'>
       <geometry>
         <mesh filename="package://mybot_description/meshes/PIR-M01-002-0_HolderWing.STL" scale="0.001 0.001 0.001"/>
       </geometry>
-      <material name="grey"/>
+      <material name="black"/>
       <origin rpy="-${M_PI/2} -${M_PI} 0" xyz="${0.20995*2} -0.06 -${0.05/2}"/>
     </visual>
@@ -223,5 +223,5 @@
     <visual name = 'back_arm'>
       <geometry>
-        <box size="0.4199 0.05 0.100"/>
+        <box size="0.19 0.100 0.05"/>
       </geometry>
       <material name="grey"/>
@@ -229,7 +229,35 @@
     </visual>
     <!-- this collision is for the back arm unit -->
+    <visual name = 'base_left_pallet'>
+      <geometry>
+        <mesh filename="package://mybot_description/meshes/PIR-M01-003-0_HolderWingWide.STL" scale="0.001 0.001 0.001"/>
+      </geometry>
+      <material name="black"/>
+      <origin rpy="${M_PI/2} 0 0" xyz="0 0.085 ${-0.05/2}"/>
+    </visual>
+    <visual name = 'base_right_pallet'>
+      <geometry>
+        <mesh filename="package://mybot_description/meshes/PIR-M01-003-0_HolderWingWide.STL" scale="0.001 0.001 0.001"/>
+      </geometry>
+      <material name="black"/>
+      <origin rpy="-${M_PI/2} 0 0" xyz="0 -0.085 ${0.05/2}"/>
+    </visual>
+    <visual name = 'traction_left_pallet'>
+      <geometry>
+        <mesh filename="package://mybot_description/meshes/PIR-M01-002-0_HolderWing.STL" scale="0.001 0.001 0.001"/>
+      </geometry>
+      <material name="black"/>
+      <origin rpy="${M_PI/2} -${M_PI} 0" xyz="${0.20995*2} 0.06 ${0.05/2}"/>
+    </visual>]
+    <visual name = 'traction_right_pallet'>
+      <geometry>
+        <mesh filename="package://mybot_description/meshes/PIR-M01-002-0_HolderWing.STL" scale="0.001 0.001 0.001"/>
+      </geometry>
+      <material name="black"/>
+      <origin rpy="-${M_PI/2} -${M_PI} 0" xyz="${0.20995*2} -0.06 -${0.05/2}"/>
+    </visual>
     <collision name = 'back_arm'>
       <geometry>
-        <box size="0.4199 0.05 0.100"/>
+        <box size="0.19 0.100 0.05"/>
       </geometry>
       <origin rpy="0 0 0" xyz="0.20995 0.0 0.0"/>
@@ -265,5 +293,5 @@
         <mesh filename="package://mybot_description/meshes/dxl_mx106.dae"/>
       </geometry>
-      <material name="grey"/>
+      <material name="black"/>
       <origin rpy="0 0 0" xyz="0.0005 0.075 0.0521"/>
     </visual>
@@ -274,5 +302,5 @@
         <mesh filename="package://mybot_description/meshes/dxl_mx106.dae"/>
       </geometry>
-      <material name="grey"/>
+      <material name="black"/>
       <origin rpy="0 0 ${M_PI}" xyz="0.1765 -0.075 0.0521"/>
     </visual>
@@ -327,5 +355,5 @@
         <mesh filename="package://mybot_description/meshes/dxl_mx106.dae"/>
       </geometry>
-      <material name="grey"/>
+      <material name="black"/>
       <origin rpy="0 0 0" xyz="0.0005 -0.075 0.0521"/>
     </visual>
@@ -335,5 +363,5 @@
         <mesh filename="package://mybot_description/meshes/dxl_mx106.dae"/>
       </geometry>
-      <material name="grey"/>
+      <material name="black"/>
       <origin rpy="0 0 ${M_PI}" xyz="0.1765 0.075 0.0521"/>
     </visual>

Commit message: Add the instal dependencies script

File: mybot_description/urdf/piro.urdf.xacro (robot description, xacro)
@@ -202,7 +202,4 @@
     </inertial>
   </link>
-  <gazebo reference="traction_left_pallet">
-    <material>Gazebo/Black</material>
-  </gazebo>
   <!-- This joint binds the base body (represented by the link base_link) and the back arm unit (represented by the link link1_t). it can rotate with the y axis fixed, it has an upper limit of 0.7 (40 degrees) and a lower limit of -1.74 (-100 degrees) -->
   <joint name="joint1_t" type="revolute">
@@ -819,5 +816,5 @@
 	</link>
   <gazebo reference="ground_sonar">
-    <material>Gazebo/Blue</material>
+    <material>Gazebo/Gold</material>
   </gazebo>
 	<joint name="ground_sonar_base" type="fixed">

Commit message: Remove  obstacle_sonar_up

File: mybot_description/urdf/piro.urdf.xacro (robot description, xacro)
@@ -761,40 +761,4 @@
   </joint>
   <!-- Sonares -->
-  <link name="obstacle_sonar_up">
-    <visual>
-      <geometry>
-        <mesh filename="package://mybot_description/meshes/maxsonar.dae"/>
-      </geometry>
-      <material name="grey"/>
-    </visual>
-    <collision>
-      <geometry>
-        <mesh filename="package://mybot_description/meshes/maxsonar.dae"/>
-      </geometry>
-    </collision>
-    <inertial>
-      <mass value="1e-5"/>
-      <origin rpy="0 0 0" xyz="0 0 0"/>
-      <inertia ixx="1e-6" ixy="0" ixz="0" iyy="1e-6" iyz="0" izz="1e-6"/>
-    </inertial>
-    <visual>
-      <geometry>
-        <box size="0.005 0.07 0.0221"/>
-      </geometry>
-      <material name="grey"/>
-      <origin rpy="0 0 0" xyz="-0.0025 -0.02395 0.0"/>
-    </visual>
-    <collision>
-      <geometry>
-        <box size="0.005 0.07 0.0221"/>
-      </geometry>
-      <origin rpy="0 0 0" xyz="-0.0025 -0.02395 0.0"/>
-    </collision>
-  </link>
-  <joint name="obstacle_sonar_up_base" type="fixed">
-    <parent link="garra_tracao_f2"/>
-    <child link="obstacle_sonar_up"/>
-    <origin rpy="0 0 0" xyz="0.024 0.075 0.19615"/>
-  </joint>
 <link name="ground_sonar" >
 		<visual>

Commit message: Create a new base_link and rename the base_link to box_link

File: mybot_description/urdf/piro.urdf.xacro (robot description, xacro)
@@ -19,7 +19,22 @@
   <!-- Dimensoes do sup_apoio -->
   <!-- Posicoes da base do sup_apoio para o centro do base link -->
-  <!-- Parametros do base_link-->
+  <!-- Parametros do box_link-->
+<link name="base_link">
+    <!-- This visual represents the base body-->
+    <visual name = 'base_body'>
+      <geometry>
+        <box size= "0.3219 0.1461 0.2357"/>
+      </geometry>
+  </visual>
+  </link>
+  <joint name="base_joint" type="fixed">
+    <origin xyz="0.0 0.0 0.0" rpy="0.0 0.0 0.0"/>
+    <parent link="base_link"/>
+    <child link="box_link"/>
+    <axis xyz="0.0 0.0 0.0"/>
+    <limit lower="0.0" upper="0.0" effort="0.0" velocity="0.0"/>
+  </joint>>
   <!-- This link represents the base_body, the central stem and the central's claw base -->
-  <link name="base_link">
+  <link name="box_link">
     <!-- This visual represents the base body-->
     <visual name = 'base_body'>
@@ -74,7 +89,7 @@
     </inertial>
   </link>
-  <!-- this joint binds the base body (represented by the link base_link) with the central claw unit (represented by the link garra_ap). It can rotate with the z axis fixed, it has an upper limit of 3,14 (180 degrees) and a lower limit of -3,14 (-180 degrees) -->
+  <!-- this joint binds the base body (represented by the link box_link) with the central claw unit (represented by the link garra_ap). It can rotate with the z axis fixed, it has an upper limit of 3,14 (180 degrees) and a lower limit of -3,14 (-180 degrees) -->
   <joint name="joint_garra_ap" type="revolute">
-    <parent link="base_link"/>
+    <parent link="box_link"/>
     <child link="garra_ap"/>
     <origin rpy="0 0 ${M_PI}" xyz="0.0 0.0722 0.3554"/>
@@ -135,7 +150,7 @@
     </inertial>
   </link>
-  <!-- This joint binds the base body (represented by the link base_link) and the front arm unit (represented by the link link1_f). it can rotate with the y axis fixed, it has an upper limit of 0.7 (40 degrees) and a lower limit of -1.74 (-100 degrees) -->
+  <!-- This joint binds the base body (represented by the link box_link) and the front arm unit (represented by the link link1_f). it can rotate with the y axis fixed, it has an upper limit of 0.7 (40 degrees) and a lower limit of -1.74 (-100 degrees) -->
   <joint name="joint1_b" type="revolute">
-    <parent link="base_link"/>
+    <parent link="box_link"/>
     <child link="link1_b"/>
     <!-- <origin rpy=" 0 -0.60 3.141592" xyz="-0.13 0.0 0.079"/> -->
@@ -202,7 +217,7 @@
     </inertial>
   </link>
-  <!-- This joint binds the base body (represented by the link base_link) and the back arm unit (represented by the link link1_t). it can rotate with the y axis fixed, it has an upper limit of 0.7 (40 degrees) and a lower limit of -1.74 (-100 degrees) -->
+  <!-- This joint binds the base body (represented by the link box_link) and the back arm unit (represented by the link link1_t). it can rotate with the y axis fixed, it has an upper limit of 0.7 (40 degrees) and a lower limit of -1.74 (-100 degrees) -->
   <joint name="joint1_f" type="revolute">
-    <parent link="base_link"/>
+    <parent link="box_link"/>
     <child link="link1_f"/>
     <!-- <origin rpy="0 -0.60 0" xyz="0.13 0.0 0.079"/> -->
@@ -669,5 +684,5 @@
   <!-- Dimensoes do suporte do sonar alto -->
   <!-- Posicao do suporte do sonar alto -->
-  <!-- Posicao do sonar de chao (em relacao ao base_link)-->
+  <!-- Posicao do sonar de chao (em relacao ao box_link)-->
   <!-- Posicoes dos frames virtuais -->
   <!-- Apoio -->
@@ -751,10 +766,10 @@
     </link>
   <joint name="zed_camera_joint" type="fixed">
-    <parent link="base_link"/>
+    <parent link="box_link"/>
     <child link="zed_center"/>
     <origin rpy="0 0 0" xyz="0.17 0.0 -0.1"/>
   </joint>
   <joint name="flir_camera_joint" type="fixed">
-    <parent link="base_link"/>
+    <parent link="box_link"/>
     <child link="flir_camera"/>
     <origin rpy="0 0 0" xyz="0.17 0.0 -0.05"/>
@@ -783,5 +798,5 @@
   </gazebo>
 	<joint name="ground_sonar_base" type="fixed">
-		<parent link="base_link" />
+		<parent link="box_link" />
 		<child link="ground_sonar" />
 		<origin xyz="0 0 -0.155" rpy="0 ${M_PI/2} 0" />
@@ -796,5 +811,5 @@
 	<link name="cabo_tracao_b2"/>
 	<joint name="joint_cabo_ap" type="fixed">
-		<parent link="base_link" />
+		<parent link="box_link" />
 		<child link="cabo_ap" />
 		<origin xyz="${x_joint_cabo_ap} ${y_joint_cabo_ap} ${z_joint_cabo_ap + h_ap/2}" rpy="0 0 0" />
