Commit message: Remove unecessary comments

File: mybot_description/urdf/piro.urdf.xacro (robot description, xacro)
@@ -8,18 +8,7 @@
   <xacro:include filename="$(find mybot_description)/urdf/piro.gazebo.xacro" />
   <xacro:property name="M_PI" value="3.141592" />
-  <!-- BASE LINK-->
-  <!-- Dimensoes da unidade de apoio -->
-  <!-- Dimensoes da caixa eletronica -->
-  <!--
-	<xacro:property name="l_eletr_ap" value="0.240" />
-	<xacro:property name="h_eletr_ap" value="0.120" />
-	<xacro:property name="w_eletr_ap" value="0.120" />
-  -->
-  <!-- Suporte da garra da unidade de apoio -->
-  <!-- Dimensoes do sup_apoio -->
-  <!-- Posicoes da base do sup_apoio para o centro do base link -->
   <!-- Parametros do box_link-->
-<link name="base_link">
-    <!-- This visual represents the base body-->
+  <link name="base_link">
+    <!-- This visual represents the dummy link for robot base body-->
     <visual name = 'base_body'>
       <geometry>
@@ -34,6 +23,6 @@
     <axis xyz="0.0 0.0 0.0"/>
     <limit lower="0.0" upper="0.0" effort="0.0" velocity="0.0"/>
-  </joint>>
-  <!-- This link represents the base_body, the central stem and the central's claw base -->
+  </joint>
+  <!-- This link represents the base body of the robot, the central stem and the central's claw base -->
   <link name="box_link">
     <!-- This visual represents the base body-->
@@ -677,32 +666,4 @@
     </inertial>
   </link>
-  <!-- SENSORES -->
-  <!-- Hokuyo -->
-  <!-- Posicao do Hokuyo (em relacao a junta 3)-->
-  <!-- Posicao do sonar baixo (em relacao a junta 3)-->
-  <!-- Posicao do sonar alto (em relacao a garra)-->
-  <!-- Dimensoes do suporte do sonar alto -->
-  <!-- Posicao do suporte do sonar alto -->
-  <!-- Posicao do sonar de chao (em relacao ao box_link)-->
-  <!-- Posicoes dos frames virtuais -->
-  <!-- Apoio -->
-  <!-- Camera -->
-  <!--link name="stereo_camera_link">
-    <visual>
-      <geometry>
-        <box size="0.03 0.175 0.033"/>
-        <material>Gazebo/Orange</material>
-      </geometry>
-    </visual>
-    <collision>
-      <geometry>
-          <box size="0.03 0.175 0.033"/>
-      </geometry>
-    </collision>
-    <inertial>
-      <mass value="0.001"/>
-      <inertia ixx="1e-6" ixy="0" ixz="0" iyy="1e-6" iyz="0" izz="1e-6"/>
-    </inertial>
-  </link-->
   <link name="zed_left_camera">
         <visual>
@@ -802,37 +763,4 @@
 		<origin xyz="0 0 -0.155" rpy="0 ${M_PI/2} 0" />
 	</joint>
-  <!-- FRAMES VIRTUAIS NO CABO -->
-  <!-- Tracao -->
-  <!--
-	<link name="cabo_ap"/>
-	<link name="cabo_tracao_f1"/>
-	<link name="cabo_tracao_f2"/>
-	<link name="cabo_tracao_b1"/>
-	<link name="cabo_tracao_b2"/>
-	<joint name="joint_cabo_ap" type="fixed">
-		<parent link="box_link" />
-		<child link="cabo_ap" />
-		<origin xyz="${x_joint_cabo_ap} ${y_joint_cabo_ap} ${z_joint_cabo_ap + h_ap/2}" rpy="0 0 0" />
-	</joint>
-	<joint name="joint_cabo_tracao_f1" type="fixed">
-		<parent link="tracao_f" />
-		<child link="cabo_tracao_f1" />
-		<origin xyz="${x_joint_garra_tracao1} ${y_joint_cabo_tracao} ${z_joint_cabo_tracao + h_tracao/2 + z_tracao}" rpy="0 0 0" />
-	</joint>
-	<joint name="joint_cabo_tracao_f2" type="fixed">
-		<parent link="tracao_f" />
-		<child link="cabo_tracao_f2" />
-		<origin xyz="${x_joint_garra_tracao2} ${y_joint_cabo_tracao} ${z_joint_cabo_tracao + h_tracao/2 + z_tracao}" rpy="0 0 0" />
-	</joint>
-	<joint name="joint_cabo_tracao_b1" type="fixed">
-		<parent link="tracao_b" />
-		<child link="cabo_tracao_b1" />
-		<origin xyz="${x_joint_garra_tracao1} ${y_joint_cabo_tracao} ${z_joint_cabo_tracao + h_tracao/2 + z_tracao}" rpy="0 0 0" />
-	</joint>
-	<joint name="joint_cabo_tracao_b2" type="fixed">
-		<parent link="tracao_b" />
-		<child link="cabo_tracao_b2" />
-		<origin xyz="${x_joint_garra_tracao2} ${y_joint_cabo_tracao} ${z_joint_cabo_tracao + h_tracao/2 + z_tracao}" rpy="0 0 0" />
-	</joint>-->
   <!-- ROS Control-->
   <!-- Juntas -->

Commit message: Modify the claw supports and location to aproximate the real model

File: mybot_description/urdf/piro.urdf.xacro (robot description, xacro)
@@ -122,14 +122,14 @@
     <visual name = 'central_traction'>
       <geometry>
-        <mesh filename="package://mybot_description/meshes/Shaft_piro3_V2.dae"/>
-      </geometry>
-      <origin rpy="1.57 0 0" xyz="0.0 0.05 0.0"/>
+         <mesh filename="package://mybot_description/meshes/wheel_elir.STL" scale="0.001 0.001 0.001"/>
+      </geometry>
+      <origin rpy="0 0 0" xyz="0.0 0.0 0.0"/>
     </visual>
     <!-- This collision is for the central traction unit -->
     <collision name = 'central_traction'>
       <geometry>
-        <mesh filename="package://mybot_description/meshes/Shaft_piro3_V2.dae"/>
-      </geometry>
-      <origin rpy="1.57 0 0" xyz="0.0 0.05 0.0"/>
+         <mesh filename="package://mybot_description/meshes/wheel_elir.STL" scale="0.001 0.001 0.001"/>
+      </geometry>
+      <origin rpy="0 0 0" xyz="0.0 0.0 0.0"/>
     </collision>
     <inertial>
@@ -293,19 +293,19 @@
     <!-- This visual represents the front traction claw f2 support -->
     <!-- Need to check mesh design to see if dimensions is the same as the actual dimensions of piro3 -->
+    <visual name = 'front_traction_claw_f1_support'>
+      <geometry>
+        <box size="0.051 0.045 0.036 "/>
+      </geometry>
+      <material name="black"/>
+      <origin rpy="0 0 0" xyz="${0.006 +0.051/2} ${0.05+0.045/2} ${0.05}"/>
+    </visual>
+    <!-- This visual represents the front traction claw f1 support -->
+    <!-- Need to check mesh design to see if dimensions is the same as the actual dimensions of piro3 -->
     <visual name = 'front_traction_claw_f2_support'>
       <geometry>
-        <mesh filename="package://mybot_description/meshes/dxl_mx106.dae"/>
-      </geometry>
-      <material name="black"/>
-      <origin rpy="0 0 0" xyz="0.0005 0.075 0.0521"/>
-    </visual>
-    <!-- This visual represents the front traction claw f1 support -->
-    <!-- Need to check mesh design to see if dimensions is the same as the actual dimensions of piro3 -->
-    <visual name = 'front_traction_claw_f1_support'>
-      <geometry>
-        <mesh filename="package://mybot_description/meshes/dxl_mx106.dae"/>
-      </geometry>
-      <material name="black"/>
-      <origin rpy="0 0 ${M_PI}" xyz="0.1765 -0.075 0.0521"/>
+        <box size="0.051 0.045 0.036 "/>
+      </geometry>
+      <material name="black"/>
+      <origin rpy="0 0 0" xyz="${0.233 -0.006 -0.051/2} ${-0.05-0.045/2} ${0.05}"/>
     </visual>
     <!-- this collision is for the front traction body -->
@@ -319,5 +319,5 @@
     <collision name = 'front_traction_claw_f2_support'>
       <geometry>
-        <mesh filename="package://mybot_description/meshes/dxl_mx106.dae"/>
+        <box size="0.051 0.045 0.036 "/>
       </geometry>
       <origin rpy="0 0 0" xyz="0.0005 0.075 0.0521"/>
@@ -326,5 +326,5 @@
     <collision name = 'front_traction_claw_f1_support'>
       <geometry>
-        <mesh filename="package://mybot_description/meshes/dxl_mx106.dae"/>
+        <box size="0.051 0.045 0.036 "/>
       </geometry>
       <origin rpy="0 0 ${M_PI}" xyz="0.1765 -0.075 0.0521"/>
@@ -357,16 +357,16 @@
     <visual name = 'back_traction_claw_f1_support'>
       <geometry>
-        <mesh filename="package://mybot_description/meshes/dxl_mx106.dae"/>
-      </geometry>
-      <material name="black"/>
-      <origin rpy="0 0 0" xyz="0.0005 -0.075 0.0521"/>
+        <box size="0.051 0.045 0.036 "/>
+      </geometry>
+      <material name="black"/>
+      <origin rpy="0 0 0" xyz="${0.006 +0.051/2} ${0.05+0.045/2} ${0.05}"/>
     </visual>
     <!-- This visual represents the  back traction claw f2 support -->
     <visual name = 'back_traction_claw_f2_support'>
       <geometry>
-        <mesh filename="package://mybot_description/meshes/dxl_mx106.dae"/>
-      </geometry>
-      <material name="black"/>
-      <origin rpy="0 0 ${M_PI}" xyz="0.1765 0.075 0.0521"/>
+        <box size="0.051 0.045 0.036 "/>
+      </geometry>
+      <material name="black"/>
+      <origin rpy="0 0 0" xyz="${0.233 -0.006 -0.051/2} ${-0.05-0.045/2} ${0.05}"/>
     </visual>
     <!-- this collision is for the back traction body -->
@@ -380,5 +380,5 @@
     <collision name = 'back_traction_claw_f1_support'>
       <geometry>
-        <mesh filename="package://mybot_description/meshes/dxl_mx106.dae"/>
+        <box size="0.051 0.045 0.036 "/>
       </geometry>
       <origin rpy="0 0 0" xyz="0.0005 -0.075 0.0521"/>
@@ -387,5 +387,5 @@
     <collision name = 'back_traction_claw_f2_support'>
       <geometry>
-        <mesh filename="package://mybot_description/meshes/dxl_mx106.dae"/>
+        <box size="0.051 0.045 0.036 "/>
       </geometry>
       <origin rpy="0 0 ${M_PI}" xyz="0.1765 0.075 0.0521"/>
@@ -401,5 +401,5 @@
     <parent link="tracao_f"/>
     <child link="garra_tracao_f1"/>
-    <origin rpy="0 0 ${M_PI}" xyz="0.0005 0.09 0.06985"/>
+    <origin rpy="0 0 ${M_PI}" xyz="${0.006+0.011} ${0.05+0.028} ${0.05+0.018+0.0045}"/>
     <limit effort="1000.0" lower="-3.14" upper="3.14" velocity="0.5"/>
     <axis xyz="0 0 1"/>
@@ -414,5 +414,5 @@
       </geometry>
       <material name="grey"/>
-      <origin rpy="0 0 0" xyz="0.0 0.012 0.0"/>
+      <origin rpy="0 0 0" xyz="0.0 0.0 0.0"/>
     </visual>
     <!-- this collision is for the front f1 claw unit -->
@@ -421,5 +421,5 @@
         <mesh filename="package://mybot_description/meshes/claw.dae"/>
       </geometry>
-      <origin rpy="0 0 0" xyz="0.0 0.012 0.0"/>
+      <origin rpy="0 0 0" xyz="0.0 0.0 0.0"/>
     </collision>
     <inertial>
@@ -433,5 +433,5 @@
     <parent link="garra_tracao_f1"/>
     <child link="eixo_tracao_f1"/>
-    <origin rpy="0 0 0" xyz="0.0 0.06 0.172"/>
+    <origin rpy="0 0 0" xyz="0.0 0.025 0.172"/>
     <axis xyz="0 1 0"/>
     <dynamics damping="0.7" friction="1.0" />
@@ -443,17 +443,15 @@
     <visual>
       <geometry>
-        <mesh filename="package://mybot_description/meshes/Shaft_piro3_V2.dae"/>
-      </geometry>
-      <material name="grey"/>
-      <!-- <origin rpy="0 0 0" xyz="0.0 0.0 0.0"/> -->
-      <origin rpy="1.57 0 0" xyz="0.0 0.045 0.0"/>
+         <mesh filename="package://mybot_description/meshes/wheel_elir.STL" scale="0.001 0.001 0.001"/>
+      </geometry>
+      <material name="grey"/>
+      <origin rpy="0 0 0" xyz="0.0 0.0 0.0"/>
     </visual>
     <!-- This collision is for the front f1 traction unit -->
     <collision>
       <geometry>
-        <mesh filename="package://mybot_description/meshes/Shaft_piro3_V2.dae"/>
-      </geometry>
-      <!-- <origin rpy="0 0 0" xyz="0.0 0.0 0.0"/> -->
-      <origin rpy="1.57 0 0" xyz="0.0 0.045 0.0"/>
+         <mesh filename="package://mybot_description/meshes/wheel_elir.STL" scale="0.001 0.001 0.001"/>
+      </geometry>
+      <origin rpy="0 0 0" xyz="0.0 0.0 0.0"/>
     </collision>
     <inertial>
@@ -467,5 +465,5 @@
     <parent link="tracao_f"/>
     <child link="garra_tracao_f2"/>
-    <origin rpy="0 0 0" xyz="0.1765 -0.09 0.06985"/>
+    <origin rpy="0 0 0" xyz="${0.233 -0.006 -0.011} ${-0.05-0.028} ${0.05+0.018+0.0045}"/>
     <limit effort="1000.0" lower="-3.14" upper="3.14" velocity="0.5"/>
     <axis xyz="0 0 1"/>
@@ -480,5 +478,5 @@
       </geometry>
       <material name="grey"/>
-      <origin rpy="0 0 0" xyz="0.0 0.012 0.0"/>
+      <origin rpy="0 0 0" xyz="0.0 0.0 0.0"/>
     </visual>
     <!-- this collision is for the front f2 claw unit -->
@@ -487,5 +485,5 @@
         <mesh filename="package://mybot_description/meshes/claw.dae"/>
       </geometry>
-      <origin rpy="0 0 0" xyz="0.0 0.012 0.0"/>
+      <origin rpy="0 0 0" xyz="0.0 0.0 0.0"/>
     </collision>
     <inertial>
@@ -509,17 +507,17 @@
     <visual>
       <geometry>
-        <mesh filename="package://mybot_description/meshes/Shaft_piro3_V2.dae"/>
+         <mesh filename="package://mybot_description/meshes/wheel_elir.STL" scale="0.001 0.001 0.001"/>
       </geometry>
       <!-- <origin rpy="0 0 0" xyz="0.0 0.0 0.0"/> -->
       <material name="grey"/>
-      <origin rpy="1.57 0 0" xyz="0.0 0.055 0.0"/>
+      <origin rpy="0 0 0" xyz="0.0 0.0 0.0"/>
     </visual>
     <!-- This collision is for the front f2 traction unit -->
     <collision>
       <geometry>
-        <mesh filename="package://mybot_description/meshes/Shaft_piro3_V2.dae"/>
+         <mesh filename="package://mybot_description/meshes/wheel_elir.STL" scale="0.001 0.001 0.001"/>
       </geometry>
       <!-- <origin rpy="0 0 0" xyz="0.0 0.0 0.0"/> -->
-      <origin rpy="1.57 0 0" xyz="0.0 0.055 0.0"/>
+      <origin rpy="1.57 0 0" xyz="0.0 0.0 0.0"/>
     </collision>
     <inertial>
@@ -535,5 +533,5 @@
     <parent link="tracao_b"/>
     <child link="garra_tracao_b1"/>
-    <origin rpy="0 0 0" xyz="0.0005 -0.09 0.06985"/>
+    <origin rpy="0 0 ${M_PI}" xyz="${0.006+0.011} ${0.05+0.028} ${0.05+0.018+0.0045}"/>
     <limit effort="1000.0" lower="-3.14" upper="3.14" velocity="0.5"/>
     <axis xyz="0 0 1"/>
@@ -548,5 +546,5 @@
       </geometry>
       <material name="grey"/>
-      <origin rpy="0 0 0" xyz="0.0 0.012 0.0"/>
+      <origin rpy="0 0 0" xyz="0.0 0.0 0.0"/>
     </visual>
     <!-- this collision is for the back t1 claw unit -->
@@ -555,5 +553,5 @@
         <mesh filename="package://mybot_description/meshes/claw.dae"/>
       </geometry>
-      <origin rpy="0 0 0" xyz="0.0 0.012 0.0"/>
+      <origin rpy="0 0 0" xyz="0.0 0.0 0.0"/>
     </collision>
     <inertial>
@@ -578,17 +576,17 @@
     <visual>
       <geometry>
-        <mesh filename="package://mybot_description/meshes/Shaft_piro3_V2.dae"/>
+         <mesh filename="package://mybot_description/meshes/wheel_elir.STL" scale="0.001 0.001 0.001"/>
       </geometry>
       <!-- <origin rpy="0 0 0" xyz="0.0 0.0 0.0"/> -->
       <material name="grey"/>
-      <origin rpy="1.57 0 0" xyz="0.0 0.045 0.0"/>
+      <origin rpy="0 0 0" xyz="0.0 0.0 0.0"/>
     </visual>
     <!-- This collision is for the back t1 traction unit -->
     <collision>
       <geometry>
-        <mesh filename="package://mybot_description/meshes/Shaft_piro3_V2.dae"/>
+         <mesh filename="package://mybot_description/meshes/wheel_elir.STL" scale="0.001 0.001 0.001"/>
       </geometry>
       <!-- <origin rpy="0 0 0" xyz="0.0 0.0 0.0"/> -->
-      <origin rpy="1.57 0 0" xyz="0.0 0.045 0.0"/>
+      <origin rpy="0 0 0" xyz="0.0 0.0 0.0"/>
     </collision>
     <inertial>
@@ -603,5 +601,5 @@
     <parent link="tracao_b"/>
     <child link="garra_tracao_b2"/>
-    <origin rpy="0 0 ${M_PI}" xyz="0.1765 0.09 0.06985"/>
+    <origin rpy="0 0 0" xyz="${0.233 -0.006 -0.011} ${-0.05-0.028} ${0.05+0.018+0.0045}"/>
     <limit effort="1000.0" lower="-3.14" upper="3.14" velocity="0.5"/>
     <axis xyz="0 0 1"/>
@@ -616,5 +614,5 @@
       </geometry>
       <material name="grey"/>
-      <origin rpy="0 0 0" xyz="0.0 0.012 0.0"/>
+      <origin rpy="0 0 0" xyz="0.0 0.0 0.0"/>
     </visual>
     <!-- this collision is for the back t2 claw unit -->
@@ -623,5 +621,5 @@
         <mesh filename="package://mybot_description/meshes/claw.dae"/>
       </geometry>
-      <origin rpy="0 0 0" xyz="0.0 0.012 0.0"/>
+      <origin rpy="0 0 0" xyz="0.0 0.0 0.0"/>
     </collision>
     <inertial>
@@ -646,17 +644,17 @@
     <visual>
       <geometry>
-        <mesh filename="package://mybot_description/meshes/Shaft_piro3_V2.dae"/>
+         <mesh filename="package://mybot_description/meshes/wheel_elir.STL" scale="0.001 0.001 0.001"/>
       </geometry>
       <!-- <origin rpy="0 0 0" xyz="0.0 0.0 0.0"/> -->
       <material name="grey"/>
-      <origin rpy="1.57 0 0" xyz="0.0 0.055 0.0"/>
+      <origin rpy="0 0 0" xyz="0.0 0.0 0.0"/>
     </visual>
     <!-- This collision is for the back t2 traction unit -->
     <collision>
       <geometry>
-        <mesh filename="package://mybot_description/meshes/Shaft_piro3_V2.dae"/>
+         <mesh filename="package://mybot_description/meshes/wheel_elir.STL" scale="0.001 0.001 0.001"/>
       </geometry>
       <!-- <origin rpy="0 0 0" xyz="0.0 0.0 0.0"/> -->
-      <origin rpy="1.57 0 0" xyz="0.0 0.055 0.0"/>
+      <origin rpy="0 0 0" xyz="0.0 0.0 0.0"/>
     </collision>
     <inertial>

Commit message: Modify the wheel mesh and location to aproximate the real model

File: mybot_description/urdf/piro.urdf.xacro (robot description, xacro)
@@ -297,5 +297,5 @@
         <box size="0.051 0.045 0.036 "/>
       </geometry>
-      <material name="black"/>
+      <material name="grey"/>
       <origin rpy="0 0 0" xyz="${0.006 +0.051/2} ${0.05+0.045/2} ${0.05}"/>
     </visual>
@@ -306,5 +306,5 @@
         <box size="0.051 0.045 0.036 "/>
       </geometry>
-      <material name="black"/>
+      <material name="grey"/>
       <origin rpy="0 0 0" xyz="${0.233 -0.006 -0.051/2} ${-0.05-0.045/2} ${0.05}"/>
     </visual>
@@ -359,5 +359,5 @@
         <box size="0.051 0.045 0.036 "/>
       </geometry>
-      <material name="black"/>
+      <material name="grey"/>
       <origin rpy="0 0 0" xyz="${0.006 +0.051/2} ${0.05+0.045/2} ${0.05}"/>
     </visual>
@@ -367,5 +367,5 @@
         <box size="0.051 0.045 0.036 "/>
       </geometry>
-      <material name="black"/>
+      <material name="grey"/>
       <origin rpy="0 0 0" xyz="${0.233 -0.006 -0.051/2} ${-0.05-0.045/2} ${0.05}"/>
     </visual>
@@ -433,5 +433,5 @@
     <parent link="garra_tracao_f1"/>
     <child link="eixo_tracao_f1"/>
-    <origin rpy="0 0 0" xyz="0.0 0.025 0.172"/>
+    <origin rpy="0 0 0" xyz="0.0 ${0.052+0.006} 0.172"/>
     <axis xyz="0 1 0"/>
     <dynamics damping="0.7" friction="1.0" />
@@ -446,5 +446,5 @@
       </geometry>
       <material name="grey"/>
-      <origin rpy="0 0 0" xyz="0.0 0.0 0.0"/>
+      <origin rpy="0 0 0" xyz="-0.0275 0 ${-0.061/2}"/>
     </visual>
     <!-- This collision is for the front f1 traction unit -->
@@ -453,5 +453,5 @@
          <mesh filename="package://mybot_description/meshes/wheel_elir.STL" scale="0.001 0.001 0.001"/>
       </geometry>
-      <origin rpy="0 0 0" xyz="0.0 0.0 0.0"/>
+      <origin rpy="0 0 0" xyz="-0.0275 0 ${-0.061/2}"/>
     </collision>
     <inertial>
@@ -497,5 +497,5 @@
     <parent link="garra_tracao_f2"/>
     <child link="eixo_tracao_f2"/>
-    <origin rpy="0 0 0" xyz="0.0 0.06 0.172"/>
+    <origin rpy="0 0 0" xyz="0.0 ${0.052+0.006} 0.172"/>
     <axis xyz="0 1 0"/>
     <dynamics damping="0.7" friction="1.0" />
@@ -509,7 +509,6 @@
          <mesh filename="package://mybot_description/meshes/wheel_elir.STL" scale="0.001 0.001 0.001"/>
       </geometry>
-      <!-- <origin rpy="0 0 0" xyz="0.0 0.0 0.0"/> -->
-      <material name="grey"/>
-      <origin rpy="0 0 0" xyz="0.0 0.0 0.0"/>
+      <material name="grey"/>
+      <origin rpy="0 0 0" xyz="-0.0275 0 ${-0.061/2}"/>
     </visual>
     <!-- This collision is for the front f2 traction unit -->
@@ -518,6 +517,5 @@
          <mesh filename="package://mybot_description/meshes/wheel_elir.STL" scale="0.001 0.001 0.001"/>
       </geometry>
-      <!-- <origin rpy="0 0 0" xyz="0.0 0.0 0.0"/> -->
-      <origin rpy="1.57 0 0" xyz="0.0 0.0 0.0"/>
+      <origin rpy="0 0 0" xyz="-0.0275 0 ${-0.061/2}"/>
     </collision>
     <inertial>
@@ -566,5 +564,5 @@
     <parent link="garra_tracao_b1"/>
     <child link="eixo_tracao_b1"/>
-    <origin rpy="0 0 0" xyz="0.0 0.06 0.172"/>
+    <origin rpy="0 0 0" xyz="0.0 ${0.052+0.006} 0.172"/>
     <axis xyz="0 1 0"/>
     <dynamics damping="0.7" friction="1.0" />
@@ -578,7 +576,6 @@
          <mesh filename="package://mybot_description/meshes/wheel_elir.STL" scale="0.001 0.001 0.001"/>
       </geometry>
-      <!-- <origin rpy="0 0 0" xyz="0.0 0.0 0.0"/> -->
-      <material name="grey"/>
-      <origin rpy="0 0 0" xyz="0.0 0.0 0.0"/>
+      <material name="grey"/>
+      <origin rpy="0 0 0" xyz="-0.0275 0 ${-0.061/2}"/>
     </visual>
     <!-- This collision is for the back t1 traction unit -->
@@ -587,6 +584,5 @@
          <mesh filename="package://mybot_description/meshes/wheel_elir.STL" scale="0.001 0.001 0.001"/>
       </geometry>
-      <!-- <origin rpy="0 0 0" xyz="0.0 0.0 0.0"/> -->
-      <origin rpy="0 0 0" xyz="0.0 0.0 0.0"/>
+      <origin rpy="0 0 0" xyz="-0.0275 0 ${-0.061/2}"/>
     </collision>
     <inertial>
@@ -634,5 +630,5 @@
     <parent link="garra_tracao_b2"/>
     <child link="eixo_tracao_b2"/>
-    <origin rpy="0 0 0" xyz="0.0 0.06 0.172"/>
+    <origin rpy="0 0 0" xyz="0.0 ${0.052+0.006} 0.172"/>
     <axis xyz="0 1 0"/>
     <dynamics damping="0.7" friction="1.0" />
@@ -646,7 +642,6 @@
          <mesh filename="package://mybot_description/meshes/wheel_elir.STL" scale="0.001 0.001 0.001"/>
       </geometry>
-      <!-- <origin rpy="0 0 0" xyz="0.0 0.0 0.0"/> -->
-      <material name="grey"/>
-      <origin rpy="0 0 0" xyz="0.0 0.0 0.0"/>
+      <material name="grey"/>
+      <origin rpy="0 0 0" xyz="-0.0275 0 ${-0.061/2}"/>
     </visual>
     <!-- This collision is for the back t2 traction unit -->
@@ -655,6 +650,5 @@
          <mesh filename="package://mybot_description/meshes/wheel_elir.STL" scale="0.001 0.001 0.001"/>
       </geometry>
-      <!-- <origin rpy="0 0 0" xyz="0.0 0.0 0.0"/> -->
-      <origin rpy="0 0 0" xyz="0.0 0.0 0.0"/>
+      <origin rpy="0 0 0" xyz="-0.0275 0 ${-0.061/2}"/>
     </collision>
     <inertial>
