Commit message: Add new wheel mesh

File: mybot_description/urdf/piro.urdf.xacro (robot description, xacro)
@@ -112,5 +112,5 @@
     <parent link="garra_ap"/>
     <child link="eixo_tracao_ap"/>
-    <origin rpy="0 0 0" xyz="0.0 0.049 0.172"/>
+    <origin rpy="0 0 0" xyz="0.0 ${0.052+0.006} 0.172"/>
     <axis xyz="0 1 0"/>
     <dynamics damping="0.7" friction="1.0" />
@@ -124,5 +124,5 @@
          <mesh filename="package://mybot_description/meshes/wheel_elir.STL" scale="0.001 0.001 0.001"/>
       </geometry>
-      <origin rpy="0 0 0" xyz="0.0 0.0 0.0"/>
+      <origin rpy="0 0 0" xyz="${-0.030} 0 ${-0.030}"/>
     </visual>
     <!-- This collision is for the central traction unit -->
@@ -131,5 +131,5 @@
          <mesh filename="package://mybot_description/meshes/wheel_elir.STL" scale="0.001 0.001 0.001"/>
       </geometry>
-      <origin rpy="0 0 0" xyz="0.0 0.0 0.0"/>
+      <origin rpy="0 0 0" xyz="${-0.030} 0 ${-0.030}"/>
     </collision>
     <inertial>
@@ -446,5 +446,5 @@
       </geometry>
       <material name="grey"/>
-      <origin rpy="0 0 0" xyz="-0.0275 0 ${-0.061/2}"/>
+      <origin rpy="0 0 0" xyz="-0.03 0 ${-0.061/2}"/>
     </visual>
     <!-- This collision is for the front f1 traction unit -->
@@ -453,5 +453,5 @@
          <mesh filename="package://mybot_description/meshes/wheel_elir.STL" scale="0.001 0.001 0.001"/>
       </geometry>
-      <origin rpy="0 0 0" xyz="-0.0275 0 ${-0.061/2}"/>
+      <origin rpy="0 0 0" xyz="-0.03 0 -0.03"/>
     </collision>
     <inertial>
@@ -510,5 +510,5 @@
       </geometry>
       <material name="grey"/>
-      <origin rpy="0 0 0" xyz="-0.0275 0 ${-0.061/2}"/>
+      <origin rpy="0 0 0" xyz="-0.03 0 -0.03"/>
     </visual>
     <!-- This collision is for the front f2 traction unit -->
@@ -517,5 +517,5 @@
          <mesh filename="package://mybot_description/meshes/wheel_elir.STL" scale="0.001 0.001 0.001"/>
       </geometry>
-      <origin rpy="0 0 0" xyz="-0.0275 0 ${-0.061/2}"/>
+      <origin rpy="0 0 0" xyz="-0.03 0 -0.03"/>
     </collision>
     <inertial>
@@ -577,5 +577,5 @@
       </geometry>
       <material name="grey"/>
-      <origin rpy="0 0 0" xyz="-0.0275 0 ${-0.061/2}"/>
+      <origin rpy="0 0 0" xyz="-0.03 0 -0.03"/>
     </visual>
     <!-- This collision is for the back t1 traction unit -->
@@ -584,5 +584,5 @@
          <mesh filename="package://mybot_description/meshes/wheel_elir.STL" scale="0.001 0.001 0.001"/>
       </geometry>
-      <origin rpy="0 0 0" xyz="-0.0275 0 ${-0.061/2}"/>
+      <origin rpy="0 0 0" xyz="-0.03 0 -0.03"/>
     </collision>
     <inertial>
@@ -643,5 +643,5 @@
       </geometry>
       <material name="grey"/>
-      <origin rpy="0 0 0" xyz="-0.0275 0 ${-0.061/2}"/>
+      <origin rpy="0 0 0" xyz="-0.03 0 -0.03"/>
     </visual>
     <!-- This collision is for the back t2 traction unit -->
@@ -650,5 +650,5 @@
          <mesh filename="package://mybot_description/meshes/wheel_elir.STL" scale="0.001 0.001 0.001"/>
       </geometry>
-      <origin rpy="0 0 0" xyz="-0.0275 0 ${-0.061/2}"/>
+      <origin rpy="0 0 0" xyz="-0.03 0 -0.03"/>
     </collision>
     <inertial>
