Commit message: Change base_joint origin

File: mybot_description/urdf/elir.urdf.xacro (robot description, xacro)
@@ -13,10 +13,10 @@
     <visual name = 'base_body'>
       <geometry>
-        <box size= "0.3219 0.1461 0.2357"/>
+        <box size= "0.01 0.01 0.01"/>
       </geometry>
   </visual>
   </link>
   <joint name="base_joint" type="fixed">
-    <origin xyz="0.0 0.0 0.0" rpy="0.0 0.0 0.0"/>
+    <origin xyz="0.0 0.0 ${0.2357/2}" rpy="0.0 0.0 0.0"/>
     <parent link="base_link"/>
     <child link="box_link"/>

Commit message: Remove dummy base_link visual

File: mybot_description/urdf/elir.urdf.xacro (robot description, xacro)
@@ -10,10 +10,4 @@
   <!-- Parametros do box_link-->
   <link name="base_link">
-    <!-- This visual represents the dummy link for robot base body-->
-    <visual name = 'base_body'>
-      <geometry>
-        <box size= "0.01 0.01 0.01"/>
-      </geometry>
-  </visual>
   </link>
   <joint name="base_joint" type="fixed">
