Commit message: Change robot color to silver

File: elir_description/urdf/elir.urdf.xacro (robot description, xacro)
@@ -25,5 +25,5 @@
         <box size= "0.3219 0.1461 0.2357"/>
       </geometry>
-      <material name="grey"/>
+      <material name="silver"/>
     </visual>
     <!-- This visual represents the central stem -->
@@ -32,5 +32,5 @@
         <box size="0.0367 0.0367 0.279"/>
       </geometry>
-      <material name="grey"/>
+      <material name="silver"/>
       <!-- <xacro:insert_block name="a.test_central_stem_origin" /> -->
       <origin rpy="0 0 0" xyz="0 0.0303 0.23365"/>
@@ -88,5 +88,5 @@
         <mesh filename="package://elir_description/meshes/claw.dae"/>
       </geometry>
-      <material name="grey"/>
+      <material name="silver"/>
     </visual>
     <!-- This collision is for the central claw unit -->
@@ -148,5 +148,5 @@
         <box size="0.185 0.102 0.102"/>
       </geometry>
-      <material name="grey"/>
+      <material name="silver"/>
       <origin rpy="0 0 0" xyz="0.1985 0.0 0.0"/>
     </visual> -->
@@ -156,5 +156,5 @@
         <box size="0.19 0.100 0.05"/>
       </geometry>
-      <material name="grey"/>
+      <material name="silver"/>
       <origin rpy="0 0 0" xyz="0.20995 0.0 0.0"/>
     </visual>
@@ -215,5 +215,5 @@
         <box size="0.185 0.102 0.102"/>
       </geometry>
-      <material name="grey"/>
+      <material name="silver"/>
       <origin rpy="0 0 0" xyz="0.1985 0.0 0.0"/>
     </visual> -->
@@ -223,5 +223,5 @@
         <box size="0.19 0.100 0.05"/>
       </geometry>
-      <material name="grey"/>
+      <material name="silver"/>
       <origin rpy="0 0 0" xyz="0.20995 0.0 0.0"/>
     </visual>
@@ -282,5 +282,5 @@
         <box size="0.233 0.100 0.100"/>
       </geometry>
-      <material name="grey"/>
+      <material name="silver"/>
       <origin rpy="0 0 0" xyz="0.1165 0.0 0.0201"/>
     </visual>
@@ -345,5 +345,5 @@
         <box size="0.233 0.100 0.100"/>
       </geometry>
-      <material name="grey"/>
+      <material name="silver"/>
       <origin rpy="0 0 0" xyz="0.1165 0.0 0.0201"/>
     </visual>
@@ -407,5 +407,5 @@
         <mesh filename="package://elir_description/meshes/claw.dae"/>
       </geometry>
-      <material name="grey"/>
+      <material name="silver"/>
       <origin rpy="0 0 0" xyz="0.0 0.0 0.0"/>
     </visual>
@@ -439,5 +439,5 @@
          <mesh filename="package://elir_description/meshes/wheel_elir.STL" scale="0.001 0.001 0.001"/>
       </geometry>
-      <material name="grey"/>
+      <material name="silver"/>
       <origin rpy="0 0 0" xyz="-0.03 0 ${-0.061/2}"/>
     </visual>
@@ -471,5 +471,5 @@
         <mesh filename="package://elir_description/meshes/claw.dae"/>
       </geometry>
-      <material name="grey"/>
+      <material name="silver"/>
       <origin rpy="0 0 0" xyz="0.0 0.0 0.0"/>
     </visual>
@@ -503,5 +503,5 @@
          <mesh filename="package://elir_description/meshes/wheel_elir.STL" scale="0.001 0.001 0.001"/>
       </geometry>
-      <material name="grey"/>
+      <material name="silver"/>
       <origin rpy="0 0 0" xyz="-0.03 0 -0.03"/>
     </visual>
@@ -537,5 +537,5 @@
         <mesh filename="package://elir_description/meshes/claw.dae"/>
       </geometry>
-      <material name="grey"/>
+      <material name="silver"/>
       <origin rpy="0 0 0" xyz="0.0 0.0 0.0"/>
     </visual>
@@ -570,5 +570,5 @@
          <mesh filename="package://elir_description/meshes/wheel_elir.STL" scale="0.001 0.001 0.001"/>
       </geometry>
-      <material name="grey"/>
+      <material name="silver"/>
       <origin rpy="0 0 0" xyz="-0.03 0 -0.03"/>
     </visual>
@@ -603,5 +603,5 @@
         <mesh filename="package://elir_description/meshes/claw.dae"/>
       </geometry>
-      <material name="grey"/>
+      <material name="silver"/>
       <origin rpy="0 0 0" xyz="0.0 0.0 0.0"/>
     </visual>
@@ -636,5 +636,5 @@
          <mesh filename="package://elir_description/meshes/wheel_elir.STL" scale="0.001 0.001 0.001"/>
       </geometry>
-      <material name="grey"/>
+      <material name="silver"/>
       <origin rpy="0 0 0" xyz="-0.03 0 -0.03"/>
     </visual>

File: elir_description/urdf/materials.xacro (robot description, xacro)
@@ -25,3 +25,6 @@
     <color rgba="1.0 1.0 1.0 1.0"/>
   </material>
+  <material name="silver">
+    <color rgba="${222/255} ${255/255} ${254/255} 1.0"/>
+  </material>
 </robot>

Commit message: Change traction unit from mx106 mesh to box

File: elir_description/urdf/elir.urdf.xacro (robot description, xacro)
@@ -40,5 +40,5 @@
     <visual name = 'central_claw_base'>
       <geometry>
-        <mesh filename="package://elir_description/meshes/dxl_mx106.dae"/>
+        <box size="0.051 0.045 0.036 "/>
       </geometry>
       <material name="black"/>
@@ -62,5 +62,5 @@
     <collision name ='central_claw_base'>
       <geometry>
-        <mesh filename="package://elir_description/meshes/dxl_mx106.dae"/>
+        <box size="0.051 0.045 0.036 "/>
       </geometry>
       <origin rpy="0 0 0" xyz="0.0 0.0722 0.3554"/>

Commit message: Add dummy end-effector to the robots and the urdf to collada convert script

File: elir_description/urdf/elir.urdf.xacro (robot description, xacro)
@@ -211,11 +211,4 @@
   <!-- This link represents the back arm unit  -->
   <link name="link1_f">
-    <!-- <visual>
-      <geometry>
-        <box size="0.185 0.102 0.102"/>
-      </geometry>
-      <material name="silver"/>
-      <origin rpy="0 0 0" xyz="0.1985 0.0 0.0"/>
-    </visual> -->
     <!-- This visual represents the back arm unit -->
     <visual name = 'front_arm'>
@@ -330,4 +323,29 @@
     </inertial>
   </link>
+  <link name="f_eef_ref"/>
+  <joint name="eef_ref_tracao_f" type="fixed">
+    <parent link="tracao_f"/>
+    <child link="f_eef_ref"/>
+    <origin rpy="0 0.0 0" xyz="0.233 0.0 0.0"/>
+    <limit effort="1000.0" lower="-1.0" upper="2.18" velocity="0.5"/>
+    <axis xyz="0 1 0"/>
+  </joint>
+  <joint name="joint_eef_f" type="fixed">
+    <parent link="f_eef_ref"/>
+    <child link="eef_tracao_f"/>
+    <origin rpy="0 0.0 0" xyz="0.0 0.0 0.0"/>
+    <limit effort="1000.0" lower="-1.0" upper="2.18" velocity="0.5"/>
+    <axis xyz="0 1 0"/>
+  </joint>
+  <link name="eef_tracao_f">
+    <!-- This visual represents the front traction body -->
+    <visual name = 'eef_box'>
+      <geometry>
+        <box size="0.01 0.01 0.01"/>
+      </geometry>
+      <material name="black"/>
+      <origin rpy="0 0 0" xyz="${0.01/2} 0.0 0.0"/>
+    </visual>
+  </link>
   <!-- This joint binds the back arm unit (represented by the link link1_t) and the back traction body unit (represented by the link tracao_b). It can rotate with the y axis fixed, it has an upper limit of 2.18 (125 degrees) and a lower limit of -1.0 (-57 degrees) -->
   <joint name="joint2_b" type="revolute">
@@ -390,4 +408,30 @@
       <inertia ixx="0.5622" ixy="0.161" ixz="0.0008" iyy="1.0746" iyz="0.0" izz="1.2126"/>
     </inertial>
+  </link>
+  <!-- This link represents the front traction body unit that contains front traction body, claw f1 support and claw f2 support -->
+  <link name="b_eef_ref"/>
+  <joint name="eef_ref_tracao_b" type="fixed">
+    <parent link="tracao_b"/>
+    <child link="b_eef_ref"/>
+    <origin rpy="0 0.0 0" xyz="0.233 0.0 0.0"/>
+    <limit effort="1000.0" lower="-1.0" upper="2.18" velocity="0.5"/>
+    <axis xyz="0 1 0"/>
+  </joint>
+  <joint name="joint_eef_b" type="fixed">
+    <parent link="b_eef_ref"/>
+    <child link="eef_tracao_b"/>
+    <origin rpy="0 0.0 0" xyz="0.0 0.0 0.0"/>
+    <limit effort="1000.0" lower="-1.0" upper="2.18" velocity="0.5"/>
+    <axis xyz="0 1 0"/>
+  </joint>
+  <link name="eef_tracao_b">
+    <!-- This visual represents the front traction body -->
+    <visual name = 'eef_box'>
+      <geometry>
+        <box size="0.01 0.01 0.01"/>
+      </geometry>
+      <material name="black"/>
+      <origin rpy="0 0 0" xyz="${0.01/2} 0.0 0.0"/>
+    </visual>
   </link>
   <!-- This joint binds the front traction body unit (represented by the link tracao_f) and the front f1 claw unit (represented by the link garra_tracao_f1). It can rotate with the z axis fixed, it has an upper limit of 3.14 (360 degrees) and lower limit of -3.14 (-360 degrees) -->

Commit message: Add trajectory controllers, update world launch

File: elir_description/urdf/elir.urdf.xacro (robot description, xacro)
@@ -800,39 +800,39 @@
       <hardwareInterface>hardware_interface/EffortJointInterface</hardwareInterface>
     </joint>
+    <actuator name="servo13">
+      <hardwareInterface>hardware_interface/EffortJointInterface</hardwareInterface>
+      <mechanicalReduction>1</mechanicalReduction>
+    </actuator>
+</transmission>
+  <transmission name="tran_joint_1b">
+    <type>transmission_interface/SimpleTransmission</type>
+    <joint name="joint1_b">
+      <hardwareInterface>hardware_interface/EffortJointInterface</hardwareInterface>
+    </joint>
+    <actuator name="servo12">
+      <hardwareInterface>hardware_interface/EffortJointInterface</hardwareInterface>
+      <mechanicalReduction>1</mechanicalReduction>
+    </actuator>
+</transmission>
+  <transmission name="tran_joint_2f">
+    <type>transmission_interface/SimpleTransmission</type>
+    <joint name="joint2_f">
+      <hardwareInterface>hardware_interface/EffortJointInterface</hardwareInterface>
+    </joint>
+    <actuator name="servo14">
+      <hardwareInterface>hardware_interface/EffortJointInterface</hardwareInterface>
+      <mechanicalReduction>1</mechanicalReduction>
+    </actuator>
+</transmission>
+  <transmission name="tran_joint_2b">
+    <type>transmission_interface/SimpleTransmission</type>
+    <joint name="joint2_b">
+      <hardwareInterface>hardware_interface/EffortJointInterface</hardwareInterface>
+    </joint>
     <actuator name="servo11">
-      <hardwareInterface>EffortJointInterface</hardwareInterface>
-      <mechanicalReduction>1</mechanicalReduction>
-    </actuator>
-  </transmission>
-  <transmission name="tran_joint_2f">
-    <type>transmission_interface/SimpleTransmission</type>
-    <joint name="joint2_f">
-      <hardwareInterface>hardware_interface/EffortJointInterface</hardwareInterface>
-    </joint>
-    <actuator name="servo13">
-      <hardwareInterface>EffortJointInterface</hardwareInterface>
-      <mechanicalReduction>1</mechanicalReduction>
-    </actuator>
-  </transmission>
-  <transmission name="tran_joint_1t">
-    <type>transmission_interface/SimpleTransmission</type>
-    <joint name="joint1_b">
-      <hardwareInterface>hardware_interface/EffortJointInterface</hardwareInterface>
-    </joint>
-    <actuator name="servo22">
-      <hardwareInterface>EffortJointInterface</hardwareInterface>
-      <mechanicalReduction>1</mechanicalReduction>
-    </actuator>
-  </transmission>
-  <transmission name="tran_joint_2t">
-    <type>transmission_interface/SimpleTransmission</type>
-    <joint name="joint2_b">
-      <hardwareInterface>hardware_interface/EffortJointInterface</hardwareInterface>
-    </joint>
-    <actuator name="servo24">
-      <hardwareInterface>EffortJointInterface</hardwareInterface>
-      <mechanicalReduction>1</mechanicalReduction>
-    </actuator>
-  </transmission>
+      <hardwareInterface>hardware_interface/EffortJointInterface</hardwareInterface>
+      <mechanicalReduction>1</mechanicalReduction>
+    </actuator>
+</transmission>
   <!-- Garras -->
   <transmission name="tran_claw_c1">

Commit message: change joint limits

File: elir_description/urdf/elir.urdf.xacro (robot description, xacro)
@@ -139,5 +139,5 @@
     <!-- <origin rpy=" 0 -0.60 3.141592" xyz="-0.13 0.0 0.079"/> -->
     <origin rpy=" 0 -0.6 ${M_PI}" xyz="-0.13 0.0 0.079"/>
-    <limit effort="1000.0" lower="-1.74" upper="0.7" velocity="0.5"/>
+    <limit effort="1000.0" lower="-3.14" upper="3.14" velocity="0.5"/>
     <axis xyz="0 1 0"/>
   </joint>
@@ -206,5 +206,5 @@
     <!-- <origin rpy="0 -0.60 0" xyz="0.13 0.0 0.079"/> -->
     <origin rpy=" 0 -0.6 0" xyz="0.13 0.0 0.079"/>
-    <limit effort="1000.0" lower="-1.74" upper="0.7" velocity="0.5"/>
+    <limit effort="1000.0" lower="-5" upper="5" velocity="0.5"/>
     <axis xyz="0 1 0"/>
   </joint>
@@ -265,5 +265,5 @@
     <child link="tracao_f"/>
     <origin rpy="0 0.57 0" xyz="0.39 0.0 0.0"/>
-    <limit effort="1000.0" lower="-1.0" upper="2.18" velocity="0.5"/>
+    <limit effort="1000.0" lower="-5" upper="5" velocity="0.5"/>
     <axis xyz="0 1 0"/>
   </joint>
@@ -353,5 +353,5 @@
     <child link="tracao_b"/>
     <origin rpy="0 0.57 0" xyz="0.39 0.0 0.0"/>
-    <limit effort="1000.0" lower="-1.0" upper="2.18" velocity="0.5"/>
+    <limit effort="1000.0" lower="-3.14" upper="3.14" velocity="0.5"/>
     <axis xyz="0 1 0"/>
   </joint>

Commit message: change joint limits

File: elir_description/urdf/elir.urdf.xacro (robot description, xacro)
@@ -206,5 +206,5 @@
     <!-- <origin rpy="0 -0.60 0" xyz="0.13 0.0 0.079"/> -->
     <origin rpy=" 0 -0.6 0" xyz="0.13 0.0 0.079"/>
-    <limit effort="1000.0" lower="-5" upper="5" velocity="0.5"/>
+    <limit effort="1000.0" lower="-3.14" upper="3.14" velocity="0.5"/>
     <axis xyz="0 1 0"/>
   </joint>
@@ -265,5 +265,5 @@
     <child link="tracao_f"/>
     <origin rpy="0 0.57 0" xyz="0.39 0.0 0.0"/>
-    <limit effort="1000.0" lower="-5" upper="5" velocity="0.5"/>
+    <limit effort="1000.0" lower="-3.14" upper="3.14" velocity="0.5"/>
     <axis xyz="0 1 0"/>
   </joint>

Commit message: change joint x location and

File: elir_description/urdf/elir.urdf.xacro (robot description, xacro)
@@ -138,5 +138,5 @@
     <child link="link1_b"/>
     <!-- <origin rpy=" 0 -0.60 3.141592" xyz="-0.13 0.0 0.079"/> -->
-    <origin rpy=" 0 -0.6 ${M_PI}" xyz="-0.13 0.0 0.079"/>
+    <origin rpy=" 0 -0.6 ${M_PI}" xyz="-0.14595 0.0 0.079"/>
     <limit effort="1000.0" lower="-3.14" upper="3.14" velocity="0.5"/>
     <axis xyz="0 1 0"/>
@@ -205,5 +205,5 @@
     <child link="link1_f"/>
     <!-- <origin rpy="0 -0.60 0" xyz="0.13 0.0 0.079"/> -->
-    <origin rpy=" 0 -0.6 0" xyz="0.13 0.0 0.079"/>
+    <origin rpy=" 0 -0.6 0" xyz="0.14595 0.0 0.079"/>
     <limit effort="1000.0" lower="-3.14" upper="3.14" velocity="0.5"/>
     <axis xyz="0 1 0"/>
@@ -264,5 +264,5 @@
     <parent link="link1_f"/>
     <child link="tracao_f"/>
-    <origin rpy="0 0.57 0" xyz="0.39 0.0 0.0"/>
+    <origin rpy="0 0.6 0" xyz="0.39 0.0 0.0"/>
     <limit effort="1000.0" lower="-3.14" upper="3.14" velocity="0.5"/>
     <axis xyz="0 1 0"/>
@@ -352,5 +352,5 @@
     <parent link="link1_b"/>
     <child link="tracao_b"/>
-    <origin rpy="0 0.57 0" xyz="0.39 0.0 0.0"/>
+    <origin rpy="0 0.6 0" xyz="0.39 0.0 0.0"/>
     <limit effort="1000.0" lower="-3.14" upper="3.14" velocity="0.5"/>
     <axis xyz="0 1 0"/>

Commit message: Add trajectory controllers and servers
Add the claw trajectory controllers and the services to open and close the claws;

File: elir_description/urdf/elir.urdf.xacro (robot description, xacro)
@@ -73,5 +73,5 @@
   </link>
   <!-- this joint binds the base body (represented by the link box_link) with the central claw unit (represented by the link garra_ap). It can rotate with the z axis fixed, it has an upper limit of 3,14 (180 degrees) and a lower limit of -3,14 (-180 degrees) -->
-  <joint name="joint_garra_ap" type="revolute">
+  <joint name="joint_garra_tracao_ap" type="revolute">
     <parent link="box_link"/>
     <child link="garra_ap"/>
@@ -795,40 +795,40 @@
   <!-- ROS Control-->
   <!-- Juntas -->
-  <transmission name="tran_joint_1f">
+  <transmission name="transmission_joint_1f">
     <type>transmission_interface/SimpleTransmission</type>
     <joint name="joint1_f">
       <hardwareInterface>hardware_interface/EffortJointInterface</hardwareInterface>
     </joint>
-    <actuator name="servo13">
+    <actuator name="servos_11_12">
       <hardwareInterface>hardware_interface/EffortJointInterface</hardwareInterface>
       <mechanicalReduction>1</mechanicalReduction>
     </actuator>
 </transmission>
-  <transmission name="tran_joint_1b">
+  <transmission name="transmission_joint_1b">
     <type>transmission_interface/SimpleTransmission</type>
     <joint name="joint1_b">
       <hardwareInterface>hardware_interface/EffortJointInterface</hardwareInterface>
     </joint>
-    <actuator name="servo12">
+    <actuator name="servos_111_112">
       <hardwareInterface>hardware_interface/EffortJointInterface</hardwareInterface>
       <mechanicalReduction>1</mechanicalReduction>
     </actuator>
 </transmission>
-  <transmission name="tran_joint_2f">
+  <transmission name="transmission_joint_2f">
     <type>transmission_interface/SimpleTransmission</type>
     <joint name="joint2_f">
       <hardwareInterface>hardware_interface/EffortJointInterface</hardwareInterface>
     </joint>
-    <actuator name="servo14">
+    <actuator name="servos_21_22">
       <hardwareInterface>hardware_interface/EffortJointInterface</hardwareInterface>
       <mechanicalReduction>1</mechanicalReduction>
     </actuator>
 </transmission>
-  <transmission name="tran_joint_2b">
+  <transmission name="transmission_joint_2b">
     <type>transmission_interface/SimpleTransmission</type>
     <joint name="joint2_b">
       <hardwareInterface>hardware_interface/EffortJointInterface</hardwareInterface>
     </joint>
-    <actuator name="servo11">
+    <actuator name="servos_121_122">
       <hardwareInterface>hardware_interface/EffortJointInterface</hardwareInterface>
       <mechanicalReduction>1</mechanicalReduction>
@@ -836,50 +836,50 @@
 </transmission>
   <!-- Garras -->
-  <transmission name="tran_claw_c1">
-    <type>transmission_interface/SimpleTransmission</type>
-    <joint name="joint_garra_ap">
-      <hardwareInterface>hardware_interface/EffortJointInterface</hardwareInterface>
-    </joint>
-    <actuator name="servo9">
+  <transmission name="transmission_claw_ap">
+    <type>transmission_interface/SimpleTransmission</type>
+    <joint name="joint_garra_tracao_ap">
+      <hardwareInterface>hardware_interface/EffortJointInterface</hardwareInterface>
+    </joint>
+    <actuator name="servo_71">
       <hardwareInterface>EffortJointInterface</hardwareInterface>
       <mechanicalReduction>1</mechanicalReduction>
     </actuator>
   </transmission>
-  <transmission name="tran_claw_f1">
+  <transmission name="transmission_claw_f1">
     <type>transmission_interface/SimpleTransmission</type>
     <joint name="joint_garra_tracao_f1">
       <hardwareInterface>hardware_interface/EffortJointInterface</hardwareInterface>
     </joint>
-    <actuator name="servo15">
+    <actuator name="servo_31">
       <hardwareInterface>EffortJointInterface</hardwareInterface>
       <mechanicalReduction>1</mechanicalReduction>
     </actuator>
   </transmission>
-  <transmission name="tran_claw_f2">
+  <transmission name="transmission_claw_f2">
     <type>transmission_interface/SimpleTransmission</type>
     <joint name="joint_garra_tracao_f2">
       <hardwareInterface>hardware_interface/EffortJointInterface</hardwareInterface>
     </joint>
-    <actuator name="servo17">
+    <actuator name="servo_41">
       <hardwareInterface>EffortJointInterface</hardwareInterface>
       <mechanicalReduction>1</mechanicalReduction>
     </actuator>
   </transmission>
-  <transmission name="tran_claw_t1">
+  <transmission name="transmission_claw_b1">
     <type>transmission_interface/SimpleTransmission</type>
     <joint name="joint_garra_tracao_b1">
       <hardwareInterface>hardware_interface/EffortJointInterface</hardwareInterface>
     </joint>
-    <actuator name="servo25">
+    <actuator name="servo_131">
       <hardwareInterface>EffortJointInterface</hardwareInterface>
       <mechanicalReduction>1</mechanicalReduction>
     </actuator>
   </transmission>
-  <transmission name="tran_claw_t2">
+  <transmission name="transmission_claw_b2">
     <type>transmission_interface/SimpleTransmission</type>
     <joint name="joint_garra_tracao_b2">
       <hardwareInterface>hardware_interface/EffortJointInterface</hardwareInterface>
     </joint>
-    <actuator name="servo27">
+    <actuator name="servo_141">
       <hardwareInterface>EffortJointInterface</hardwareInterface>
       <mechanicalReduction>1</mechanicalReduction>
@@ -887,50 +887,50 @@
   </transmission>
   <!-- Velocity Controllers -->
-  <transmission name="tran_tracao_1c">
+  <transmission name="transmission_traction_ap">
     <type>transmission_interface/SimpleTransmission</type>
     <joint name="joint_eixo_tracao_ap">
       <hardwareInterface>hardware_interface/VelocityJointInterface</hardwareInterface>
     </joint>
-    <actuator name="servo10">
+    <actuator name="servo_81">
       <hardwareInterface>VelocityJointInterface</hardwareInterface>
       <mechanicalReduction>1</mechanicalReduction>
     </actuator>
   </transmission>
-  <transmission name="tran_tracao_1f">
+  <transmission name="transmission_traction_f1">
     <type>transmission_interface/SimpleTransmission</type>
     <joint name="joint_eixo_tracao_f1">
       <hardwareInterface>hardware_interface/VelocityJointInterface</hardwareInterface>
     </joint>
-    <actuator name="servo16">
+    <actuator name="servo_51">
       <hardwareInterface>VelocityJointInterface</hardwareInterface>
       <mechanicalReduction>1</mechanicalReduction>
     </actuator>
   </transmission>
-  <transmission name="tran_tracao_2f">
+  <transmission name="transmission_traction_f2">
     <type>transmission_interface/SimpleTransmission</type>
     <joint name="joint_eixo_tracao_f2">
       <hardwareInterface>hardware_interface/VelocityJointInterface</hardwareInterface>
     </joint>
-    <actuator name="servo18">
+    <actuator name="servo_61">
       <hardwareInterface>VelocityJointInterface</hardwareInterface>
       <mechanicalReduction>1</mechanicalReduction>
     </actuator>
   </transmission>
-  <transmission name="tran_tracao_1t">
+  <transmission name="transmission_traction_b1">
     <type>transmission_interface/SimpleTransmission</type>
     <joint name="joint_eixo_tracao_b1">
       <hardwareInterface>hardware_interface/VelocityJointInterface</hardwareInterface>
     </joint>
-    <actuator name="servo26">
+    <actuator name="servo_151">
       <hardwareInterface>VelocityJointInterface</hardwareInterface>
       <mechanicalReduction>1</mechanicalReduction>
     </actuator>
   </transmission>
-  <transmission name="tran_tracao_2t">
+  <transmission name="transmission_traction_b2">
     <type>transmission_interface/SimpleTransmission</type>
     <joint name="joint_eixo_tracao_b2">
       <hardwareInterface>hardware_interface/VelocityJointInterface</hardwareInterface>
     </joint>
-    <actuator name="servo28">
+    <actuator name="servo_161">
       <hardwareInterface>VelocityJointInterface</hardwareInterface>
       <mechanicalReduction>1</mechanicalReduction>
