Commit message: modify f1 and f2 claw locations on URDF

File: elir_description/urdf/elir.urdf.xacro (robot description, xacro)
@@ -285,5 +285,5 @@
       </geometry>
       <material name="grey"/>
-      <origin rpy="0 0 0" xyz="${0.006 +0.051/2} ${0.05+0.045/2} ${0.05}"/>
+      <origin rpy="0 0 0" xyz="${0.006 +0.051/2} -${0.05+0.045/2} ${0.05}"/>
     </visual>
     <!-- This visual represents the front traction claw f1 support -->
@@ -294,5 +294,5 @@
       </geometry>
       <material name="grey"/>
-      <origin rpy="0 0 0" xyz="${0.233 -0.006 -0.051/2} ${-0.05-0.045/2} ${0.05}"/>
+      <origin rpy="0 0 0" xyz="${0.233 -0.006 -0.051/2} ${0.05+0.045/2} ${0.05}"/>
     </visual>
     <!-- this collision is for the front traction body -->
@@ -439,5 +439,5 @@
     <parent link="tracao_f"/>
     <child link="garra_tracao_f1"/>
-    <origin rpy="0 0 ${M_PI}" xyz="${0.006+0.011} ${0.05+0.028} ${0.05+0.018+0.0045}"/>
+    <origin rpy="0 0 0" xyz="${0.006+0.011} -${0.05+0.028} ${0.05+0.018+0.0045}"/>
     <limit effort="1000.0" lower="-3.14" upper="3.14" velocity="0.5"/>
     <axis xyz="0 0 1"/>
@@ -503,5 +503,5 @@
     <parent link="tracao_f"/>
     <child link="garra_tracao_f2"/>
-    <origin rpy="0 0 0" xyz="${0.233 -0.006 -0.011} ${-0.05-0.028} ${0.05+0.018+0.0045}"/>
+    <origin rpy="0 0 ${M_PI}" xyz="${0.233 -0.006 -0.011} ${0.05+0.028} ${0.05+0.018+0.0045}"/>
     <limit effort="1000.0" lower="-3.14" upper="3.14" velocity="0.5"/>
     <axis xyz="0 0 1"/>

Commit message: change joint limits

File: elir_description/urdf/elir.urdf.xacro (robot description, xacro)
@@ -139,5 +139,5 @@
     <!-- <origin rpy=" 0 -0.60 3.141592" xyz="-0.13 0.0 0.079"/> -->
     <origin rpy=" 0 -0.6 ${M_PI}" xyz="-0.14595 0.0 0.079"/>
-    <limit effort="1000.0" lower="-3.14" upper="3.14" velocity="0.5"/>
+    <limit effort="1000.0" lower="-0.7" upper="1.5" velocity="0.5"/>
     <axis xyz="0 1 0"/>
   </joint>
@@ -206,5 +206,5 @@
     <!-- <origin rpy="0 -0.60 0" xyz="0.13 0.0 0.079"/> -->
     <origin rpy=" 0 -0.6 0" xyz="0.14595 0.0 0.079"/>
-    <limit effort="1000.0" lower="-3.14" upper="3.14" velocity="0.5"/>
+    <limit effort="1000.0" lower="-0.7" upper="1.5" velocity="0.5"/>
     <axis xyz="0 1 0"/>
   </joint>
@@ -265,5 +265,5 @@
     <child link="tracao_f"/>
     <origin rpy="0 0.6 0" xyz="0.39 0.0 0.0"/>
-    <limit effort="1000.0" lower="-3.14" upper="3.14" velocity="0.5"/>
+    <limit effort="1000.0" lower="-1.0" upper="1.0" velocity="0.5"/>
     <axis xyz="0 1 0"/>
   </joint>
@@ -353,5 +353,5 @@
     <child link="tracao_b"/>
     <origin rpy="0 0.6 0" xyz="0.39 0.0 0.0"/>
-    <limit effort="1000.0" lower="-3.14" upper="3.14" velocity="0.5"/>
+    <limit effort="1000.0" lower="-1.0" upper="1.0" velocity="0.5"/>
     <axis xyz="0 1 0"/>
   </joint>
